File: hardware/Opto.kicad_sch (KiCad schematic)
At the start: 3 parts, among them U8 PC817

Commit message: added external firmware to repo, add usb connector (molex 4pin 90deg) on schematic
Parts:
- renumbered R31 to R32, R40 to R45, U8 to U9
Changed lines of the file:
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@@
   (symbol (lib_id "Isolator:PC817") (at 153.67 90.17 0)
     (in_bom yes) (on_board yes)
-    (property "Reference" "U8" (id 0) (at 153.67 81.915 0))
+    (property "Reference" "U9" (id 0) (at 153.67 81.915 0))
     (property "Value" "PC817" (id 1) (at 153.67 84.2264 0))
     (property "Footprint" "Package_DIP:DIP-4_W7.62mm" (id 2) (at 148.59 95.25 0)
@@
   (symbol (lib_id "Device:R") (at 140.97 87.63 270)
     (in_bom yes) (on_board yes)
-    (property "Reference" "R31" (id 0) (at 140.97 82.3722 90))
+    (property "Reference" "R32" (id 0) (at 140.97 82.3722 90))
     (property "Value" "3.3k" (id 1) (at 140.97 84.6836 90))
     (property "Footprint" "Resistor_SMD:R_0603_1608Metric" (id 2) (at 140.97 85.852 90)
@@
   (symbol (lib_id "Device:R") (at 162.56 82.55 180)
     (in_bom yes) (on_board yes)
-    (property "Reference" "R40" (id 0) (at 164.338 81.3816 0)
+    (property "Reference" "R45" (id 0) (at 164.338 81.3816 0)
       (effects (font (size 1.27 1.27)) (justify right))
     )

Commit message: added additional USB port and overall board update
Parts:
- renumbered R32 to R31, R45 to R40, U9 to U8
Changed lines of the file:
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@@
   (symbol (lib_id "Isolator:PC817") (at 153.67 90.17 0)
     (in_bom yes) (on_board yes)
-    (property "Reference" "U9" (id 0) (at 153.67 81.915 0))
+    (property "Reference" "U8" (id 0) (at 153.67 81.915 0))
     (property "Value" "PC817" (id 1) (at 153.67 84.2264 0))
     (property "Footprint" "Package_DIP:DIP-4_W7.62mm" (id 2) (at 148.59 95.25 0)
@@
   (symbol (lib_id "Device:R") (at 140.97 87.63 270)
     (in_bom yes) (on_board yes)
-    (property "Reference" "R32" (id 0) (at 140.97 82.3722 90))
+    (property "Reference" "R31" (id 0) (at 140.97 82.3722 90))
     (property "Value" "3.3k" (id 1) (at 140.97 84.6836 90))
     (property "Footprint" "Resistor_SMD:R_0603_1608Metric" (id 2) (at 140.97 85.852 90)
@@
   (symbol (lib_id "Device:R") (at 162.56 82.55 180)
     (in_bom yes) (on_board yes)
-    (property "Reference" "R45" (id 0) (at 164.338 81.3816 0)
+    (property "Reference" "R40" (id 0) (at 164.338 81.3816 0)
       (effects (font (size 1.27 1.27)) (justify right))
     )
@@
   (symbol (lib_id "power:GND") (at 144.78 95.25 0)
     (in_bom yes) (on_board yes)
-    (property "Reference" "#PWR?" (id 0) (at 144.78 101.6 0)
+    (property "Reference" "#PWR0165" (id 0) (at 144.78 101.6 0)
       (effects (font (size 1.27 1.27)) hide)
     )
@@
   (symbol (lib_id "power:GND") (at 162.56 95.25 0)
     (in_bom yes) (on_board yes)
-    (property "Reference" "#PWR?" (id 0) (at 162.56 101.6 0)
+    (property "Reference" "#PWR0164" (id 0) (at 162.56 101.6 0)
       (effects (font (size 1.27 1.27)) hide)
     )
@@
   (symbol (lib_id "power:+3.3V") (at 162.56 77.47 0)
     (in_bom yes) (on_board yes)
-    (property "Reference" "#PWR?" (id 0) (at 162.56 81.28 0)
+    (property "Reference" "#PWR0163" (id 0) (at 162.56 81.28 0)
       (effects (font (size 1.27 1.27)) hide)
     )

Commit message: switched all screw terminals for corresponding molexes n-pins 90 deg
Parts:
- renumbered R31 to R33, R40 to R75, U8 to U10
Changed lines of the file:
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@@
   (symbol (lib_id "Isolator:PC817") (at 153.67 90.17 0)
     (in_bom yes) (on_board yes)
-    (property "Reference" "U8" (id 0) (at 153.67 81.915 0))
+    (property "Reference" "U10" (id 0) (at 153.67 81.915 0))
     (property "Value" "PC817" (id 1) (at 153.67 84.2264 0))
     (property "Footprint" "Package_DIP:DIP-4_W7.62mm" (id 2) (at 148.59 95.25 0)
@@
   (symbol (lib_id "Device:R") (at 140.97 87.63 270)
     (in_bom yes) (on_board yes)
-    (property "Reference" "R31" (id 0) (at 140.97 82.3722 90))
+    (property "Reference" "R33" (id 0) (at 140.97 82.3722 90))
     (property "Value" "3.3k" (id 1) (at 140.97 84.6836 90))
     (property "Footprint" "Resistor_SMD:R_0603_1608Metric" (id 2) (at 140.97 85.852 90)
@@
   (symbol (lib_id "Device:R") (at 162.56 82.55 180)
     (in_bom yes) (on_board yes)
-    (property "Reference" "R40" (id 0) (at 164.338 81.3816 0)
+    (property "Reference" "R75" (id 0) (at 164.338 81.3816 0)
       (effects (font (size 1.27 1.27)) (justify right))
     )
@@
   (symbol (lib_id "power:GND") (at 144.78 95.25 0)
     (in_bom yes) (on_board yes)
-    (property "Reference" "#PWR0165" (id 0) (at 144.78 101.6 0)
+    (property "Reference" "#PWR0162" (id 0) (at 144.78 101.6 0)
       (effects (font (size 1.27 1.27)) hide)
     )
@@
   (symbol (lib_id "power:GND") (at 162.56 95.25 0)
     (in_bom yes) (on_board yes)
-    (property "Reference" "#PWR0164" (id 0) (at 162.56 101.6 0)
+    (property "Reference" "#PWR0161" (id 0) (at 162.56 101.6 0)
       (effects (font (size 1.27 1.27)) hide)
     )
@@
   (symbol (lib_id "power:+3.3V") (at 162.56 77.47 0)
     (in_bom yes) (on_board yes)
-    (property "Reference" "#PWR0163" (id 0) (at 162.56 81.28 0)
+    (property "Reference" "#PWR0160" (id 0) (at 162.56 81.28 0)
       (effects (font (size 1.27 1.27)) hide)
     )

Commit message: fixed HV measurement
Parts:
- renumbered R33 to R32, R75 to R45, U10 to U9
Changed lines of the file:
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@@
   (symbol (lib_id "Isolator:PC817") (at 153.67 90.17 0)
     (in_bom yes) (on_board yes)
-    (property "Reference" "U10" (id 0) (at 153.67 81.915 0))
+    (property "Reference" "U9" (id 0) (at 153.67 81.915 0))
     (property "Value" "PC817" (id 1) (at 153.67 84.2264 0))
     (property "Footprint" "Package_DIP:DIP-4_W7.62mm" (id 2) (at 148.59 95.25 0)
@@
   (symbol (lib_id "Device:R") (at 140.97 87.63 270)
     (in_bom yes) (on_board yes)
-    (property "Reference" "R33" (id 0) (at 140.97 82.3722 90))
+    (property "Reference" "R32" (id 0) (at 140.97 82.3722 90))
     (property "Value" "3.3k" (id 1) (at 140.97 84.6836 90))
     (property "Footprint" "Resistor_SMD:R_0603_1608Metric" (id 2) (at 140.97 85.852 90)
@@
   (symbol (lib_id "Device:R") (at 162.56 82.55 180)
     (in_bom yes) (on_board yes)
-    (property "Reference" "R75" (id 0) (at 164.338 81.3816 0)
+    (property "Reference" "R45" (id 0) (at 164.338 81.3816 0)
       (effects (font (size 1.27 1.27)) (justify right))
     )
@@
   (symbol (lib_id "power:GND") (at 144.78 95.25 0)
     (in_bom yes) (on_board yes)
-    (property "Reference" "#PWR0162" (id 0) (at 144.78 101.6 0)
+    (property "Reference" "#PWR0159" (id 0) (at 144.78 101.6 0)
       (effects (font (size 1.27 1.27)) hide)
     )
@@
   (symbol (lib_id "power:GND") (at 162.56 95.25 0)
     (in_bom yes) (on_board yes)
-    (property "Reference" "#PWR0161" (id 0) (at 162.56 101.6 0)
+    (property "Reference" "#PWR0158" (id 0) (at 162.56 101.6 0)
       (effects (font (size 1.27 1.27)) hide)
     )
@@
   (symbol (lib_id "power:+3.3V") (at 162.56 77.47 0)
     (in_bom yes) (on_board yes)
-    (property "Reference" "#PWR0160" (id 0) (at 162.56 81.28 0)
+    (property "Reference" "#PWR0157" (id 0) (at 162.56 81.28 0)
       (effects (font (size 1.27 1.27)) hide)
     )

Commit message: changed the logic behind the error latch circuit and added some 3d models for used harwin connectors
Parts:
- renumbered R32 to R34, R45 to R44, U9 to U11
Changed lines of the file:
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@@
   (symbol (lib_id "Isolator:PC817") (at 153.67 90.17 0)
     (in_bom yes) (on_board yes)
-    (property "Reference" "U9" (id 0) (at 153.67 81.915 0))
+    (property "Reference" "U11" (id 0) (at 153.67 81.915 0))
     (property "Value" "PC817" (id 1) (at 153.67 84.2264 0))
     (property "Footprint" "Package_DIP:DIP-4_W7.62mm" (id 2) (at 148.59 95.25 0)
@@
   (symbol (lib_id "Device:R") (at 140.97 87.63 270)
     (in_bom yes) (on_board yes)
-    (property "Reference" "R32" (id 0) (at 140.97 82.3722 90))
+    (property "Reference" "R34" (id 0) (at 140.97 82.3722 90))
     (property "Value" "3.3k" (id 1) (at 140.97 84.6836 90))
     (property "Footprint" "Resistor_SMD:R_0603_1608Metric" (id 2) (at 140.97 85.852 90)
@@
   (symbol (lib_id "Device:R") (at 162.56 82.55 180)
     (in_bom yes) (on_board yes)
-    (property "Reference" "R45" (id 0) (at 164.338 81.3816 0)
+    (property "Reference" "R44" (id 0) (at 164.338 81.3816 0)
       (effects (font (size 1.27 1.27)) (justify right))
     )
@@
   (symbol (lib_id "power:GND") (at 144.78 95.25 0)
     (in_bom yes) (on_board yes)
-    (property "Reference" "#PWR0159" (id 0) (at 144.78 101.6 0)
+    (property "Reference" "#PWR0165" (id 0) (at 144.78 101.6 0)
       (effects (font (size 1.27 1.27)) hide)
     )
@@
   (symbol (lib_id "power:GND") (at 162.56 95.25 0)
     (in_bom yes) (on_board yes)
-    (property "Reference" "#PWR0158" (id 0) (at 162.56 101.6 0)
+    (property "Reference" "#PWR0164" (id 0) (at 162.56 101.6 0)
       (effects (font (size 1.27 1.27)) hide)
     )
@@
   (symbol (lib_id "power:+3.3V") (at 162.56 77.47 0)
     (in_bom yes) (on_board yes)
-    (property "Reference" "#PWR0157" (id 0) (at 162.56 81.28 0)
+    (property "Reference" "#PWR0163" (id 0) (at 162.56 81.28 0)
       (effects (font (size 1.27 1.27)) hide)
     )

Commit message: erased all traces, finished USB section, started HV section, swapped most footprints of R to be of the same type 0603 similary with caps (where it could be done), swapped optos for those used in Smart Fuses. Overall cleaned up the schematic of unnecessary circuitry ( gotta get that extra weight off ), also major rearragment of the components
Parts:
- renumbered R34 to R33, R44 to R75, U11 to U10
Changed lines of the file:
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@@
   (symbol (lib_id "Isolator:PC817") (at 153.67 90.17 0)
     (in_bom yes) (on_board yes)
-    (property "Reference" "U11" (id 0) (at 153.67 81.915 0))
+    (property "Reference" "U10" (id 0) (at 153.67 81.915 0))
     (property "Value" "PC817" (id 1) (at 153.67 84.2264 0))
     (property "Footprint" "Package_DIP:DIP-4_W7.62mm" (id 2) (at 148.59 95.25 0)
@@
   (symbol (lib_id "Device:R") (at 140.97 87.63 270)
     (in_bom yes) (on_board yes)
-    (property "Reference" "R34" (id 0) (at 140.97 82.3722 90))
+    (property "Reference" "R33" (id 0) (at 140.97 82.3722 90))
     (property "Value" "3.3k" (id 1) (at 140.97 84.6836 90))
     (property "Footprint" "Resistor_SMD:R_0603_1608Metric" (id 2) (at 140.97 85.852 90)
@@
   (symbol (lib_id "Device:R") (at 162.56 82.55 180)
     (in_bom yes) (on_board yes)
-    (property "Reference" "R44" (id 0) (at 164.338 81.3816 0)
+    (property "Reference" "R75" (id 0) (at 164.338 81.3816 0)
       (effects (font (size 1.27 1.27)) (justify right))
     )
