File: hardware/Safety.kicad_sch (KiCad schematic)
At the start: 1 part, among them K2 ALDP105W

Commit message: finished remaking whole schematic
Parts:
- renumbered K2 to K1
Changed lines of the file:
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@@
   (symbol (lib_id "PUTM_EV_BMS_library:ALDP105W") (at 148.59 78.105 0)
     (in_bom yes) (on_board yes)
-    (property "Reference" "K2" (id 0) (at 148.59 63.7032 0))
+    (property "Reference" "K1" (id 0) (at 148.59 63.7032 0))
     (property "Value" "ALDP105W" (id 1) (at 148.59 66.0146 0))
     (property "Footprint" "RELAY_ALDP105W" (id 2) (at 148.59 78.105 0)

Commit message: added additional USB port and overall board update
Parts:
- renumbered K1 to K3
Connections:
- net PullDownSafety/SIGNAL renamed PullDownSafety/IN
Changed lines of the file:
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@@
+    (stroke (width 0) (type default) (color 0 0 0 0))
+  )
+  (wire (pts (xy 135.89 85.725) (xy 138.43 85.725))
+    (stroke (width 0) (type default) (color 0 0 0 0))
+  )
+  (wire (pts (xy 112.395 85.725) (xy 114.935 85.725))
     (stroke (width 0) (type default) (color 0 0 0 0))
   )
@@
   )
   (wire (pts (xy 158.75 70.485) (xy 161.29 70.485))
-    (stroke (width 0) (type default) (color 0 0 0 0))
-  )
-  (wire (pts (xy 112.395 85.725) (xy 114.935 85.725))
-    (stroke (width 0) (type default) (color 0 0 0 0))
-  )
-  (wire (pts (xy 135.89 85.725) (xy 138.43 85.725))
     (stroke (width 0) (type default) (color 0 0 0 0))
   )
@@
   (symbol (lib_id "power:+5V") (at 137.16 69.215 0)
     (in_bom yes) (on_board yes)
-    (property "Reference" "#PWR?" (id 0) (at 137.16 73.025 0)
+    (property "Reference" "#PWR0128" (id 0) (at 137.16 73.025 0)
       (effects (font (size 1.27 1.27)) hide)
     )
@@
   (symbol (lib_id "PUTM_EV_BMS_library:ALDP105W") (at 148.59 78.105 0)
     (in_bom yes) (on_board yes)
-    (property "Reference" "K1" (id 0) (at 148.59 63.7032 0))
+    (property "Reference" "K3" (id 0) (at 148.59 63.7032 0))
     (property "Value" "ALDP105W" (id 1) (at 148.59 66.0146 0))
     (property "Footprint" "RELAY_ALDP105W" (id 2) (at 148.59 78.105 0)
@@
       (effects (font (size 1.27 1.27)) (justify left top))
     )
-    (pin "SIGNAL" input (at 135.89 85.725 0)
+    (pin "SIGNAL" input (at 114.935 85.725 180)
+      (effects (font (size 1.27 1.27)) (justify left))
+    )
+    (pin "IN" input (at 135.89 85.725 0)
       (effects (font (size 1.27 1.27)) (justify right))
     )
-    (pin "IN" input (at 114.935 85.725 180)
-      (effects (font (size 1.27 1.27)) (justify left))
-    )
   )

Commit message: switched all screw terminals for corresponding molexes n-pins 90 deg
Parts:
- renumbered K3 to K1
Changed lines of the file:
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@@
   (symbol (lib_id "PUTM_EV_BMS_library:ALDP105W") (at 148.59 78.105 0)
     (in_bom yes) (on_board yes)
-    (property "Reference" "K3" (id 0) (at 148.59 63.7032 0))
+    (property "Reference" "K1" (id 0) (at 148.59 63.7032 0))
     (property "Value" "ALDP105W" (id 1) (at 148.59 66.0146 0))
     (property "Footprint" "RELAY_ALDP105W" (id 2) (at 148.59 78.105 0)

Commit message: added missing led for safety indication
Parts:
- renumbered K1 to K2
Changed lines of the file:
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@@
   (symbol (lib_id "power:+5V") (at 137.16 69.215 0)
     (in_bom yes) (on_board yes)
-    (property "Reference" "#PWR0128" (id 0) (at 137.16 73.025 0)
+    (property "Reference" "#PWR0127" (id 0) (at 137.16 73.025 0)
       (effects (font (size 1.27 1.27)) hide)
     )
@@
   (symbol (lib_id "PUTM_EV_BMS_library:ALDP105W") (at 148.59 78.105 0)
     (in_bom yes) (on_board yes)
-    (property "Reference" "K1" (id 0) (at 148.59 63.7032 0))
+    (property "Reference" "K2" (id 0) (at 148.59 63.7032 0))
     (property "Value" "ALDP105W" (id 1) (at 148.59 66.0146 0))
     (property "Footprint" "RELAY_ALDP105W" (id 2) (at 148.59 78.105 0)

Commit message: sync
Parts:
- renumbered K2 to K1
Changed lines of the file:
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@@
   (symbol (lib_id "power:+5V") (at 137.16 69.215 0)
     (in_bom yes) (on_board yes)
-    (property "Reference" "#PWR0127" (id 0) (at 137.16 73.025 0)
+    (property "Reference" "#PWR0128" (id 0) (at 137.16 73.025 0)
       (effects (font (size 1.27 1.27)) hide)
     )
@@
   (symbol (lib_id "PUTM_EV_BMS_library:ALDP105W") (at 148.59 78.105 0)
     (in_bom yes) (on_board yes)
-    (property "Reference" "K2" (id 0) (at 148.59 63.7032 0))
+    (property "Reference" "K1" (id 0) (at 148.59 63.7032 0))
     (property "Value" "ALDP105W" (id 1) (at 148.59 66.0146 0))
     (property "Footprint" "RELAY_ALDP105W" (id 2) (at 148.59 78.105 0)

Commit message: remade pcb so it fits into 100 x 100 mm and some minor modifications
Parts:
- renumbered K1 to K3
Changed lines of the file:
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@@
   (symbol (lib_id "power:+5V") (at 137.16 69.215 0)
     (in_bom yes) (on_board yes)
-    (property "Reference" "#PWR0128" (id 0) (at 137.16 73.025 0)
+    (property "Reference" "#PWR0126" (id 0) (at 137.16 73.025 0)
       (effects (font (size 1.27 1.27)) hide)
     )
@@
   (symbol (lib_id "PUTM_EV_BMS_library:ALDP105W") (at 148.59 78.105 0)
     (in_bom yes) (on_board yes)
-    (property "Reference" "K1" (id 0) (at 148.59 63.7032 0))
+    (property "Reference" "K3" (id 0) (at 148.59 63.7032 0))
     (property "Value" "ALDP105W" (id 1) (at 148.59 66.0146 0))
     (property "Footprint" "RELAY_ALDP105W" (id 2) (at 148.59 78.105 0)
