File: hardware/PwrInsulator.kicad_sch (KiCad schematic)
At the start: 5 parts, among them P1 AM1LS-0303S-NZ

Commit message: minor changes
Parts:
- renumbered C1 to C8, C2 to C9, L1 to L2, P1 to P2, R12 to R15
Changed lines of the file:
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@@
   (symbol (lib_id "Device:L") (at 123.825 88.265 90)
     (in_bom yes) (on_board yes)
-    (property "Reference" "L1" (id 0) (at 123.825 83.439 90))
+    (property "Reference" "L2" (id 0) (at 123.825 83.439 90))
     (property "Value" "6.8uH" (id 1) (at 123.825 85.7504 90))
     (property "Footprint" "Inductor_SMD:L_1206_3216Metric" (id 2) (at 123.825 88.265 0)
@@
   (symbol (lib_id "PUTM_EV_BMS_library:AM1LS-0505S-NZ") (at 142.875 93.345 0)
     (in_bom yes) (on_board yes)
-    (property "Reference" "P1" (id 0) (at 142.875 81.534 0))
+    (property "Reference" "P2" (id 0) (at 142.875 81.534 0))
     (property "Value" "AM1LS-0303S-NZ" (id 1) (at 142.875 83.8454 0))
     (property "Footprint" "AM1LS:AM1LS" (id 2) (at 142.875 93.345 0)
@@
   (symbol (lib_id "Device:C_Small") (at 128.905 93.345 0)
     (in_bom yes) (on_board yes)
-    (property "Reference" "C1" (id 0) (at 123.19 92.075 0)
+    (property "Reference" "C8" (id 0) (at 123.19 92.075 0)
       (effects (font (size 1.27 1.27)) (justify left))
     )
@@
   (symbol (lib_id "Device:R") (at 165.735 93.345 180)
     (in_bom yes) (on_board yes)
-    (property "Reference" "R12" (id 0) (at 167.513 92.1766 0)
+    (property "Reference" "R15" (id 0) (at 167.513 92.1766 0)
       (effects (font (size 1.27 1.27)) (justify right))
     )
@@
   (symbol (lib_id "Device:C_Small") (at 156.845 93.345 0)
     (in_bom yes) (on_board yes)
-    (property "Reference" "C2" (id 0) (at 159.1818 92.1766 0)
+    (property "Reference" "C9" (id 0) (at 159.1818 92.1766 0)
       (effects (font (size 1.27 1.27)) (justify left))
     )

Commit message: schemat sync
Parts:
- P1: renamed from P2; value AM1LS-0303S-NZ -> AM1LS-0505S-NZ
- renumbered C8 to C1, C9 to C2, L2 to L1, R15 to R12
Changed lines of the file:
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@@
   (symbol (lib_id "Device:L") (at 123.825 88.265 90)
     (in_bom yes) (on_board yes)
-    (property "Reference" "L2" (id 0) (at 123.825 83.439 90))
+    (property "Reference" "L1" (id 0) (at 123.825 83.439 90))
     (property "Value" "6.8uH" (id 1) (at 123.825 85.7504 90))
     (property "Footprint" "Inductor_SMD:L_1206_3216Metric" (id 2) (at 123.825 88.265 0)
@@
   (symbol (lib_id "PUTM_EV_BMS_library:AM1LS-0505S-NZ") (at 142.875 93.345 0)
     (in_bom yes) (on_board yes)
-    (property "Reference" "P2" (id 0) (at 142.875 81.534 0))
-    (property "Value" "AM1LS-0303S-NZ" (id 1) (at 142.875 83.8454 0))
+    (property "Reference" "P1" (id 0) (at 142.875 81.534 0))
+    (property "Value" "AM1LS-0505S-NZ" (id 1) (at 142.875 83.8454 0))
     (property "Footprint" "AM1LS:AM1LS" (id 2) (at 142.875 93.345 0)
       (effects (font (size 1.27 1.27)) hide)
@@
   (symbol (lib_id "Device:C_Small") (at 128.905 93.345 0)
     (in_bom yes) (on_board yes)
-    (property "Reference" "C8" (id 0) (at 123.19 92.075 0)
+    (property "Reference" "C1" (id 0) (at 123.19 92.075 0)
       (effects (font (size 1.27 1.27)) (justify left))
     )
@@
   (symbol (lib_id "Device:R") (at 165.735 93.345 180)
     (in_bom yes) (on_board yes)
-    (property "Reference" "R15" (id 0) (at 167.513 92.1766 0)
+    (property "Reference" "R12" (id 0) (at 167.513 92.1766 0)
       (effects (font (size 1.27 1.27)) (justify right))
     )
@@
   (symbol (lib_id "Device:C_Small") (at 156.845 93.345 0)
     (in_bom yes) (on_board yes)
-    (property "Reference" "C9" (id 0) (at 159.1818 92.1766 0)
+    (property "Reference" "C2" (id 0) (at 159.1818 92.1766 0)
       (effects (font (size 1.27 1.27)) (justify left))
     )
