File: hardware/Fan_low_side_driver.kicad_sch (KiCad schematic)
At the start: 3 parts, among them Q2 2N7002

Commit message: done
Parts:
- removed Q2: 2N7002, Package_TO_SOT_SMD:SOT-23, symbol Transistor_FET:2N7002
- added Q21: 2SK3065, Package_TO_SOT_SMD:SOT-89-3, symbol Device:Q_NMOS_GDS
Connections:
- net GND: now also Q21.3 (S)
- net IN: now also Q21.2 (D)
- net at R30.1, R30.1: now also Q21.1 (G)
Changed lines of the file:
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@@
     (effects (font (size 1.27 1.27)) (justify left))
+  )
+  (symbol (lib_id "Device:Q_NMOS_GDS") (at 137.16 82.55 0) (unit 1)
+    (in_bom yes) (on_board yes) (dnp no) (fields_autoplaced)
+    (property "Reference" "Q21" (at 143.51 81.915 0)
+      (effects (font (size 1.27 1.27)) (justify left))
+    )
+    (property "Value" "2SK3065" (at 143.51 84.455 0)
+      (effects (font (size 1.27 1.27)) (justify left))
+    )
+    (property "Footprint" "Package_TO_SOT_SMD:SOT-89-3" (at 142.24 80.01 0)
+      (effects (font (size 1.27 1.27)) hide)
+    )
+    (property "Datasheet" "~" (at 137.16 82.55 0)
+      (effects (font (size 1.27 1.27)) hide)
+    )
+    (pin "1")
+    (pin "2")
+    (pin "3")
+    (instances
+      (project "PUTM_EV_BMS_HV_Master_2021"
+        (path "/b456cffc-d9d7-4c91-91f2-36ec9a65dd1b/ba7f6eba-eb84-4567-9005-77208e6eb457/ce1d9a8b-d4b7-4d85-81bb-9249ce3cc6c9"
+          (reference "Q21") (unit 1)
+        )
+        (path "/b456cffc-d9d7-4c91-91f2-36ec9a65dd1b/ba7f6eba-eb84-4567-9005-77208e6eb457/ec6354b8-3aa0-4986-9bb0-f936060b4d56"
+          (reference "Q15") (unit 1)
+        )
+        (path "/b456cffc-d9d7-4c91-91f2-36ec9a65dd1b/ba7f6eba-eb84-4567-9005-77208e6eb457/4b9fce07-f075-4aec-bd3a-2cc8d2465a53"
+          (reference "Q16") (unit 1)
+        )
+        (path "/b456cffc-d9d7-4c91-91f2-36ec9a65dd1b/ba7f6eba-eb84-4567-9005-77208e6eb457/f0444f92-b7ef-40df-b219-ae3ca6754286"
+          (reference "Q17") (unit 1)
+        )
+        (path "/b456cffc-d9d7-4c91-91f2-36ec9a65dd1b/ba7f6eba-eb84-4567-9005-77208e6eb457/3bdf3e63-db06-4489-843c-40336b7b22f8"
+          (reference "Q18") (unit 1)
+        )
+        (path "/b456cffc-d9d7-4c91-91f2-36ec9a65dd1b/ba7f6eba-eb84-4567-9005-77208e6eb457/daf8b322-01dd-446b-9474-a54548001751"
+          (reference "Q19") (unit 1)
+        )
+        (path "/b456cffc-d9d7-4c91-91f2-36ec9a65dd1b/ba7f6eba-eb84-4567-9005-77208e6eb457/2858aedd-8480-47be-b5f3-f06b807d82d6"
+          (reference "Q20") (unit 1)
+        )
+      )
+    )
   )
   (symbol (lib_id "power:GND") (at 139.7 91.44 0) (unit 1)
@@
         )
       )
-    )
-  )
-  (symbol (lib_id "Transistor_FET:2N7002") (at 137.16 82.55 0) (unit 1)
-    (in_bom yes) (on_board yes) (dnp no)
-    (property "Reference" "Q2" (at 142.3416 81.3816 0)
-      (effects (font (size 1.27 1.27)) (justify left))
-    )
-    (property "Value" "2N7002" (at 142.3416 83.693 0)
-      (effects (font (size 1.27 1.27)) (justify left))
-    )
-    (property "Footprint" "Package_TO_SOT_SMD:SOT-23" (at 142.24 84.455 0)
-      (effects (font (size 1.27 1.27) italic) (justify left) hide)
-    )
-    (property "Datasheet" "https://www.onsemi.com/pub/Collateral/NDS7002A-D.PDF" (at 137.16 82.55 0)
-      (effects (font (size 1.27 1.27)) (justify left) hide)
-    )
-    (pin "1")
-    (pin "2")
-    (pin "3")
-    (instances
-      (project "PUTM_EV_BMS_HV_Master_2021"
-        (path "/b456cffc-d9d7-4c91-91f2-36ec9a65dd1b/6eb4a2b1-8e5b-451b-b593-8aaaa3a4213e"
-          (reference "Q2") (unit 1)
-        )
-        (path "/b456cffc-d9d7-4c91-91f2-36ec9a65dd1b/ba7f6eba-eb84-4567-9005-77208e6eb457"
-          (reference "Q8") (unit 1)
-        )
-        (path "/b456cffc-d9d7-4c91-91f2-36ec9a65dd1b/ba7f6eba-eb84-4567-9005-77208e6eb457/ce1d9a8b-d4b7-4d85-81bb-9249ce3cc6c9"
-          (reference "Q8") (unit 1)
-        )
-        (path "/b456cffc-d9d7-4c91-91f2-36ec9a65dd1b/ba7f6eba-eb84-4567-9005-77208e6eb457/ec6354b8-3aa0-4986-9bb0-f936060b4d56"
-          (reference "Q9") (unit 1)
-        )
-        (path "/b456cffc-d9d7-4c91-91f2-36ec9a65dd1b/ba7f6eba-eb84-4567-9005-77208e6eb457/4b9fce07-f075-4aec-bd3a-2cc8d2465a53"
-          (reference "Q10") (unit 1)
-        )
-        (path "/b456cffc-d9d7-4c91-91f2-36ec9a65dd1b/ba7f6eba-eb84-4567-9005-77208e6eb457/f0444f92-b7ef-40df-b219-ae3ca6754286"
-          (reference "Q11") (unit 1)
-        )
-        (path "/b456cffc-d9d7-4c91-91f2-36ec9a65dd1b/ba7f6eba-eb84-4567-9005-77208e6eb457/3bdf3e63-db06-4489-843c-40336b7b22f8"
-          (reference "Q12") (unit 1)
-        )
-        (path "/b456cffc-d9d7-4c91-91f2-36ec9a65dd1b/ba7f6eba-eb84-4567-9005-77208e6eb457/daf8b322-01dd-446b-9474-a54548001751"
-          (reference "Q13") (unit 1)
-        )
-        (path "/b456cffc-d9d7-4c91-91f2-36ec9a65dd1b/ba7f6eba-eb84-4567-9005-77208e6eb457/2858aedd-8480-47be-b5f3-f06b807d82d6"
-          (reference "Q14") (unit 1)
-        )
-      )

Commit message: updated components to comply with new resolutions
Parts:
- removed Q21: 2SK3065, Package_TO_SOT_SMD:SOT-89-3, symbol Device:Q_NMOS_GDS
- removed R30: 100, Resistor_SMD:R_0603_1608Metric, symbol Device:R_Small
- removed R30: 10K, Resistor_SMD:R_0603_1608Metric, symbol Device:R_Small
