File: hardware/Memory.kicad_sch (KiCad schematic)
At the start: 7 parts, among them J15 Micro_SD_Card_Det_Hirose_DM3AT

Commit message: components layout
Parts:
- removed R82, R83, R84, R85, R87: 10k, Resistor_SMD:R_0603_1608Metric, symbol Device:R_Small
Connections:
- net +3V3: no longer names the net of C53.1, J15.4 (VDD)
