File: hardware/CurrentSense.kicad_sch (KiCad schematic)
At the start: 13 parts, among them IC3 MCP3562T-E_NC, IC4 MCP1501-10E_SN, IC5 REF193GSZ-REEL

Commit message: fixed some footprints; shorted pcb board to 60x100; re-designed the HV & current measuring as well as LTC communication, all are in one TS section;
Parts:
- removed C41, C44: 10uF, Capacitor_SMD:C_0603_1608Metric, symbol Device:C_Small
- removed C42, C43, C46: 100nF, Capacitor_SMD:C_0603_1608Metric, symbol Device:C_Small
- removed C45: 1nF, Capacitor_SMD:C_0603_1608Metric, symbol Device:C_Small
- removed FB2, FB3: GZ1608D601TF, Inductor_SMD:L_0603_1608Metric, symbol Device:Ferrite_Bead_Small
- removed IC3: MCP3562T-E_NC, MCP3561T-E_NC:QFN40P300X300X60-21N-D, symbol MCP3562T-E_NC:MCP3562T-E_NC
- removed IC4: MCP1501-10E_SN, MCP1501-10E_SN:SOIC127P600X175-8N, symbol MCP1501-10E_SN:MCP1501-10E_SN
- removed IC5: REF193GSZ-REEL, MCP1501-10E_SN:SOIC127P600X175-8N, symbol REF196GSZ-REEL:REF196GSZ-REEL
- removed L5, L6: 1mH, Inductor_SMD:L_1206_3216Metric, symbol Device:L_Small
Connections:
- no-connect marks 4 -> 0
Other:
- note removed: "1.024V REF"
- note removed: "Adjustable sens ref for measurments of full range with offset"
- note removed: "Current Sense"
- note removed: "MCP35621T can be used for current sens signal measurements only (can handle any combinasions of inputs) LEM signal = V_REF + 1.25 * CURRENT / 200A in range -100A to 100A it's 0.250V to 1.750V"
- note removed: "Sensor Reference"
