File: hardware/PUTM_EV_BMS_HV_MASTER_2023.kicad_sch (KiCad schematic)
At the start: 19 parts, among them U1 STM32G484RETx, Y1 X322516MLB4SI, Y2 Q13FC1350000400

Commit message: major schematic changes
Parts:
- removed C1, C2: 20pF, Capacitor_SMD:C_0603_1608Metric, symbol Device:C_Small
- removed C3, C4: 25pF, Capacitor_SMD:C_0603_1608Metric, symbol Device:C_Small
- removed D1, D2, D3: SML-D12U1WT86, LED_SMD:LED_0603_1608Metric, symbol Device:LED_Small_ALT
- removed H3: M3, MountingHole:MountingHole_3.2mm_M3_Pad_Via, symbol Mechanical:MountingHole_Pad
- removed R1, R2, R3, R5, R6: 1k, Resistor_SMD:R_0603_1608Metric, symbol Device:R_Small
- removed R4: 10k, Resistor_SMD:R_0603_1608Metric, symbol Device:R_Small
- removed U1: STM32G484RETx, Package_QFP:LQFP-64_10x10mm_P0.5mm, symbol MCU_ST_STM32G4:STM32G484RETx
- removed Y1: X322516MLB4SI, Crystal:Crystal_SMD_3225-4Pin_3.2x2.5mm, symbol Device:Crystal_GND24_Small
- removed Y2: Q13FC1350000400, Crystal:Crystal_SMD_3215-2Pin_3.2x1.5mm, symbol Device:Crystal_Small
- added D4: SP0505BAHT, Package_TO_SOT_SMD:SOT-23-6, symbol Power_Protection:SP0505BAHT
- added D5, D6: CDBU0530, Diode_SMD:D_0603_1608Metric, symbol Device:D_Zener_Small
- added F1: 0ZCH0050FF2G, Fuse:Fuse_1210_3225Metric, symbol Device:Fuse_Small
- added H3, H4: M3, MountingHole:MountingHole_3.2mm_M3, symbol Mechanical:MountingHole
- added J1: M300-MV30645M1, M300-MV30645M1:M300MV30645M1, symbol M300-MV30645M1:M300-MV30645M1
- added J2: M80-5103422, Samacsys:M80-51034YY, symbol Samacsys2:M80-5103422
- added J3: M80-5100442, Samacsys:M80-51004YY, symbol Samacsys2:M80-5100442
- added J4: FTSH-107-01-L-DV-K-A, ftsh-107-01-l-dv-k-a:FTSH-107-XX-YYY-DV-K-A, symbol ftsh-107-01-l-dv-k-a:FTSH-107-01-L-DV-K-A
- added J5: M80-5101422, Samacsys:M80-51014YY, symbol Samacsys2:M80-5101422
- added J6: USB4145-03-0070-C, Samacsys:USB4145030070C, symbol Samacsys2:USB4145-03-0070-C
- added R7, R8: 5.1k, Resistor_SMD:R_0603_1608Metric, symbol Device:R_Small
- added RN1: 33R, Resistor_SMD:R_Array_Convex_8x0602, symbol Device:R_Pack08
Connections:
- net +3V3: now also J4.3 (Pin_3)
- net GND: now also D4.2 (A), D5.2 (A), D6.2 (A), J2.20, J2.22, J2.23, J2.26, J2.27, J2.3, J2.6, J2.9, J3.1, J4.11 (Pin_11), J4.5 (Pin_5), J4.7 (Pin_7), J6.A1 (GND), J6.A12 (GND), J6.B1 (GND), J6.B12 (GND), J6.MH (SHIELD), R7.2, R8.2, RN1.11 (R6.2), RN1.13 (R4.2), RN1.14 (R3.2), RN1.3 (R3.1), RN1.4 (R4.1), RN1.6 (R6.1)
- net MISO: now also RN1.8 (R8.1)
- net MOSI: now also RN1.7 (R7.1)
- net NRST: now also J4.12 (Pin_12)
- net SCK: now also RN1.5 (R5.1)
- net SWCLK: now also J4.6 (Pin_6)
- net SWDIO: now also J4.4 (Pin_4)
- net ~{EXT_CS_I}: now also RN1.1 (R1.1)
- net ~{EXT_CS_V}: now also RN1.2 (R2.1)
- new net: F1.2, J3.3
- new net: J6.B5 (CC2), R7.1
- new net: J6.A5 (CC1), R8.1
- new net +12V: J5.10, J5.11, J5.12, J5.13, J5.14, J5.8, J5.9
- new net +5V: F1.1
- new net AIR Control/AIR_M-: J1.1
- new net AIR Control/AIR_P-: J1.3
- new net AIR Control/AIR_PRE-: J1.2
- new net AIR_M_DETECTION: J2.13
- new net AIR_PRE_DETECTION: J2.12
- new net AIR_P_DETECTION: J2.28
- new net AMS_FAULT_COCKPIT: J2.21
- new net AMS_SAFETY_1: J2.4
- new net AMS_SAFETY_2: J2.5
- new net BOOT0: J2.29
- new net CANFD1+: J2.7
- new net CANFD1-: J2.24
- new net CANFD2+: J2.8
- new net CANFD2-: J2.25
- new net CHARGER_DETECTION: J2.10
- new net CUR_SENS_REF: D5.1 (K), J3.2
- new net CUR_SENS_SIG: D6.1 (K), J3.4
- new net D+: J6.A6 (D+), J6.B6 (D+)
- new net D-: J6.A7 (D-), J6.B7 (D-)
- new net EXT_RESET: J2.11
- new net EX_D+: J2.17
- new net EX_D-: J2.16
- new net EX_VBUS: J2.34
- new net FAN1-: J5.1
- new net FAN2-: J5.2
- new net FAN3-: J5.3
- new net FAN4-: J5.4
- new net FAN5-: J5.5
- new net FAN6-: J5.6
- new net FAN7-: J5.7
- new net IMD_SENSENSOR: J2.30
- new net MISO_C: D4.4 (K), J2.33, RN1.9 (R8.2)
- new net MOSI_C: D4.3 (K), J2.32, RN1.10 (R7.2)
- new net SAFETY_TSMS_IN: J2.1, J2.18
- new net SCK_C: D4.5 (K), J2.31, RN1.12 (R5.2)
- new net TSMS: J1.4, J1.5, J1.6
- new net VBUS: J6.A4 (VBUS), J6.A9 (VBUS), J6.B4 (VBUS), J6.B9 (VBUS)
- new net VDD: J2.19, J2.2
- new net ~{EXT_CS_I}_C: D4.6 (K), J2.14, RN1.16 (R1.2)
- new net ~{EXT_CS_V}_C: D4.1 (K), J2.15, RN1.15 (R2.2)
- no-connect marks 0 -> 9
Other:
- sheet Safeties and related renamed Safety
- removed sheet Measurements
- added sheet AIR Control (AirControl.kicad_sch)
- added sheet Current Sense (CurrentSense.kicad_sch)
- added sheet HV Measurements (HvMeasurements.kicad_sch)
- added sheet MCU (Mcu.kicad_sch)
- added sheet Opto Isolation (OptoIsolation.kicad_sch)
- sheet Fan drivers ports: added FAN1-, FAN2-, FAN3-, FAN4-, FAN5-, FAN6-, FAN7-; removed none
- note added: "AIR CTRL"
- note added: "CURRENT SENS"
- note added: "Debug"
- note added: "Fans"
- note added: "HV Measurements"
- note added: "Main Connector"
- note added: "USB"
- note removed: "Clocks"
- note removed: "MCU"
- note removed: "Miscellaneous"

Commit message: fixed some footprints; shorted pcb board to 60x100; re-designed the HV & current measuring as well as LTC communication, all are in one TS section;
Parts:
- removed D4: SP0505BAHT, Package_TO_SOT_SMD:SOT-23-6, symbol Power_Protection:SP0505BAHT
- removed D5, D6: CDBU0530, Diode_SMD:D_0603_1608Metric, symbol Device:D_Zener_Small
- removed RN1: 33R, Resistor_SMD:R_Array_Convex_8x0602, symbol Device:R_Pack08
- added C18, C58: 100nF/1kV, Capacitor_SMD:C_1812_4532Metric, symbol c2824c562jggacauto:C2824C562JGGACAUTO
- added C27, C40, C44, C49: 22uF, Capacitor_SMD:C_0805_2012Metric, symbol Device:C_Small
- added C30, C34, C36, C39, C41, C42, C43, C46, C47, C48, C50, C51: 100nF, Capacitor_SMD:C_0603_1608Metric, symbol Device:C_Small
- added C31: 10nF, Capacitor_SMD:C_0603_1608Metric, symbol Device:C_Small
- added C35: 4.7uF, Capacitor_SMD:C_0603_1608Metric, symbol Device:C_Small
- added C45: 1nF, Capacitor_SMD:C_0603_1608Metric, symbol Device:C_Small
- added C53: 5.6nF/2000V, Capacitor_SMD:C_3640_9110Metric, symbol c2824c562jggacauto:C2824C562JGGACAUTO
- added D4: ESDA5V3SC5, Package_TO_SOT_SMD:SOT-23-6, symbol Power_Protection:ESDA5V3SC5
- added FB3, FB4: GZ1608D601TF, Inductor_SMD:L_0603_1608Metric, symbol Device:Ferrite_Bead_Small
- added IC10: MCP3564T-E, Package_DFN_QFN:UQFN-20-1EP_3x3mm_P0.4mm_EP1.85x1.85mm, symbol Samacsys_kicad_sym:MCP3564T-E
- added IC11, IC7: ISO6760, Package_SO:SOIC-16W_7.5x10.3mm_P1.27mm, symbol Samacsys_kicad_sym:ISO6760
- added IC3: MCP3562T-E_NC, MCP3561T-E_NC:QFN40P300X300X60-21N-D, symbol MCP3562T-E_NC:MCP3562T-E_NC
- added IC4: MCP1501-10E_SN, MCP1501-10E_SN:SOIC127P600X175-8N, symbol MCP1501-10E_SN:MCP1501-10E_SN
- added IC5, IC9: REF193GSZ-REEL, MCP1501-10E_SN:SOIC127P600X175-8N, symbol REF196GSZ-REEL:REF196GSZ-REEL
- added IC6: UCC12040DVE, Package_SO:SOIC-16W_7.5x10.3mm_P1.27mm, symbol Samacsys2:UCC12040DVE
- added IC8: 3.3V/0.6A, Package_TO_SOT_SMD:SOT-89-3, symbol AP7365-33YRG-13:AP7365-33YRG-13
- added J10, J7: M300-MV10345M1, Samacsys:M300MV10345M1, symbol Samacsys_kicad_sym:M300-MV10345M1
- added J8: M80-5100442, Samacsys:M80-51004YY, symbol Samacsys2:M80-5100442
- added J9: M80-5100622, Samacsys:M80-51006YY, symbol Samacsys2:M80-5100622
- added L6, L7, L8: 4.7uH, Inductor_SMD:L_1206_3216Metric, symbol Device:L_Small
- added R20, R21: 1k, Resistor_SMD:R_0603_1608Metric, symbol Device:R_Small
- added R22: 200R, Resistor_SMD:R_0603_1608Metric, symbol Device:R_Small
- added RD1, RD2: CDMM20M0F2500, CDMM:CDMM, symbol CDMM:CDMM2M50D4000DET
- added U11: LTC6820IMS, Package_SO:MSOP-16_3x4.039mm_P0.5mm, symbol PUTM_EV_BMS_library:LTC6820IMS
Connections:
- net +3V3: now also C27.1, C34.1, C36.1, C41.1, C42.1, C43.1, IC3.18 (DVDD), IC3.19 (AVDD), IC4.1 (VDD), IC4.3 (~{SHDN}), U11.1 (EN), U11.6 (VDD), U11.9 (VDD); no longer J4.3 (Pin_3)
- net +5V: now also L6.1, L7.1
- net CUR_SENS_REF: now also C45.2, IC3.4 (CH1), IC4.7 (OUT), IC4.8 (FB)
- net CUR_SENS_SIG: now also IC3.3 (CH0)
- net GND: now also C27.2, C34.2, C35.2, C36.2, C41.2, C42.2, C43.2, C44.2, C45.1, C46.1, C53.1, IC3.1 (REFIN-), IC3.17 (DGND), IC3.20 (AGND), IC3.21 (EP), IC4.2 (GND), IC4.4 (GND), IC4.5 (GND), IC4.6 (GND), IC5.4 (GND), IC6.2 (GNDP), IC6.4 (SYNC), IC6.6 (NC), IC6.7 (NC), IC6.8 (NC), R21.1, U11.14 (GND)
- net MISO: now also U11.3 (MISO)
- net MOSI: now also U11.2 (MOSI)
- net SCK: now also IC3.12 (SCK), U11.4 (SCK)
- net SDI: now also IC3.13 (SDI)
- net SDO: now also IC3.14 (SDO)
- net ~{SENS_CS}: now also IC3.11 (~{CS})
- net AIR Control/AIR_M- renamed AIR Control/DRAIN1
- net AIR Control/AIR_P- renamed AIR Control/DRAIN3
- net AIR Control/AIR_PRE- renamed AIR Control/DRAIN2
- new net: FB4.1, L8.2
- new net: C44.1, FB3.2, IC5.2 (VSS), IC5.3 (~{SLEEP})
- new net: J7.1 (Pin_1), RD1.1
- new net: C35.1, IC6.1 (EN), IC6.3 (VINP), L7.2
- new net: R20.1, R21.2, U11.15 (ICMP)
- new net: R20.2, U11.16 (IBIAS)
- new net: FB3.1, L6.2
- new net: C49.1, FB4.2, IC9.2 (VSS), IC9.3 (~{SLEEP})
- new net: J10.1 (Pin_1), RD2.1
- new net: D4.2 (K), D4.5 (NC)
- new net +3.3V: J4.3 (Pin_3)
- new net +3.3VISO: C30.1, C31.1, C48.1, C50.2, IC10.18 (DVDD), IC10.19 (AVDD), IC8.3 (VO)
- new net +5VISO: C40.1, C47.2, IC6.13 (SEL), IC6.14 (VISO), IC8.2 (VI), R22.2
- new net 3V_REF: C46.2, C51.2, IC3.2 (REFIN+), IC5.6 (REF_OUT), IC9.6 (REF_OUT)
- new net GNDISO: C30.2, C31.2, C40.2, C47.1, C48.2, C50.1, IC10.17 (DGND), IC10.20 (AGND), IC10.21 (EPAD), IC6.10 (NCS), IC6.11 (NCS), IC6.12 (NCS), IC6.15 (GNDS), IC6.16 (GNDS), IC6.9 (GNDS), IC8.1 (GND), J10.3 (Pin_3), J7.3 (Pin_3), R22.1, RD1.2, RD2.2
- new net HV_+3.3V: C39.1
- new net HV_+5V: L8.1
- new net HV_GND: C39.2, C49.2, C51.1, IC9.4 (GND)
- new net HV_MES+: RD1.3, RD2.3
- new net I+: U11.11 (IP)
- new net I-: U11.10 (IM)
- new net LTC_1_OUT_I+: J9.4
- new net LTC_1_OUT_I-: J9.1
- new net LTC_2_OUT_I+: J9.3
- new net LTC_2_OUT_I-: J9.6
- new net LTC_CHASSIS: C53.2, J9.2, J9.5
- new net MASTER_MODE: U11.12 (MSTR)
- new net PHASE: U11.8 (PHA)
- new net POLARITY: U11.7 (POL)
- new net SLOW: U11.13 (SLOW)
- new net ~{CS}: U11.5 (~{CS})
- no-connect marks 9 -> 24
Other:
- removed sheet Connectors
- removed sheet HV Measurements
- sheet AIR Control ports: added DRAIN1, DRAIN2, DRAIN3, SIGNAL1, SIGNAL2, SIGNAL3, VDD; removed AIR_M-, AIR_P-, AIR_PRE-, SIGNAL_AIR_M, SIGNAL_AIR_P, SIGNAL_AIR_PRE, TSMS
- sheet Opto Isolation ports: added OPT_OUT0, OPT_OUT1, OPT_OUT2, OPT_OUT3, OPT_OUT4, OPT_OUT5, OPT_OUT6, OPT_OUT7, ~{OPT_IN0}, ~{OPT_IN1}, ~{OPT_IN2}, ~{OPT_IN3}, ~{OPT_IN4}, ~{OPT_IN5}, ~{OPT_IN6}, ~{OPT_IN7}; removed AUX_AIR_M, AUX_AIR_P, AUX_AIR_PRE, BOOT, BOOT0, CHARGER, DETECT_AIR_M, DETECT_AIR_P, DETECT_AIR_PRE, DETECT_CHARGER, DETECT_SAFETY, EXT_RESET, IMD, NRST, SENS_IMD, TSMS
- note added: "1.024V REF"
- note added: "24bit ADC"
- note added: "3V REF"
- note added: "Adjustable sens ref for measurments of full range with offset"
- note added: "Current Sense"
- note added: "IN"
- note added: "ISO"
- note added: "LTC SPI"
- note added: "LV"
- note added: "MCP35621T can be used for current sens signal measurements only (can handle any combinasions of inputs) LEM signal = V_REF + 1.25 * CURRENT / 200A in range -100A to 100A it's 0.250V to 1.750V"
- note added: "SPI iso"
- note added: "Sensor Reference"
- note added: "TS"
- note removed: "Connectors"
- note removed: "Debug"
- note removed: "Fan drivers"
- note removed: "Fans"
- note removed: "Measurements"

Commit message: new beginings tbc
Parts:
- removed C44, C49: 22uF, Capacitor_SMD:C_0805_2012Metric, symbol Device:C_Small
- removed C45: 1nF, Capacitor_SMD:C_0603_1608Metric, symbol Device:C_Small
- removed C46, C51: 100nF, Capacitor_SMD:C_0603_1608Metric, symbol Device:C_Small
- removed FB3, FB4: GZ1608D601TF, Inductor_SMD:L_0603_1608Metric, symbol Device:Ferrite_Bead_Small
- removed IC10: MCP3564T-E, Package_DFN_QFN:UQFN-20-1EP_3x3mm_P0.4mm_EP1.85x1.85mm, symbol Samacsys_kicad_sym:MCP3564T-E
- removed IC3: MCP3562T-E_NC, MCP3561T-E_NC:QFN40P300X300X60-21N-D, symbol MCP3562T-E_NC:MCP3562T-E_NC
- removed IC4: MCP1501-10E_SN, MCP1501-10E_SN:SOIC127P600X175-8N, symbol MCP1501-10E_SN:MCP1501-10E_SN
- removed IC5, IC9: REF193GSZ-REEL, MCP1501-10E_SN:SOIC127P600X175-8N, symbol REF196GSZ-REEL:REF196GSZ-REEL
- removed IC6: UCC12040DVE, Package_SO:SOIC-16W_7.5x10.3mm_P1.27mm, symbol Samacsys2:UCC12040DVE
- removed J3, J8: M80-5100442, Samacsys:M80-51004YY, symbol Samacsys2:M80-5100442
- removed J9: M80-5100622, Samacsys:M80-51006YY, symbol Samacsys2:M80-5100622
- removed L6, L7, L8: 4.7uH, Inductor_SMD:L_1206_3216Metric, symbol Device:L_Small
- added C59: 22uF, Capacitor_SMD:C_0805_2012Metric, symbol Device:C_Small
- added IC3: OPA1679-Q1, Package_DFN_QFN:QFN-16-1EP_4x4mm_P0.65mm_EP2.7x2.7mm, symbol Samacsys_kicad_sym:OPA1679-Q1
- added IC4: ADS131M04, Package_DFN_QFN:WQFN-20-1EP_3x3mm_P0.4mm_EP1.7x1.7mm, symbol Samacsys_kicad_sym:ADS131M04
- added IC5: LTC1799, Package_TO_SOT_SMD:SOT-23-5, symbol Samacsys_kicad_sym:LTC1799
- added IC6: LTC6820IMS, Package_SO:MSOP-16_3x4.039mm_P0.5mm, symbol Samacsys_kicad_sym:LTC6820IMS
- added J11, J8: M80-5100442, Samacsys:M80-51004YY, symbol Samacsys_kicad_sym:M80-5100442
- added R26: 8.2k, Resistor_SMD:R_0603_1608Metric, symbol Device:R_Small
- added R27: 0, Resistor_SMD:R_0603_1608Metric, symbol Device:R_Small
- added R30, R31: 1k, Resistor_SMD:R_0603_1608Metric, symbol Device:R_Small
- added U4: UCC12040DVE, Package_SO:SOIC-16W_7.5x10.3mm_P1.27mm, symbol Samacsys_kicad_sym:UCC12040DVE
- C18, C58: value 100nF/1kV -> 10nF/1kV; footprint Capacitor_SMD:C_1812_4532Metric -> Capacitor_SMD:C_1206_3216Metric
- C27: value 22uF -> 220nF; footprint Capacitor_SMD:C_0805_2012Metric -> Capacitor_SMD:C_0603_1608Metric
- C35: value 4.7uF -> 100nF
Connections:
- net +3.3VISO: now also C35.1, C41.2, C42.1, C43.1, IC3.3 (V+), IC4.18 (DVDD), IC4.19 (AVDD), IC5.1 (VDD), IC6.1 (EN), IC6.12 (MSTR), IC6.6 (VIO), IC6.7 (POL), IC6.8 (PHA), IC6.9 (VDD), R26.2
- net +3V3: no longer C27.1, C41.1, C42.1, C43.1
- net +5V: now also C59.1, U4.1 (EN), U4.3 (VINP)
- net +5VISO: now also U4.13 (SEL), U4.14 (VISO)
- net CUR_SENS_REF: now also J11.1 (Pin_1)
- net CUR_SENS_SIG: now also J11.2 (Pin_2)
- net GND: now also C59.2, U4.2 (GNDP), U4.4 (SYNC); no longer C27.2, C35.2, C41.2, C42.2, C43.2, C53.1
- net GNDISO: now also C27.1, C35.2, C41.1, C42.2, C43.2, IC3.10 (V-), IC3.17 (PAD), IC4.17 (DGND), IC4.2 (CH0-), IC4.20 (AGND), IC4.21 (PAD), IC4.4 (CH1-), IC5.2 (GND), IC5.4 (DIV), IC6.13 (SLOW), IC6.14 (GND), J11.3 (Pin_3), J11.4 (Pin_4), R31.1, U4.15 (GNDS), U4.16 (GNDS), U4.9 (GNDS)
- net I+: now also C58.1, IC6.10 (IM)
- net I-: now also C18.1, IC6.11 (IP)
- net OUT-: now reaches C58.2
- net OUT-: now also J8.2 (Pin_2)
- net OUT+: now reaches C18.2
- net OUT+: now also J8.1 (Pin_1)
- net LTC_CHASSIS: no longer names the net of C53.2
- new net: IC5.3 (SET), R26.1
- new net: J8.3 (Pin_3), J8.4 (Pin_4)
- new net: IC3.13 (NC), IC3.16 (NC)
- new net: IC6.15 (ICMP), R30.1, R31.2
- new net: IC6.16 (IBIAS), R30.2
- new net: IC3.1 (-), IC3.15
- new net: IC3.7, IC3.8 (-)
- new net: U4.10 (NC), U4.11 (NC), U4.12 (NC)
- new net: U4.6 (NC), U4.7 (NC), U4.8 (NC)
- new net: C27.2, IC4.16 (CAP)
- new net: IC3.5 (-), IC3.6
- new net 8.192MHZ: IC4.15 (CLKIN), IC5.5 (OUT)
Other:
- removed sheet Current Sense
- note removed: "HV Measurements"
- note removed: "SPI iso"
- moved on the sheet: C18, C30, C31, C50, C53, C58, J10, J5, J7, RD1, RD2

Commit message: changes tbc
Parts:
- removed C36, C39: 100nF, Capacitor_SMD:C_0603_1608Metric, symbol Device:C_Small
- removed U11: LTC6820IMS, Package_SO:MSOP-16_3x4.039mm_P0.5mm, symbol PUTM_EV_BMS_library:LTC6820IMS
- C34: value 100nF -> 10nF
- R20: value 1k -> 0; now not fitted
- R21: value 1k -> 0
- R27: now not fitted
Connections:
- net +3.3VISO: now also R20.2
- net +3V3: no longer C34.1
- net +5V: no longer F1.1
- net +5VISO: now also F1.1, R27.2
- net CUR_SENS_REF: no longer J11.1 (Pin_1)
- net CUR_SENS_SIG: no longer J11.2 (Pin_2)
- net GND: no longer C34.2, R21.1
- net GNDISO: now also C34.2, R21.2; no longer J11.4 (Pin_4)
- net CAR_I_REF: now reaches IC3.11 (+)
- net CAR_I_REF: now also C34.1, R20.1, R21.1, R27.1
- net CAR_I_REF_ADC: now reaches IC3.12 (-)
- net CAR_I_REF_ADC: now also IC3.14, IC4.6 (CH2-)
- net ACU_V_ADC: now reaches IC3.1 (-), IC3.15
- net ACU_V_ADC: now also IC4.1 (CH0+)
- net ACU_V: now reaches IC3.2 (+)
- net CAR_I_ADC: now reaches IC3.7, IC3.8 (-)
- net CAR_I_ADC: now also IC4.5 (CH2+)
- net CAR_I: now reaches IC3.9 (+)
- net at F1.2: now also J11.4 (Pin_4)
- net CAR_V: now reaches IC3.4 (+)
- net CAR_V_ADC: now reaches IC3.5 (-), IC3.6
- net CAR_V_ADC: now also IC4.3 (CH1+)
- no-connect marks 24 -> 16
Other:
- sheet Safety ports: added none; removed AMS_FAULT_LED, AMS_FAULT_MCU, SIGNAL_AIR_M, SIGNAL_AIR_P, SIGNAL_AIR_PRE
- note removed: "1.024V REF"
- moved on the sheet: C35, C41, F1, IC11, IC3A, IC3B, IC3C, IC3D, IC3E, IC5, IC7, J10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

Commit message: sync
Parts:
- removed J11, J8: M80-5100442, Samacsys:M80-51004YY, symbol Samacsys_kicad_sym:M80-5100442
- removed J5: M80-5101422, Samacsys:M80-51014YY, symbol Samacsys2:M80-5101422
- added C36: 10nF/1kV, Capacitor_SMD:C_1206_3216Metric, symbol c2824c562jggacauto:C2824C562JGGACAUTO
- added D5: ESDA5V3SC5, Package_TO_SOT_SMD:SOT-23-6, symbol Power_Protection:ESDA5V3SC5
- added J3: M80-51014XX, Samacsys:M80-51014YY, symbol Samacsys_kicad_sym:M80-51014XX
- added J5, J8: M80-51004XX, Samacsys:M80-51004YY, symbol Samacsys_kicad_sym:M80-51004XX
- added R17, R18: 10k, Resistor_SMD:R_0603_1608Metric, symbol Device:R_Small
- added RN13: 100, Resistor_SMD:R_Array_Convex_4x0603, symbol Device:R_Pack04_Split
- D4: Mouser Price/Stock https://www.mouser.pl/ProductDetail/Nexperia/PESD4USB5BTTS-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 -> https://www.mouser.pl/ProductDetail/STMicroelectronics/ESDA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
Connections:
- net +12V: now also J3.10 (Pin_10), J3.11 (Pin_11), J3.12 (Pin_12), J3.13 (Pin_13), J3.14 (Pin_14), J3.8 (Pin_8), J3.9 (Pin_9)
- net ACU_V: now also RN13.8 (R1.2); no longer IC3.2 (+)
- net CAR_I: now also RN13.6 (R3.2); no longer IC3.9 (+)
- net CAR_I_REF: now also RN13.5 (R4.2); no longer C34.1, IC3.11 (+), R20.1, R21.1, R27.1
- net CAR_I_REF_ADC: now also D4.1 (A), RN13.4 (R4.1)
- net CAR_V: now also RN13.7 (R2.2); no longer IC3.4 (+)
- net FAN1-: now also J3.1 (Pin_1)
- net FAN2-: now also J3.2 (Pin_2)
- net FAN3-: now also J3.3 (Pin_3)
- net FAN4-: now also J3.4 (Pin_4)
- net FAN5-: now also J3.5 (Pin_5)
- net FAN6-: now also J3.6 (Pin_6)
- net FAN7-: now also J3.7 (Pin_7)
- net GND: now also C53.1
- net GNDISO: now also C53.2, D4.2 (K), D4.5 (NC), C36.1, D5.2 (K), D5.5 (NC), J8.4 (Pin_4), R18.2
- net I+: now also D5.3 (A)
- net I-: now also D5.4 (A)
- net OUT+: now also J5.1 (Pin_1)
- net OUT-: now also J5.2 (Pin_2)
- net at F1.2: now also J8.3 (Pin_3)
- net at D4.3 (A): now also R17.1, RN13.3 (R3.1)
- net at D4.4 (A): now also IC3.4 (+), RN13.2 (R2.1)
- net at D4.6 (A): now also IC3.2 (+), RN13.1 (R1.1)
- net HV_MES+: no longer names the net of RD1.3
- net HV_MES+: no longer RD2.3
- new net: C36.2, J5.3 (Pin_3), J5.4 (Pin_4)
- new net: C34.1, IC3.11 (+), R20.1, R21.1, R27.1
- new net: IC3.9 (+), R17.2, R18.1
- no-connect marks 16 -> 18
Other:
- moved on the sheet: C18, C27, C30, C31, C34, C35, C41, C42, C43, C50, C53, C58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

Commit message: sync
Parts:
- removed RD1, RD2: CDMM20M0F2500, CDMM:CDMM, symbol CDMM:CDMM2M50D4000DET
- added J11, J9: CDMM20M0F2500DET, Samacsys:CDMM20M0F2500DET, symbol Samacsys_kicad_sym:CDMM20M0F2500DET
Connections:
- net GNDISO: now also J11.2, J9.2
- net at J7.1 (Pin_1): now also J11.1
- net at J10.1 (Pin_1): now also J9.1
- no-connect marks 18 -> 19
Other:
- sheet Opto Isolation ports: added OPT_IN1, OPT_IN2, OPT_IN3, OPT_IN4, OPT_IN5, OPT_IN6, OPT_IN7, OPT_IN8, ~{OPT_OUT1}, ~{OPT_OUT2}, ~{OPT_OUT3}, ~{OPT_OUT4}, ~{OPT_OUT5}, ~{OPT_OUT6}, ~{OPT_OUT7}, ~{OPT_OUT8}; removed OPT_OUT0, OPT_OUT1, OPT_OUT2, OPT_OUT3, OPT_OUT4, OPT_OUT5, OPT_OUT6, OPT_OUT7, ~{OPT_IN0}, ~{OPT_IN1}, ~{OPT_IN2}, ~{OPT_IN3}, ~{OPT_IN4}, ~{OPT_IN5}, ~{OPT_IN6}, ~{OPT_IN7}
- note removed: "AIR CTRL"
- note removed: "CURRENT SENS"

Commit message: sync
Parts:
- removed J1: M300-MV30645M1, M300-MV30645M1:M300MV30645M1, symbol M300-MV30645M1:M300-MV30645M1
- removed J2: M80-5103422, Samacsys:M80-51034YY, symbol Samacsys2:M80-5103422
- removed J4: FTSH-107-01-L-DV-K-A, ftsh-107-01-l-dv-k-a:FTSH-107-XX-YYY-DV-K-A, symbol ftsh-107-01-l-dv-k-a:FTSH-107-01-L-DV-K-A
- removed J6: USB4145-03-0070-C, Samacsys:USB4145030070C, symbol Samacsys2:USB4145-03-0070-C
- added J1: M80-5100642, Samacsys:M80-51006YY, symbol Samacsys_kicad_sym:M80-5100642
- added J12: M80-51034XX, Samacsys:M80-51034YY, symbol Samacsys_kicad_sym:M80-51034XX
- added J2: USB_C_Receptacle_USB2.0_14P, Connector_USB:USB_C_Receptacle_JAE_DX07S024WJ3R400, symbol Connector:USB_C_Receptacle_USB2.0_14P
- added J4: FTSH-107-01-L-D-K, Samacsys:FTSH-107-XX-YYY-D-K, symbol Samacsys_kicad_sym:FTSH-107-01-L-D-K
- added R16: 120, Resistor_SMD:R_0603_1608Metric, symbol Device:R_Small
Connections:
- net +3.3V: now also J4.3 (Pin_3)
- net AIR Control/DRAIN1: now also J1.1 (Pin_1)
- net AIR Control/DRAIN2: now also J1.2 (Pin_2)
- net AIR Control/DRAIN3: now also J1.3 (Pin_3)
- net AIR_M_DETECTION: now also J12.13 (Pin_13)
- net AIR_PRE_DETECTION: now also J12.12 (Pin_12)
- net AIR_P_DETECTION: now also J12.28 (Pin_28)
- net AMS_FAULT_COCKPIT: now also J12.21 (Pin_21)
- net AMS_SAFETY_1: now also J12.4 (Pin_4)
- net AMS_SAFETY_2: now also J12.5 (Pin_5)
- net BOOT0: now also J12.29 (Pin_29)
- net CANFD1+: now also J12.7 (Pin_7)
- net CANFD1-: now also J12.24 (Pin_24)
- net CANFD2+: now also J12.8 (Pin_8)
- net CANFD2-: now also J12.25 (Pin_25)
- net CHARGER_DETECTION: now also J12.10 (Pin_10)
- net D+: now also J2.A6 (D+), J2.B6 (D+)
- net D-: now also J2.A7 (D-), J2.B7 (D-)
- net EXT_RESET: now also J12.11 (Pin_11)
- net EX_D+: now also J12.17 (Pin_17)
- net EX_D-: now also J12.16 (Pin_16)
- net EX_VBUS: now also J12.34 (Pin_34)
- net GND: now also J12.20 (Pin_20), J12.22 (Pin_22), J12.23 (Pin_23), J12.26 (Pin_26), J12.27 (Pin_27), J12.3 (Pin_3), J12.6 (Pin_6), J12.9 (Pin_9), J2.A1 (GND), J2.A12 (GND), J2.B1 (GND), J2.B12 (GND), J2.S1 (SHIELD), J4.11 (Pin_11), J4.5 (Pin_5), J4.7 (Pin_7)
- net I+: now also R16.2
- net I-: now also R16.1
- net IMD_SENSENSOR: now also J12.30 (Pin_30)
- net MISO_C: now also J12.33 (Pin_33)
- net MOSI_C: now also J12.32 (Pin_32)
- net NRST: now also J4.12 (Pin_12)
- net SAFETY_TSMS_IN: now also J12.1 (Pin_1), J12.18 (Pin_18)
- net SCK_C: now also J12.31 (Pin_31)
- net SWCLK: now also J4.6 (Pin_6)
- net SWDIO: now also J4.4 (Pin_4)
- net TSMS: now also J1.4 (Pin_4), J1.5 (Pin_5), J1.6 (Pin_6)
- net VBUS: now also J2.A4 (VBUS), J2.A9 (VBUS), J2.B4 (VBUS), J2.B9 (VBUS)
- net VDD: now also J12.19 (Pin_19), J12.2 (Pin_2)
- net ~{EXT_CS_I}_C: now also J12.14 (Pin_14)
- net ~{EXT_CS_V}_C: now also J12.15 (Pin_15)
- net at R7.1: now also J2.B5 (CC2)
- net at R8.1: now also J2.A5 (CC1)
- no-connect marks 19 -> 17
