File: hardware/PUTM_EV_BMS_HV_MASTER_2023.kicad_sch (KiCad schematic)
At the start: 56 parts, among them IC11 ISO6760, IC3 OPA1679-Q1, IC4 ADS131M04, IC5 LTC1799, IC6 LTC6820IMS, IC7 ISO6760, IC8 3.3V/0.6A, J1 M80-5100642, J10 M300-MV10345M1, J11 CDMM20M0F2500DET, J12 M80-51034XX, J2 USB_C_Receptacle_USB2.0_14P, J3 M80-51014XX, J4 FTSH-107-01-L-D-K, J5 M80-51004XX, J7 M300-MV10345M1, J8 M80-51004XX, J9 CDMM20M0F2500DET, U4 UCC12040DVE

Commit message: sync
Parts:
- removed C18, C58: 10nF/1kV, Capacitor_SMD:C_1206_3216Metric, symbol c2824c562jggacauto:C2824C562JGGACAUTO
- removed C27: 220nF, Capacitor_SMD:C_0603_1608Metric, symbol Device:C_Small
- removed C30, C35, C41, C42, C43, C50: 100nF, Capacitor_SMD:C_0603_1608Metric, symbol Device:C_Small
- removed C31, C34: 10nF, Capacitor_SMD:C_0603_1608Metric, symbol Device:C_Small
- removed D4, D5: ESDA5V3SC5, Package_TO_SOT_SMD:SOT-23-6, symbol Power_Protection:ESDA5V3SC5
- removed F1: 0ZCH0050FF2G, Fuse:Fuse_1210_3225Metric, symbol Device:Fuse_Small
- removed IC3: OPA1679-Q1, Package_DFN_QFN:QFN-16-1EP_4x4mm_P0.65mm_EP2.7x2.7mm, symbol Samacsys_kicad_sym:OPA1679-Q1
- removed IC4: ADS131M04, Package_DFN_QFN:WQFN-20-1EP_3x3mm_P0.4mm_EP1.7x1.7mm, symbol Samacsys_kicad_sym:ADS131M04
- removed IC5: LTC1799, Package_TO_SOT_SMD:SOT-23-5, symbol Samacsys_kicad_sym:LTC1799
- removed IC6: LTC6820IMS, Package_SO:MSOP-16_3x4.039mm_P0.5mm, symbol Samacsys_kicad_sym:LTC6820IMS
- removed J11, J9: CDMM20M0F2500DET, Samacsys:CDMM20M0F2500DET, symbol Samacsys_kicad_sym:CDMM20M0F2500DET
- removed R16: 120, Resistor_SMD:R_0603_1608Metric, symbol Device:R_Small
- removed R17, R18: 10k, Resistor_SMD:R_0603_1608Metric, symbol Device:R_Small
- removed R20, R21, R27: 0, Resistor_SMD:R_0603_1608Metric, symbol Device:R_Small
- removed R26: 8.2k, Resistor_SMD:R_0603_1608Metric, symbol Device:R_Small
- removed R30, R31: 1k, Resistor_SMD:R_0603_1608Metric, symbol Device:R_Small
- removed R7, R8: 5.1k, Resistor_SMD:R_0603_1608Metric, symbol Device:R_Small
- removed RN13: 100, Resistor_SMD:R_Array_Convex_4x0603, symbol Device:R_Pack04_Split
- added C39, C44, C45, C46: 100nF, Capacitor_SMD:C_0603_1608Metric, symbol Device:C_Small
- added D1, D2, D3, D6: SML-D12U1WT86, LED_SMD:LED_0603_1608Metric, symbol Device:LED_Small_ALT
- added F1: 0ZCH0050FF2G, Fuse:Fuse_1210_3225Metric, symbol Device:Polyfuse_Small
- added JP1: Jumper_3_Bridged12, Jumper:SolderJumper-3_P1.3mm_Bridged2Bar12_RoundedPad1.0x1.5mm, symbol Jumper:Jumper_3_Bridged12
- added RN16: 1k, Resistor_SMD:R_Array_Convex_4x0603, symbol Device:R_Pack04_Split
Connections:
- net EX_VBUS is gone; now on net GND: J12.34 (Pin_34)
- net +3.3VISO: now also IC11.1 (VCC1), IC7.16 (VCC2), C44.1, C46.1, JP1.3 (B)
- net +3V3: now also IC11.16 (VCC2), IC7.1 (VCC1), C39.1, C45.1, D1.2 (A), D2.2 (A), D3.2 (A), D6.2 (A)
- net +5VISO: now also JP1.1 (A)
- net FAN1-: no longer J3.1 (Pin_1)
- net FAN2-: no longer J3.2 (Pin_2)
- net FAN3-: no longer J3.3 (Pin_3)
- net FAN4-: no longer J3.4 (Pin_4)
- net FAN5-: no longer J3.5 (Pin_5)
- net FAN6-: no longer J3.6 (Pin_6)
- net FAN7-: no longer J3.7 (Pin_7)
- net GND: now also IC11.9 (GND2), IC7.8 (GND1), C39.2, C45.2
- net GNDISO: now also IC11.5 (IND), IC11.6 (INE), IC11.7 (INF), IC11.8 (GND1), IC7.9 (GND2), C44.2, C46.2
- net Isolated ADC/CAR_I: now reaches J8.1 (Pin_1)
- net Isolated ADC/CAR_I_REF: now reaches J8.2 (Pin_2)
- net I_VDDISO: now reaches J8.3 (Pin_3)
- net I_VDDISO: now also F1.2
- net SHIELD: now reaches C36.2, J5.3 (Pin_3), J5.4 (Pin_4)
- net Isolated ADC/ACU_V: now reaches J7.1 (Pin_1)
- net MCU/LTC_MISO: now reaches IC11.13 (OUTC)
- net MCU/ADC_MISO: now reaches IC11.14 (OUTB)
- net MCU/~{ADC_DRY}: now reaches IC11.15 (OUTA)
- net ~{ISO_ADC_DRY}: now reaches IC11.2 (INA)
- net ISO_ADC_MISO: now reaches IC11.3 (INB)
- net ISO_LTC_MISO: now reaches IC11.4 (INC)
- net Isolated ADC/CAR_V: now reaches J10.1 (Pin_1)
- net ~{ISO_LTC_CS}: now reaches IC7.10 (OUTF)
- net ISO_LTC_SCK: now reaches IC7.11 (OUTE)
- net ISO_LTC_MOSI: now reaches IC7.12 (OUTD)
- net ~{ISO_ADC_CS}: now reaches IC7.13 (OUTC)
- net ISO_ADC_SCK: now reaches IC7.14 (OUTB)
- net ISO_ADC_MOSI: now reaches IC7.15 (OUTA)
- net MCU/ADC_MOSI: now reaches IC7.2 (INA)
- net MCU/ADC_SCK: now reaches IC7.3 (INB)
- net MCU/~{ADC_CS}: now reaches IC7.4 (INC)
- net MCU/LTC_MOSI: now reaches IC7.5 (IND)
- net MCU/LTC_SCK: now reaches IC7.6 (INE)
- net MCU/~{LTC_CS}: now reaches IC7.7 (INF)
- net AIR Control/DRAIN1 renamed AIR_M
- net AIR Control/DRAIN2 renamed AIR_P
- net AIR Control/DRAIN3 renamed AIR_PRE
- net EX_D+: no longer names the net of J12.17 (Pin_17)
- net EX_D-: no longer names the net of J12.16 (Pin_16)
- net OUT+ renamed Isolated SPI/OUT-
- net OUT- renamed Isolated SPI/OUT+
- net VBUS: no longer names the net of J2.A4 (VBUS), J2.A9 (VBUS), J2.B4 (VBUS), J2.B9 (VBUS)
- new net: F1.1, JP1.2 (C)
- new net AMS_ERR: D6.1 (K), RN16.4 (R4.1)
- new net AMS_ERROR: RN16.5 (R4.2)
- new net Fan drivers/FAN1-: J3.1 (Pin_1)
- new net Fan drivers/FAN2-: J3.2 (Pin_2)
- new net Fan drivers/FAN3-: J3.3 (Pin_3)
- new net Fan drivers/FAN4-: J3.4 (Pin_4)
- new net Fan drivers/FAN5-: J3.5 (Pin_5)
- new net Fan drivers/FAN6-: J3.6 (Pin_6)
- new net Fan drivers/FAN7-: J3.7 (Pin_7)
- new net LED1: D3.1 (K), RN16.3 (R3.1)
- new net LED2: D2.1 (K), RN16.2 (R2.1)
- new net LED3: D1.1 (K), RN16.1 (R1.1)
- new net SIGNAL_LED_1: RN16.6 (R3.2)
- new net SIGNAL_LED_2: RN16.7 (R2.2)
- new net SIGNAL_LED_3: RN16.8 (R1.2)
- no-connect marks 17 -> 18
Other:
- removed sheet Communication
- added sheet Connectivity (Connectivity.kicad_sch)
- added sheet Isolated ADC (IsolatedADC.kicad_sch)
- added sheet Isolated SPI (IsolatedSPI.kicad_sch)
- sheet MCU ports: added ADC_MISO, ADC_MOSI, ADC_SCK, BOOT, DETECT_AIR_M, DETECT_AIR_P, DETECT_AIR_PRE, DETECT_CHARGER, DETECT_TSMS, FAN_1_CTRL, FAN_2_CTRL, FAN_3_CTRL, FAN_4_CTRL, FAN_5_CTRL, FAN_6_CTRL, FAN_7_CTRL, LTC_MISO, LTC_MOSI, LTC_SCK, MCU_CANFD1_RX, MCU_CANFD1_TX, MCU_CANFD2_RX, MCU_CANFD2_TX, MCU_D+, MCU_D-, NRST, SENS_IMD, SIGNAL_AIR_M, SIGNAL_AIR_P, SIGNAL_AIR_PRE, SIGNAL_AMS_FAULT, SIGNAL_LED_1, SIGNAL_LED_2, SIGNAL_LED_3, SWCLK, SWDIO, ~{ADC_CS}, ~{ADC_DRY}, ~{EXT_CS}, ~{LTC_CS}; removed none
- sheet Safety ports: added LED_ERR, MCU_AMS_FAULT; removed none
- note added: "AIR CONNECTORS"
- note added: "AIR CONTROL"
- note added: "EX_D+"
- note added: "EX_D-"
- note added: "FAN CONNECTORS"
- note added: "FAN CONTROL"
- note added: "GALVANIC ISOLATION"
- note added: "HV CONNECTORS"
- note added: "ISO CONNECTORS"
- note added: "ISO POWER"
- note added: "LEDS"
- note added: "MAIN CONNECTOR"
- note added: "MCU"
- note added: "MISC"
- note added: "PERFS"
- note added: "POWER"
- note added: "SAFETY"
- note added: "SWD CONNECTOR"
- note added: "USB CONNECTOR"
- note removed: "24bit ADC"
- note removed: "3V REF"
- note removed: "Adjustable sens ref for measurments of full range with offset"
- note removed: "Communication"
- note removed: "Current Sense"
- note removed: "IN"
- note removed: "LTC SPI"
- note removed: "MCP35621T can be used for current sens signal measurements only (can handle any combinasions of inputs) LEM signal = V_REF + 1.25 * CURRENT / 200A in range -100A to 100A it's 0.250V to 1.750V"
- note removed: "Main Connector"
- note removed: "Power"
- note removed: "Safeties and related"
- note removed: "Sensor Reference"
- note removed: "USB"
- moved on the sheet: C36, C40, C47, C48, C53, C59, H1, H2, H3, H4, IC11, IC7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

Commit message: schematic done
Parts:
- removed H1, H2, H3, H4: M3, MountingHole:MountingHole_3.2mm_M3, symbol Mechanical:MountingHole
- removed JP1: Jumper_3_Bridged12, Jumper:SolderJumper-3_P1.3mm_Bridged2Bar12_RoundedPad1.0x1.5mm, symbol Jumper:Jumper_3_Bridged12
- added C15: 100nF, Capacitor_SMD:C_0603_1608Metric, symbol Device:C_Small
- added IC9: TPL7407LADR, Package_SO:SOIC-16_3.9x9.9mm_P1.27mm, symbol Samacsys_kicad_sym:TPL7407LADR
Connections:
- net +3V3 is gone; now on net +3.3V: C39.1, C45.1, D1.2 (A), D2.2 (A), D3.2 (A), D6.2 (A), IC11.16 (VCC2), IC7.1 (VCC1)
- net AMS_FAULT_COCKPIT is gone; now on net GND: J12.21 (Pin_21)
- net Fan drivers/FAN1- is gone; now on net FAN1-: J3.1 (Pin_1)
- net Fan drivers/FAN2- is gone; now on net FAN2-: J3.2 (Pin_2)
- net Fan drivers/FAN3- is gone; now on net FAN3-: J3.3 (Pin_3)
- net Fan drivers/FAN4- is gone; now on net FAN4-: J3.4 (Pin_4)
- net Fan drivers/FAN5- is gone; now on net FAN5-: J3.5 (Pin_5)
- net Fan drivers/FAN6- is gone; now on net FAN6-: J3.6 (Pin_6)
- net Fan drivers/FAN7- is gone; now on net FAN7-: J3.7 (Pin_7)
- net SAFETY_TSMS_IN is gone; now on net TSMS: J12.1 (Pin_1), J12.18 (Pin_18)
- net ~{EXT_CS_I}_C is gone; now on net GND: J12.14 (Pin_14)
- net +5VISO: now also F1.1
- net CANFD1+: now also J12.25 (Pin_25); no longer J12.7 (Pin_7)
- net CANFD2-: now also J12.7 (Pin_7); no longer J12.25 (Pin_25)
- net D+: now also J12.17 (Pin_17)
- net D-: now also J12.16 (Pin_16)
- net FAN1-: now also IC9.16 (OUT1)
- net FAN2-: now also IC9.15 (OUT2)
- net FAN3-: now also IC9.14 (OUT3)
- net FAN4-: now also IC9.13 (OUT4)
- net FAN5-: now also IC9.12 (OUT5)
- net FAN6-: now also IC9.11 (OUT6)
- net FAN7-: now also IC9.10 (OUT7)
- net GND: now also C15.1, IC9.8 (GND)
- net VDD: now also C15.2, IC9.9 (COM)
- net AMS_SAFETY_1 renamed SAFETY1
- net AMS_SAFETY_2 renamed SAFETY2
- net EXT_RESET renamed EXT_NRST
- net MISO_C renamed EXT_MISO
- net MOSI_C renamed EXT_MOSI
- net SCK_C renamed EXT_SCK
- new net MCU/FAN_1_CTRL: IC9.1 (IN1)
- new net MCU/FAN_2_CTRL: IC9.2 (IN2)
- new net MCU/FAN_3_CTRL: IC9.3 (IN3)
- new net MCU/FAN_4_CTRL: IC9.4 (IN4)
- new net MCU/FAN_5_CTRL: IC9.5 (IN5)
- new net MCU/FAN_6_CTRL: IC9.6 (IN6)
- new net MCU/FAN_7_CTRL: IC9.7 (IN7)
Other:
- removed sheet Fan drivers
- removed sheet Opto Isolation
- sheet Connectivity ports: added AIR1_I, AIR1_O, AIR2_I, AIR2_O, AIR3_I, AIR3_O, BOOT0_I, BOOT0_O, MV_I1, MV_I2, MV_I3, MV_O1, MV_O2, MV_O3, NRST_I, NRST_O, SPI_I1, SPI_I2, SPI_I3, SPI_I4, SPI_O1, SPI_O2, SPI_O3, SPI_O4; removed IN1, IN2, IN3, IN4, OUT1, OUT2, OUT3, OUT4
- sheet MCU ports: added BOOT0, EXT_MISO, EXT_MOSI, EXT_SCK; removed BOOT
- sheet Safety ports: added SAFETY1, SAFETY2; removed none
- note added: "ADC AND SPI"
- note added: "CONNECTIVITY"
- note removed: "EX_D+"
- note removed: "EX_D-"
- note removed: "MISC"
- note removed: "PERFS"
- moved on the sheet: D1, D2, D3, D6, F1, J1, J3, RN16A, RN16B, RN16C, RN16D

Commit message: new firmware for bga version of stm, change stm from smt to bga, smaller HV dividers, added 3rd can transciver, and other
Parts:
- removed C15: 100nF, Capacitor_SMD:C_0603_1608Metric, symbol Device:C_Small
- removed F1: 0ZCH0050FF2G, Fuse:Fuse_1210_3225Metric, symbol Device:Polyfuse_Small
- removed IC9: TPL7407LADR, Package_SO:SOIC-16_3.9x9.9mm_P1.27mm, symbol Samacsys_kicad_sym:TPL7407LADR
- added D15: 100V/3A, Diode_SMD:D_SMA, symbol Device:D_Small_Filled
- added F1: 5V/0.5A, Fuse:Fuse_0805_2012Metric, symbol Device:Fuse_Small
- IC8: value 3.3V/0.6A -> 3.3V/0.5A; footprint Package_TO_SOT_SMD:SOT-89-3 -> Package_TO_SOT_SMD:SOT-23-5; Manufacturer_Name Diodes Inc. -> Texas Instruments; Manufacturer_Part_Number AP7365-33YRG-13 -> TPS7B92033DBVR; Mouser Part Number 621-AP7365-33YRG-13 -> 595-TPS7B92033DBVR; Mouser Price/Stock https://www.mouser.co.uk/ProductDetail/Diodes-Incorporated/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 -> https://www.mouser.pl/ProductDetail/Texas-Instruments/TPS7B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
- R22: value 200R -> 200
Connections:
- net +3.3VISO: now also IC8.5 (VO); no longer IC8.3 (VO)
- net +5VISO: now also IC8.1 (VI), F1.1; no longer IC8.2 (VI)
- net GNDISO: now also IC8.2 (GND); no longer IC8.1 (GND)
- net I_VDDISO: now also F1.2
- net TSMS: now also D15.2 (A); no longer J1.4 (Pin_4), J1.5 (Pin_5), J1.6 (Pin_6)
- net UART_RX: now reaches J4.13 (Pin_13)
- net UART_TX: now reaches J4.14 (Pin_14)
- net Isolated ADC/ACU_V renamed Isolated ADC/ACU_V+
- net Isolated ADC/CAR_V renamed Isolated ADC/CAR_V+
- new net: IC8.3 (NC), IC8.4 (NC)
- new net TSMS_AIRS: D15.1 (K), J1.4 (Pin_4), J1.5 (Pin_5), J1.6 (Pin_6)
- no-connect marks 18 -> 16
Other:
- added sheet Fan Control (FanControl.kicad_sch)
- sheet Connectivity ports: added CANFD1_RX, CANFD1_TX, CANFD2_RX, CANFD2_TX, D+_I, D+_O, D-_I, D-_O; removed D+, D-, MCU_CANFD1_RX, MCU_CANFD1_TX, MCU_CANFD2_RX, MCU_CANFD2_TX, MCU_D+, MCU_D-
- sheet Isolated ADC ports: added ACU_V+, ACU_V-, CAR_V+, CAR_V-; removed ACU_V, CAR_V
- sheet MCU ports: added CANFD1_RX, CANFD1_TX, CANFD2_RX, CANFD2_TX, D+, D-, FAN1_CTRL, FAN2_CTRL, FAN3_CTRL, FAN4_CTRL, FAN5_CTRL, FAN6_CTRL, FAN7_CTRL, UART_RX, UART_TX; removed FAN_1_CTRL, FAN_2_CTRL, FAN_3_CTRL, FAN_4_CTRL, FAN_5_CTRL, FAN_6_CTRL, FAN_7_CTRL, MCU_CANFD1_RX, MCU_CANFD1_TX, MCU_CANFD2_RX, MCU_CANFD2_TX, MCU_D+, MCU_D-
- sheet Safety: file Safeties.kicad_sch -> Safety.kicad_sch
- note added: "13:PGR_TX 14:PRG_RX"
- moved on the sheet: J3

Commit message: mcu pinout done
Parts:
- added F6, F7: 5V/0.5A, Fuse:Fuse_0805_2012Metric, symbol Device:Fuse_Small
- added TP1: TestPoint_Small, Connector_Pin:Pin_D0.7mm_L6.5mm_W1.8mm_FlatFork, symbol Connector:TestPoint_Small
Connections:
- net +3.3VISO: now also F6.1; no longer C48.1, IC8.5 (VO)
- net +5VISO: now also F7.1; no longer C40.1, C47.2, IC8.1 (VI), R22.2, U4.13 (SEL), U4.14 (VISO)
- net AIR_P_DETECTION: now also J12.14 (Pin_14); no longer J12.28 (Pin_28)
- net CANFD1+: now also J12.27 (Pin_27); no longer J12.25 (Pin_25)
- net CANFD1-: now also J12.26 (Pin_26); no longer J12.24 (Pin_24)
- net CANFD2+: now also J12.25 (Pin_25); no longer J12.8 (Pin_8)
- net CANFD2-: now also J12.24 (Pin_24); no longer J12.7 (Pin_7)
- net EXT_NRST: now also J12.28 (Pin_28); no longer J12.11 (Pin_11)
- net GND: no longer J12.14 (Pin_14), J12.21 (Pin_21), J12.22 (Pin_22), J12.23 (Pin_23), J12.26 (Pin_26), J12.27 (Pin_27), J12.34 (Pin_34), J12.6 (Pin_6), J12.9 (Pin_9)
- net GNDISO: now also TP1.1
- net SAFETY1: now also J12.5 (Pin_5); no longer J12.4 (Pin_4)
- net SAFETY2: now also J12.6 (Pin_6); no longer J12.5 (Pin_5)
- net ~{EXT_CS_V}_C: no longer names the net of J12.15 (Pin_15)
- new net CANFD3+: J12.23 (Pin_23)
- new net CANFD3-: J12.22 (Pin_22)
- new net F_+3VISO: C48.1, F6.2, IC8.5 (VO)
- new net F_+5VISO: C40.1, C47.2, F7.2, IC8.1 (VI), R22.2, U4.13 (SEL), U4.14 (VISO)
- new net ~{EXT_CS}: J12.34 (Pin_34)
- no-connect marks 16 -> 23
Other:
- sheet Connectivity ports: added CANFD3+, CANFD3-, CANFD3_RX, CANFD3_TX; removed none
- sheet MCU ports: added CANFD3_RX, CANFD3_TX, DETECT_WTDG, SIGNAL_AMS_ERROR; removed SIGNAL_AMS_FAULT
- sheet Safety ports: added AMS_ERROR, WTDG_ERROR; removed MCU_AMS_FAULT
- moved on the sheet: C48, D15, F1

Commit message: mama comit
Parts:
- removed D15: 100V/3A, Diode_SMD:D_SMA, symbol Device:D_Small_Filled
- added D15: 0.5V/1A, symbol Device:D_Small
- added D17, D18, D19, D20: 1.7V/1kV, Diode_SMD:D_SMA, symbol Device:D_Small
- added F10, F11, F12, F13, F14, F15, F9: ?A/600V, symbol Device:Fuse_Small
Connections:
- net GNDISO: no longer J10.3 (Pin_3), J7.3 (Pin_3)
- net Isolated ADC/ACU_V+: now also D17.1 (K); no longer J7.1 (Pin_1)
- net Isolated ADC/CAR_V+: now also D19.1 (K); no longer J10.1 (Pin_1)
- net Isolated SPI/OUT+: now also F13.2; no longer J5.2 (Pin_2)
- net Isolated SPI/OUT-: now also F14.2; no longer J5.1 (Pin_1)
- net SHIELD: now also F15.2; no longer C36.2
- net TSMS: now also D15.2 (A)
- net TSMS_AIRS: now also D15.1 (K)
- net VBUS+: now reaches J2.A4 (VBUS), J2.A9 (VBUS), J2.B4 (VBUS), J2.B9 (VBUS)
- net BOOT0: no longer names the net of J12.29 (Pin_29)
- net EXT_NRST: no longer names the net of J12.28 (Pin_28)
- new net: F14.1, J5.1 (Pin_1)
- new net: F13.1, J5.2 (Pin_2)
- new net: D19.2 (A), F10.2
- new net: D20.1 (K), F12.2
- new net: F12.1, J10.3 (Pin_3)
- new net: C36.2, F15.1
- new net: F9.1, J7.1 (Pin_1)
- new net: D17.2 (A), F9.2
- new net: D18.1 (K), F11.2
- new net: F11.1, J7.3 (Pin_3)
- new net: F10.1, J10.1 (Pin_1)
- new net Isolated ADC/ACU_V-: D18.2 (A)
- new net Isolated ADC/CAR_V-: D20.2 (A)
- no-connect marks 23 -> 22
Other:
- sheet Connectivity ports: added none; removed BOOT0_I, BOOT0_O, NRST_I, NRST_O
- sheet MCU ports: added none; removed BOOT0
- moved on the sheet: C36, J10, J5, J7, J8
