File: hardware/PUTM_EV_BMS_HV_MASTER_2023.kicad_pcb (KiCad board)
At the start: 4 copper layers, 60 x 150 mm, 253 parts, among them IC1 RTQ2965GSP-QA, IC10 REF193GSZ-REEL, IC11 MCP3561T-E_NC, IC12 SN74LVC1G07DBVR, IC13 UCC12040DVE, IC14 ISO6763FDWR, IC15 AP7365-33YRG-13, IC16 REF193GSZ-REEL, IC17 MCP3561T-E_NC, IC2 MAX17643ATC+, IC3 MCP3562T-E_NC, IC4 MCP1501-10E_SN, IC5 REF193GSZ-REEL, IC6 SN74LVC1G07DBVR, IC7 UCC12040DVE, IC8 ISO6763FDWR, IC9 AP7365-33YRG-13, J1 M300-MV30645M1, J2 M80-5103422, J3 M80-5100442, J4 FTSH-107-01-L-DV-K-A, J5 M80-5101422, J6 USB4145-03-0070-C, J7 M80-5100622, J8 M300-MV10345M1, J9 M300-MV10345M1, K1 6-1419128-4, Q1 2N7002, Q10 2SK3065, Q11 2SK3065, Q12 2SK3065, Q13 STN4NF06L, Q2 2N7002, Q3 2N7002, Q4 STN4NF06L, Q5 STN4NF06L, Q6 2SK3065, Q7 2SK3065, Q8 2SK3065, Q9 2SK3065, T1 HM1193NL, U1 STM32G484RETx, U10 LTC6820IMS, U2 74LVC1G86, U3 74AUP1G32, U4 LM1117-3.3, U5 USBLC6-2SC6, U6 MCP2542FD-E/MF, U7 USBLC6-2SC6, U8 MCP2542FD-E/MF, U9 LTC6820IMS, Y1 X322516MLB4SI, Y2 Q13FC1350000400

Commit message: new hardware
Parts:
- IC13, IC7: footprint Samacsys:SOIC127P1030X265-16N -> Package_SO:SOIC-16W_7.5x10.3mm_P1.27mm
- IC14, IC8: footprint ISO6763FDWR:SOIC127P1030X265-16N -> Package_SO:SOIC-16W_7.5x10.3mm_P1.27mm
- moved RD1 11.1 mm to (142.8, 45.5), turned to 0 degrees
- moved RD2 10.4 mm to (120.2, 45.2), turned to 0 degrees
- moved J8 3.00 mm to (148.6, 37.0)
- moved J9 3.00 mm to (125.3, 37.0)
Connections:
- J8 pad 1: /Measurements/Isolated acu measurement/HV_GND -> Net-(J8-Pad1)
- J8 pad 3: Net-(J8-Pad3) -> /Measurements/Isolated acu measurement/HV_GND
- J9 pad 1: /Measurements/Isolated car measurement/HV_GND -> Net-(J9-Pad1)
- J9 pad 3: Net-(J9-Pad3) -> /Measurements/Isolated car measurement/HV_GND
- RD1 pad 1: Net-(J8-Pad3) -> Net-(J8-Pad1)
- RD2 pad 1: Net-(J9-Pad3) -> Net-(J9-Pad1)
Routing:
- net /Measurements/Isolated acu measurement/HV_GND: track 80.8 -> 49.8 mm
- net /Measurements/Isolated car measurement/HV_GND: track 68.5 -> 48.4 mm
- net /Measurements/Isolated car measurement/HV_MES+: track 17.7 -> 28.8 mm
- net Net-(J9-Pad1): track 0.00 -> 9.36 mm
- net Net-(J8-Pad1): track 0.00 -> 9.36 mm
- net Net-(J8-Pad3): track 9.15 -> 0.00 mm
- net Net-(J9-Pad3): track 9.02 -> 0.00 mm
- net /Measurements/Isolated acu measurement/HV_MES+: track 17.1 -> 20.8 mm
- removed copper zone on F.Cu, net /Measurements/Isolated acu measurement/HV_MES+
- removed copper zone on F.Cu, net /Measurements/Isolated car measurement/HV_MES+
Other:
- board text added: "4mm"

Commit message: fixed some footprints; shorted pcb board to 60x100; re-designed the HV & current measuring as well as LTC communication, all are in one TS section;
Parts:
- removed C59: 4.7uF, Capacitor_SMD:C_0603_1608Metric
- removed C60, C61, C63, C64, C67, C68: 100nF, Capacitor_SMD:C_0603_1608Metric
- removed C62, C65, C66: 10uF, Capacitor_SMD:C_0603_1608Metric
- removed D11, D16: SMBJ26CA-13-F, Diode_SMD:D_SMB
- removed D12, D13: TSZU52C13, Diode_SMD:D_0603_1608Metric
- removed D15: VSSB410S-E3/52T, Diode_SMD:D_SMB
- removed D5, D6: CDBU0530, Diode_SMD:D_0603_1608Metric
- removed FB1, FB2, FB5, FB6, FB7: GZ1608D601TF, Inductor_SMD:L_0603_1608Metric
- removed FL1: DLW21SN501SK2L, Samacsys:DLW21SN121HQ2L
- removed IC12: SN74LVC1G07DBVR, Package_TO_SOT_SMD:SOT-23-5
- removed IC13: UCC12040DVE, Package_SO:SOIC-16W_7.5x10.3mm_P1.27mm
- removed IC14: ISO6763FDWR, Package_SO:SOIC-16W_7.5x10.3mm_P1.27mm
- removed IC15, IC9: AP7365-33YRG-13, AP7365-33YRG-13:AP736533YRG13
- removed IC16, IC5: REF193GSZ-REEL, MCP1501-10E_SN:SOIC127P600X175-8N
- removed IC17: MCP3561T-E_NC, MCP3561T-E_NC:QFN40P300X300X60-21N-D
- removed IC3: MCP3562T-E_NC, MCP3561T-E_NC:QFN40P300X300X60-21N-D
- removed IC4: MCP1501-10E_SN, MCP1501-10E_SN:SOIC127P600X175-8N
- removed J1: M300-MV30645M1, M300-MV30645M1:M300MV30645M1
- removed J2: M80-5103422, Samacsys:M80-51034YY
- removed J3: M80-5100442, Samacsys:M80-51004YY
- removed J4: FTSH-107-01-L-DV-K-A, ftsh-107-01-l-dv-k-a:FTSH-107-XX-YYY-DV-K-A
- removed J5: M80-5101422, Samacsys:M80-51014YY
- removed J6: USB4145-03-0070-C, Samacsys:USB4145030070C
- removed J8, J9: M300-MV10345M1, M300-MV10345M1:M300MV10345M1
- removed K1: 6-1419128-4, 6-1419128-4:614191284
- removed L10: 4.7uH, Inductor_SMD:L_1206_3216Metric
- removed L11, L12, L5, L9: 1mH, Inductor_SMD:L_1206_3216Metric
- removed O1, O2, O3, O4: FOD8802DR2_IMG, Opto 2 ch:SOIC127P600X175-8N
- removed R26: 147k, Resistor_SMD:R_0603_1608Metric
- removed R27: 10.5k, Resistor_SMD:R_0603_1608Metric
- removed R30: 105k, Resistor_SMD:R_0603_1608Metric
- removed R31: 23.2k, Resistor_SMD:R_0603_1608Metric
- removed R34, R35, R62, R63, R70, R71: 2.7k, Resistor_SMD:R_0603_1608Metric
- removed R36, R37, R42, R43, R64, R65, R72, R73: 10k, Resistor_SMD:R_0603_1608Metric
- removed R40, R41: 120R, Resistor_SMD:R_0603_1608Metric
- removed R44, R45, R46, R47: 1k, Resistor_SMD:R_0603_1608Metric
- removed R68, R69: 200R, Resistor_SMD:R_0603_1608Metric
- removed RD1, RD2: CDMM20M0F2500, CDMM:CDMM
- removed RN1: 33R, Resistor_SMD:R_Array_Convex_8x0602
- removed T1: HM1193NL, Transformer_SMD:Transformer_Pulse_H1100NL
- removed U4: LM1117-3.3, Package_TO_SOT_SMD:SOT-223-3_TabPin2
- added F5: 16V/0.5A, Fuse:Fuse_1210_3225Metric, F.Cu at (178.6, 26.1)
- added J10: M300-MV10345M1, Samacsys:M300MV10345M1, F.Cu at (219.0, 56.5)
- added RN2: 2k, Resistor_SMD:R_Array_Convex_4x0603, F.Cu at (148.5, 107.7)
- added RN3: 500, Resistor_SMD:R_Array_Convex_4x0603, F.Cu at (152.6, 107.7)
- added RN4: 4x10k, Resistor_SMD:R_Array_Convex_4x0603, F.Cu at (156.8, 107.7)
- added RN5: 500, Resistor_SMD:R_Array_Convex_4x0603, F.Cu at (160.9, 107.7)
- added RN6: 2k, Resistor_SMD:R_Array_Convex_4x0603, F.Cu at (165.1, 107.7)
- added RN7: 4x10k, Resistor_SMD:R_Array_Convex_4x0603, F.Cu at (169.2, 107.7)
- added U11: LTC6820IMS, Package_SO:MSOP-16_3x4.039mm_P0.5mm, F.Cu at (156.5, 61.3)
- added U12: LMR33640DDDA, Package_SO:Texas_HSOP-8-1EP_3.9x4.9mm_P1.27mm, F.Cu at (190.3, 16.1)
- C10, C9: value 10uF/60V -> 100nF; footprint Capacitor_SMD:C_1210_3225Metric -> Capacitor_SMD:C_0603_1608Metric; moved to F.Cu
- C11: value 10pF -> 22uF; footprint Capacitor_SMD:C_0603_1608Metric -> Capacitor_SMD:C_0805_2012Metric; moved to F.Cu
- C12: value 12nF -> 22uF; footprint Capacitor_SMD:C_0603_1608Metric -> Capacitor_SMD:C_0805_2012Metric; moved to F.Cu
- C13, C14: moved to F.Cu
- C16, C27: value 100nF -> 22uF; footprint Capacitor_SMD:C_0603_1608Metric -> Capacitor_SMD:C_0805_2012Metric; moved to F.Cu
- C17, C26: value 100nF/60V -> 22uF; footprint Capacitor_SMD:C_0603_1608Metric -> Capacitor_SMD:C_0805_2012Metric; moved to F.Cu
- C18: value 100uF/12V -> 100nF/1kV; footprint Capacitor_SMD:CP_Elec_5x4.5 -> Capacitor_SMD:C_1812_4532Metric
- C19: value 47uF/12V -> 22uF; footprint Capacitor_SMD:CP_Elec_5x4.5 -> Capacitor_SMD:C_0805_2012Metric; moved to F.Cu
- C20: value 2.2uF/60V -> 22uF; footprint Capacitor_SMD:C_1210_3225Metric -> Capacitor_SMD:C_0805_2012Metric; moved to F.Cu
- C21: value 5.6nF -> 100nF; moved to F.Cu
- C22: value 2.2uF -> 100nF; moved to F.Cu
- C23, C44, C54, C55: value 10uF -> 22uF; footprint Capacitor_SMD:C_0603_1608Metric -> Capacitor_SMD:C_0805_2012Metric
- C30: value 47uF -> 100nF; moved to F.Cu
- C31: value 47uF -> 10nF; moved to F.Cu
- C34: value 22nF -> 100nF
- C35: value 22nF -> 4.7uF
- C36: value 5.6nF/2000V -> 100nF; footprint Samacsys:C2824 -> Capacitor_SMD:C_0603_1608Metric
- C40, C49, C52: value 100nF -> 22uF; footprint Capacitor_SMD:C_0603_1608Metric -> Capacitor_SMD:C_0805_2012Metric
- C41, C51: value 10uF -> 100nF
- C48: value 4.7uF -> 100nF
- C53: value 100nF -> 5.6nF/2000V; footprint Capacitor_SMD:C_0603_1608Metric -> Capacitor_SMD:C_3640_9110Metric
- C58: value 100nF -> 100nF/1kV; footprint Capacitor_SMD:C_0603_1608Metric -> Capacitor_SMD:C_1812_4532Metric
- D10, D24, D9: footprint Diode_SMD:D_SMB -> Diode_SMD:D_SOD-123
- D14: footprint Diode_SMD:D_SOD-128 -> Diode_SMD:D_SOD-123
- D17, D18, D19, D20, D21, D22, D23: footprint Diode_SMD:D_0603_1608Metric -> Diode_SMD:D_SOD-123
- D4: value SP0505BAHT -> ESDA5V3SC5
- D7: footprint Diode_SMD:D_SMA -> Diode_SMD:D_SOD-123
- F2: value 576-2920L500/24SLDR -> 5A/24V; footprint Samacsys:2920L700SLPR -> Fuse:Fuse_2920_7451Metric; moved to F.Cu
- F3: value 0ZCH0050FF2G -> 16V/0.5A
- F4: value 0ZCH0050FF2G -> 16V/0.5A; moved to F.Cu
- H3: footprint MountingHole:MountingHole_3.2mm_M3_Pad_Via -> MountingHole:MountingHole_3.2mm_M3
- IC1: value RTQ2965GSP-QA -> 3.3V/0.6A; footprint RTQ2965GSP-QA:SOIC127P600X175-9N -> Package_TO_SOT_SMD:SOT-89-3; moved to F.Cu
- IC10: value REF193GSZ-REEL -> MCP3564T-E; footprint MCP1501-10E_SN:SOIC127P600X175-8N -> Package_DFN_QFN:UQFN-20-1EP_3x3mm_P0.4mm_EP1.85x1.85mm
- IC11: value MCP3561T-E_NC -> ISO6760; footprint MCP3561T-E_NC:QFN40P300X300X60-21N-D -> Package_SO:SOIC-16W_7.5x10.3mm_P1.27mm
- IC2: value MAX17643ATC+ -> TPS54202HDDCR; footprint MAX17643ATC+:SON50P300X300X80-13N -> Package_TO_SOT_SMD:SOT-23-6; moved to F.Cu
- IC6: value SN74LVC1G07DBVR -> UCC12040DVE; footprint Package_TO_SOT_SMD:SOT-23-5 -> Package_SO:SOIC-16W_7.5x10.3mm_P1.27mm
- IC7: value UCC12040DVE -> ISO6760
- IC8: value ISO6763FDWR -> 3.3V/0.6A; footprint Package_SO:SOIC-16W_7.5x10.3mm_P1.27mm -> Package_TO_SOT_SMD:SOT-89-3
- J7: value M80-5100622 -> M300-MV10345M1; footprint Samacsys:M80-51006YY -> Samacsys:M300MV10345M1
- L2: value 33uH -> 6.8uF; footprint Inductor_SMD:L_Bourns_SRP1038C_10.0x10.0mm -> Inductor_SMD:L_TDK_VLS6045EX_VLS6045AF; moved to F.Cu
- L4: value 10uH -> 68uF; footprint Inductor_SMD:L_Coilcraft_XAL5050-XXX -> Inductor_SMD:L_TDK_VLS6045EX_VLS6045AF; moved to F.Cu
- L6, L8: value 1mH -> 4.7uH
- Q13, Q4, Q5: value STN4NF06L -> 2SK3065; footprint Package_TO_SOT_SMD:SOT-223-3_TabPin2 -> Package_TO_SOT_SMD:SOT-89-3
- R20, R21: value 2.7k -> 1k
- R22: value 10k -> 200R
- R23: value 10k -> 510k
- R24: value 20.5k -> 9k; moved to F.Cu
- R25: value 392k -> 100k; moved to F.Cu
- R28: value 40.2k -> 100k; moved to F.Cu
- R29: value 4.7R -> 13.3k; moved to F.Cu
- R4: value 10k -> 1k
- U10, U9: value LTC6820IMS -> TLP293-4; footprint Package_SO:MSOP-16_3x4.039mm_P0.5mm -> Package_SO:SOIC-16_4.55x10.3mm_P1.27mm
- moved J7 169.6 mm to (271.0, 56.5), turned to 90 degrees
- moved C45 131.3 mm to (152.8, 47.2)
- moved C43 127.2 mm to (152.8, 42.2), turned to 0 degrees
- moved C46 124.8 mm to (152.8, 49.7), turned to 0 degrees
- moved H3 123.0 mm to (142.8, 60.8)
- moved C44 122.7 mm to (152.8, 44.7), turned to 0 degrees
- moved C18 118.6 mm to (203.3, 60.4), turned to 0 degrees
- moved F3 118.2 mm to (195.7, 58.1)
- moved FB3 117.3 mm to (156.8, 52.2), turned to 0 degrees
- moved C41 116.1 mm to (148.8, 54.8), turned to 0 degrees
- moved C16 115.3 mm to (140.0, 23.7), turned to 0 degrees
- moved C36 115.3 mm to (148.8, 47.2), turned to 0 degrees
- moved C34 114.1 mm to (148.8, 42.2)
- moved F1 113.3 mm to (155.3, 66.2), turned to 0 degrees
- moved C42 113.0 mm to (148.8, 57.3)
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Connections:
- net /CLK_IN renamed /MCU/CLK_IN
- net /CLK_OUT renamed /MCU/CLK_OUT
- net /MCU_LED_1 renamed /MCU/SIGNAL_LED_1
- net /MCU_LED_2 renamed /MCU/SIGNAL_LED_2
- net /MCU_LED_3 renamed /MCU/SIGNAL_LED_3
- net /RTC_CLK_IN renamed /MCU/RTC_CLK_IN
- net /RTC_CLK_OUT renamed /MCU/RTC_CLK_OUT
- net /Safeties and related/AMS_FAULT renamed /Safety/AMS_FAULT
- net /Safeties and related/AMS_FAULT_INTER renamed /Safety/AMS_OK
- net /Safeties and related/CAP_VOLT renamed /Safety/CAP_VOLT
- net /Safeties and related/EDGE_DETECT renamed /Safety/EDGE_DETECT
- net /Safeties and related/IN_DELAY renamed /Safety/IN_DELAY
- net /Safeties and related/RELAY- renamed /Safety/RELAY-
- net AIR_M- renamed /AIR Control/DRAIN1
- net AIR_P- renamed /AIR Control/DRAIN3
- net AIR_PRE- renamed /AIR Control/DRAIN2
- net FAN1- renamed /FAN1-
- net FAN2- renamed /FAN2-
- net FAN3- renamed /FAN3-
- net FAN4- renamed /FAN4-
- net FAN5- renamed /FAN5-
- net FAN6- renamed /FAN6-
- net FAN7- renamed /FAN7-
- net SAFETY_TSMS_IN renamed TSMS
- C10 pad 1: /Power/12V_VIN -> Net-(U12-BOOT)
- C10 pad 2: GND -> /Power/SW_5V
- C11 pad 1: Net-(IC1-COMP) -> +5V
- C12 pad 1: Net-(C12-Pad1) -> GND
- C12 pad 2: GND -> Net-(IC2-VIN)
- C13 pad 1: +5V -> Net-(IC1-VI)
- C16 pad 1: +3V3 -> 12V
- C17 pad 1: Net-(IC1-BOOT) -> GND
- C17 pad 2: /Power/12V_SW -> Net-(IC2-VIN)
- C18 pad 1: Net-(C15-Pad1) -> unconnected-(C18-Pad1)
- C18 pad 2: GND -> unconnected-(C18-Pad2)
- C19 pad 1: +12V -> 12V
- C20 pad 1: /Power/5V_SW -> 12V
- C21 pad 1: Net-(IC2-SS) -> GND
- C21 pad 2: GND -> Net-(IC2-VIN)
- C22 pad 1: Net-(IC2-VCC) -> Net-(IC2-BOOT)
- C22 pad 2: GND -> /Power/SW_5V
- C23 pad 1: +3.3VA -> Net-(U1B-VDDA)
- C26 pad 1: Net-(IC2-BST) -> +5V
- C26 pad 2: Net-(IC2-LX) -> GND
- C27 pad 1: Net-(IC2-EXTVCC) -> +3V3
- C30 pad 1: +5V -> +3.3VISO
- C30 pad 2: GND -> GNDISO
- C31 pad 1: +5V -> +3.3VISO
- C31 pad 2: GND -> GNDISO
- C34 pad 1: Net-(C34-Pad1) -> +3V3
- C35 pad 1: Net-(C35-Pad1) -> Net-(IC6-EN)
- C36 pad 1: GND -> +3V3
- C36 pad 2: /Communication/LTC_CHASSIS -> GND
- C39 pad 1: +3V3 -> /HV_+3.3V
- C39 pad 2: GND -> /HV_GND
- C40 pad 1: +3V3 -> +5VISO
- C40 pad 2: GND -> GNDISO
- C41 pad 1: Net-(IC3-AVDD) -> +3V3
- C46 pad 2: /Measurements/3V_REF -> /3V_REF
- C47 pad 1: +3V3 -> GNDISO
- C47 pad 2: GND -> +5VISO
- C48 pad 1: Net-(IC7-EN) -> +3.3VISO
- C48 pad 2: GND -> GNDISO
- C49 pad 1: +3V3 -> Net-(IC9-VSS)
- C49 pad 2: GND -> /HV_GND
- C50 pad 1: /Measurements/Isolated acu measurement/HV_+3.3V -> GNDISO
- C50 pad 2: /Measurements/Isolated acu measurement/HV_GND -> +3.3VISO
- C51 pad 1: /Measurements/Isolated acu measurement/HV_+5V -> /HV_GND
- C51 pad 2: /Measurements/Isolated acu measurement/HV_GND -> /3V_REF
- C52 pad 1: /Measurements/Isolated acu measurement/HV_GND -> GND
- C52 pad 2: /Measurements/Isolated acu measurement/HV_+5V -> Net-(U12-EN)
- C53 pad 1: /Measurements/Isolated acu measurement/HV_+3.3V -> GND
- C53 pad 2: /Measurements/Isolated acu measurement/HV_GND -> /LTC_CHASSIS
- C54 pad 1: Net-(IC10-VSS) -> GND
- C54 pad 2: /Measurements/Isolated acu measurement/HV_GND -> Net-(U12-EN)
- C55 pad 1: Net-(IC11-AVDD) -> 12V
- C55 pad 2: /Measurements/Isolated acu measurement/HV_GND -> GND
- C56 pad 1: /Measurements/Isolated acu measurement/HV_GND -> GND
- C56 pad 2: /Measurements/Isolated acu measurement/3V_REF -> Net-(IC1-VI)
- C57 pad 1: /Measurements/Isolated acu measurement/HV_+3.3V -> GND
- C57 pad 2: /Measurements/Isolated acu measurement/HV_GND -> +3V3
- C58 pad 1: +3V3 -> unconnected-(C58-Pad1)
- C58 pad 2: GND -> unconnected-(C58-Pad2)
- C9 pad 1: /Power/12V_VIN -> GND
- C9 pad 2: GND -> Net-(U12-VCC)
- D14 pad 1: Net-(D14-K) -> unconnected-(D14-K-Pad1)
- D4 pad 1: /Connectors/~{EXT_CS_V}_C -> unconnected-(D4-A-Pad1)
- D4 pad 2: GND -> Net-(D4-K)
- D4 pad 3: /Connectors/MOSI_C -> unconnected-(D4-A-Pad3)
- D4 pad 4: /Connectors/MISO_C -> unconnected-(D4-A-Pad4)
- D4 pad 5: /Connectors/SCK_C -> Net-(D4-K)
- D4 pad 6: /Connectors/~{EXT_CS_I}_C -> unconnected-(D4-A-Pad6)
- F2 pad 1: /Power/12V_VIN -> Net-(U12-EN)
- F4 pad 1: /Power/5V_SW -> VDD
- F4 pad 2: VDD -> Net-(IC2-VIN)
- FB4 pad 2: Net-(IC10-VSS) -> Net-(IC9-VSS)
- IC1 pad 1: Net-(IC1-BOOT) -> GND
- IC1 pad 2: /Power/12V_VIN -> Net-(IC1-VI)
- IC1 pad 3: unconnected-(IC1-EN-Pad3) -> +3V3
- IC10 pad 1: (no net) -> unconnected-(IC10-REFIN--Pad1)
- IC10 pad 2: Net-(IC10-VSS) -> unconnected-(IC10-REFIN+-Pad2)
- IC10 pad 3: Net-(IC10-VSS) -> unconnected-(IC10-CH0-Pad3)
- IC10 pad 4: /Measurements/Isolated acu measurement/HV_GND -> unconnected-(IC10-CH1-Pad4)
- IC10 pad 5: (no net) -> unconnected-(IC10-CH2-Pad5)
- IC10 pad 6: /Measurements/Isolated acu measurement/3V_REF -> unconnected-(IC10-CH3-Pad6)
- IC10 pad 7: (no net) -> unconnected-(IC10-CH4-Pad7)
- IC10 pad 8: (no net) -> unconnected-(IC10-CH5-Pad8)
- IC11 pad 1: /Measurements/Isolated acu measurement/HV_GND -> unconnected-(IC11-VCC1-Pad1)
- IC11 pad 10: (no net) -> unconnected-(IC11-OUTF-Pad10)
- IC11 pad 11: /Measurements/Isolated acu measurement/HV_~{CS} -> unconnected-(IC11-OUTE-Pad11)
- IC11 pad 12: /Measurements/Isolated acu measurement/HV_SCK -> unconnected-(IC11-OUTD-Pad12)
- IC11 pad 13: /Measurements/Isolated acu measurement/HV_SDI -> unconnected-(IC11-OUTC-Pad13)
- IC11 pad 14: /Measurements/Isolated acu measurement/HV_SDO -> unconnected-(IC11-OUTB-Pad14)
- IC11 pad 2: /Measurements/Isolated acu measurement/3V_REF -> unconnected-(IC11-INA-Pad2)
- IC11 pad 3: /Measurements/Isolated acu measurement/HV_MES+ -> unconnected-(IC11-INB-Pad3)
- IC11 pad 4: /Measurements/Isolated acu measurement/HV_GND -> unconnected-(IC11-INC-Pad4)
- IC11 pad 5: (no net) -> unconnected-(IC11-IND-Pad5)
- IC11 pad 6: (no net) -> unconnected-(IC11-INE-Pad6)
- IC11 pad 7: (no net) -> unconnected-(IC11-INF-Pad7)
- IC11 pad 8: (no net) -> unconnected-(IC11-GND1-Pad8)
- IC11 pad 9: (no net) -> unconnected-(IC11-GND2-Pad9)
- IC2 pad 1: /Power/5V_SW -> GND
- IC2 pad 2: /Power/5V_SW -> /Power/SW_5V
- IC2 pad 3: +5V -> Net-(IC2-VIN)
- IC2 pad 4: Net-(IC2-SS) -> Net-(IC2-FB)
- IC2 pad 5: Net-(IC2-VCC) -> Net-(IC2-EN)
- IC2 pad 6: Net-(IC2-RT/SYNC) -> Net-(IC2-BOOT)
- IC6 pad 1: unconnected-(IC6-Pad1) -> Net-(IC6-EN)
- IC6 pad 2: Net-(IC8-OUTD) -> GND
- IC6 pad 3: GND -> Net-(IC6-EN)
- IC6 pad 4: MISO -> GND
- IC6 pad 5: +3V3 -> unconnected-(IC6-SYNC_OK-Pad5)
- IC7 pad 1: Net-(IC7-EN) -> unconnected-(IC7-VCC1-Pad1)
- IC7 pad 10: /Measurements/Isolated acu measurement/HV_GND -> unconnected-(IC7-OUTF-Pad10)
- IC7 pad 11: /Measurements/Isolated acu measurement/HV_GND -> unconnected-(IC7-OUTE-Pad11)
- IC7 pad 12: /Measurements/Isolated acu measurement/HV_GND -> unconnected-(IC7-OUTD-Pad12)
- IC7 pad 13: /Measurements/Isolated acu measurement/HV_+5V -> unconnected-(IC7-OUTC-Pad13)
- IC7 pad 14: /Measurements/Isolated acu measurement/HV_+5V -> unconnected-(IC7-OUTB-Pad14)
- IC7 pad 15: /Measurements/Isolated acu measurement/HV_GND -> unconnected-(IC7-OUTA-Pad15)
- IC7 pad 16: /Measurements/Isolated acu measurement/HV_GND -> unconnected-(IC7-VCC2-Pad16)
- IC7 pad 2: GND -> unconnected-(IC7-INA-Pad2)
- IC7 pad 3: Net-(IC7-EN) -> unconnected-(IC7-INB-Pad3)
- IC7 pad 4: GND -> unconnected-(IC7-INC-Pad4)
- IC7 pad 6: GND -> unconnected-(IC7-INE-Pad6)
- IC7 pad 7: GND -> unconnected-(IC7-INF-Pad7)
- IC7 pad 8: GND -> unconnected-(IC7-GND1-Pad8)
- IC7 pad 9: /Measurements/Isolated acu measurement/HV_GND -> unconnected-(IC7-GND2-Pad9)
- IC8 pad 1: +3V3 -> GNDISO
- IC8 pad 2: /~{MES_ACU_CS} -> +5VISO
- IC8 pad 3: SCK -> +3.3VISO
- J7 pad 1: /Communication/LTC_1_OUT_I- -> Net-(J7-Pin_1)
- J7 pad 2: /Communication/LTC_CHASSIS -> unconnected-(J7-Pin_2-Pad2)
- J7 pad 3: /Communication/LTC_2_OUT_I+ -> GNDISO
- L1 pad 1: Net-(FB1-Pad1) -> unconnected-(L1-Pad1)
- L2 pad 1: /Power/12V_SW -> /Power/SW_5V
- L2 pad 2: +12V -> 12V
- L3 pad 1: +3.3VA -> +3V3
- L3 pad 2: +3V3 -> Net-(U1B-VDDA)
- L4 pad 1: Net-(IC2-LX) -> /Power/SW_5V
- L7 pad 2: Net-(IC7-EN) -> Net-(IC6-EN)
- L8 pad 1: /Measurements/Isolated acu measurement/HV_+5V -> /HV_+5V
- R16 pad 2: /SIGNAL_AIR_M -> /AIR Control/SIGNAL1
- R18 pad 2: /SIGNAL_AIR_PRE -> /AIR Control/SIGNAL2
- R20 pad 1: Net-(O1-Pad1) -> Net-(U11-ICMP)
- R20 pad 2: EXT_RESET -> Net-(U11-IBIAS)
- R21 pad 1: Net-(O1-Pad3) -> GND
- R21 pad 2: AIR_P_DETECTION -> Net-(U11-ICMP)
- R22 pad 1: NRST -> GNDISO
- R22 pad 2: +3V3 -> +5VISO
- R23 pad 1: /AIR_P_DETECT -> Net-(IC2-EN)
- R23 pad 2: +3V3 -> Net-(IC2-VIN)
- R24 pad 1: Net-(C12-Pad1) -> GND
- R24 pad 2: Net-(IC1-COMP) -> Net-(U12-FB)
- R25 pad 1: GND -> Net-(U12-FB)
- R25 pad 2: Net-(IC1-RT/SYNC) -> 12V
- R28 pad 1: GND -> Net-(IC2-FB)
- R28 pad 2: Net-(IC2-RT/SYNC) -> +5V
- R29 pad 1: Net-(IC2-EXTVCC) -> GND
- R29 pad 2: +5V -> Net-(IC2-FB)
- R4 pad 1: NRST -> /MCU/NRST
- R48 pad 2: /FAN_1_CTRL -> /Fan drivers/FAN1_CTRL
- R49 pad 2: /FAN_5_CTRL -> /Fan drivers/FAN5_CTRL
- R5 pad 1: MISO -> /MCU/MES_MISO
- R52 pad 2: /FAN_2_CTRL -> /Fan drivers/FAN2_CTRL
- R53 pad 2: /FAN_6_CTRL -> /Fan drivers/FAN6_CTRL
- R56 pad 2: /FAN_3_CTRL -> /Fan drivers/FAN3_CTRL
- R57 pad 2: /FAN_7_CTRL -> /Fan drivers/FAN7_CTRL
- R6 pad 1: /LTC_MISO -> /MCU/LTC_MISO
- R60 pad 2: /FAN_4_CTRL -> /Fan drivers/FAN4_CTRL
- R66 pad 2: /SIGNAL_AIR_P -> /AIR Control/SIGNAL3
- U1 pad 1: +BATT -> unconnected-(U1B-VBAT-Pad1)
- U1 pad 10: /FAN_5_CTRL -> /MCU/FAN_5_CTRL
- U1 pad 11: /FAN_4_CTRL -> /MCU/FAN_4_CTRL
- U1 pad 12: /FAN_3_CTRL -> /MCU/FAN_3_CTRL
- U1 pad 13: /FAN_2_CTRL -> /MCU/FAN_2_CTRL
- U1 pad 14: /FAN_1_CTRL -> /MCU/FAN_1_CTRL
- U1 pad 17: /AIR_PRE_DETECT -> /MCU/DETECT_AIR_PRE
- U1 pad 18: /CARD_DETECT -> unconnected-(U1A-PA4-Pad18)
- U1 pad 19: /CARD_SCK -> unconnected-(U1A-PA5-Pad19)
- U1 pad 2: /SAFETY_DETECT -> /MCU/DETECT_TSMS
- U1 pad 20: /CARD_MISO -> unconnected-(U1A-PA6-Pad20)
- U1 pad 21: /CARD_MOSI -> unconnected-(U1A-PA7-Pad21)
- U1 pad 22: /~{CARD_CS} -> unconnected-(U1A-PC4-Pad22)
- U1 pad 26: /AIR_M_DETECT -> /MCU/DETECT_AIR_M
- U1 pad 28: +3.3VA -> Net-(U1B-VDDA)
- U1 pad 29: +3.3VA -> Net-(U1B-VDDA)
- U1 pad 30: /AIR_P_DETECT -> /MCU/DETECT_AIR_P
- U1 pad 33: /LTC_2_~{CS} -> /MCU/LTC_2_~{CS}
- U1 pad 34: /LTC_1_~{CS} -> /MCU/LTC_1_~{CS}
- U1 pad 35: /LTC_SCK -> /MCU/LTC_SCK
- U1 pad 36: /LTC_MISO -> /MCU/LTC_MISO
- U1 pad 37: /LTC_MOSI -> /MCU/LTC_MOSI
- U1 pad 38: /IMD_SENS_PWM -> /MCU/SENS_IMD
- U1 pad 39: /SIGNAL_AIR_PRE -> /MCU/SIGNAL_AIR_PRE
- U1 pad 40: /SIGNAL_AIR_P -> /MCU/SIGNAL_AIR_P
- U1 pad 41: /SIGNAL_AIR_M -> /MCU/SIGNAL_AIR_M
- U1 pad 42: /~{SENS_CS} -> /MCU/~{MES_I_SENS_CS}
- U1 pad 43: ~{EXT_CS_V} -> /MCU/~{MES_EXT_V_CS}
- U1 pad 44: ~{EXT_CS_I} -> /MCU/~{MES_EXT_I_CS}
- U1 pad 45: /MCU_D- -> /MCU/MCU_D-
- U1 pad 46: /MCU_D+ -> /MCU/MCU_D+
- U1 pad 49: SWDIO -> /MCU/SWDIO
- U1 pad 50: SWCLK -> /MCU/SWCLK
- U1 pad 51: /AMS_FAULT_MCU -> /MCU/SIGNAL_AMS_FAULT
- U1 pad 52: SCK -> /MCU/MES_SCK
- U1 pad 53: MISO -> /MCU/MES_MISO
- U1 pad 54: MOSI -> /MCU/MES_MOSI
- U1 pad 55: /~{MES_CAR_CS} -> /MCU/~{MES_V_CAR_CS}
- U1 pad 56: /MCU_CANFD2_RX -> /MCU/MCU_CANFD2_RX
- U1 pad 57: /MCU_CANFD2_TX -> /MCU/MCU_CANFD2_TX
- U1 pad 58: /MCU_CANFD1_RX -> /MCU/MCU_CANFD1_RX
- U1 pad 59: /MCU_CANFD1_TX -> /MCU/MCU_CANFD1_TX
- U1 pad 60: /~{MES_ACU_CS} -> /MCU/~{MES_V_ACU_CS}
- U1 pad 61: /BOOT -> /MCU/BOOT
- U1 pad 62: /CHARGER_DETECT -> /MCU/DETECT_CHARGER
- U1 pad 7: NRST -> /MCU/NRST
- U1 pad 8: /FAN_7_CTRL -> /MCU/FAN_7_CTRL
- U1 pad 9: /FAN_6_CTRL -> /MCU/FAN_6_CTRL
- U10 pad 1: +3V3 -> +3.3V
- U10 pad 10: /Communication/LTC_2_I- -> /Opto Isolation/OPT_OUT7
- U10 pad 11: /Communication/LTC_2_I+ -> GND
- U10 pad 12: +3V3 -> /Opto Isolation/OPT_OUT6
- U10 pad 14: GND -> /Opto Isolation/OPT_OUT5
- U10 pad 15: Net-(U10-ICMP) -> GND
- U10 pad 16: Net-(U10-IBIAS) -> /Opto Isolation/OPT_OUT4
- U10 pad 2: /LTC_MOSI -> Net-(RN6A-R1.1)
- U10 pad 3: /LTC_MISO -> +3.3V
- U10 pad 4: /LTC_SCK -> Net-(RN6B-R2.1)
- U10 pad 5: /LTC_2_~{CS} -> +3.3V
- U10 pad 6: +3V3 -> Net-(RN6C-R3.1)
- U10 pad 7: +3V3 -> +3.3V
- U10 pad 8: +3V3 -> Net-(RN6D-R4.1)
- U10 pad 9: +3V3 -> GND
- U9 pad 1: +3V3 -> +3.3V
- U9 pad 10: /Communication/LTC_1_I- -> /Opto Isolation/OPT_OUT3
- U9 pad 11: /Communication/LTC_1_I+ -> GND
- U9 pad 12: +3V3 -> /Opto Isolation/OPT_OUT2
- U9 pad 14: GND -> /Opto Isolation/OPT_OUT1
- U9 pad 15: Net-(U9-ICMP) -> GND
- U9 pad 16: Net-(U9-IBIAS) -> /Opto Isolation/OPT_OUT0
- U9 pad 2: /LTC_MOSI -> Net-(RN2A-R1.1)
- U9 pad 3: /LTC_MISO -> +3.3V
- U9 pad 4: /LTC_SCK -> Net-(RN2B-R2.1)
- U9 pad 5: /LTC_1_~{CS} -> +3.3V
- U9 pad 6: +3V3 -> Net-(RN2C-R3.1)
- U9 pad 7: +3V3 -> +3.3V
- U9 pad 8: +3V3 -> Net-(RN2D-R4.1)
- U9 pad 9: +3V3 -> GND
Routing:
- net SCK: track 183.7 -> 0.00 mm, vias 5 -> 0
- net MOSI: track 183.3 -> 0.00 mm, vias 5 -> 0
- net MISO: track 174.0 -> 0.00 mm, vias 5 -> 0
- net +3V3: track 127.9 -> 0.00 mm, vias 28 -> 0
- net /~{MES_CAR_CS}: track 123.3 -> 0.00 mm, vias 2 -> 0
- net GND: track 106.0 -> 0.00 mm, vias 291 -> 0
- net /~{MES_ACU_CS}: track 96.7 -> 0.00 mm, vias 2 -> 0
- net TSMS: track 80.2 -> 0.00 mm
- net /SIGNAL_AIR_M: track 65.7 -> 0.00 mm, vias 2 -> 0
- net /FAN_7_CTRL: track 59.4 -> 0.00 mm, vias 2 -> 0
- net NRST: track 58.9 -> 0.00 mm, vias 2 -> 0
- net /SIGNAL_AIR_P: track 58.0 -> 0.00 mm, vias 2 -> 0
- net +5V: track 55.1 -> 0.00 mm, vias 9 -> 0
- net /FAN_5_CTRL: track 53.8 -> 0.00 mm, vias 2 -> 0
- net +12V: track 51.4 -> 0.00 mm
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- removed copper zone on B.Cu, net +12V
- removed copper zone on B.Cu, net +3V3
- removed copper zone on B.Cu, net +5V
- removed copper zone on F.Cu, net +5V
- removed copper zone on F.Cu, net /Communication/LTC_CHASSIS
- removed copper zone on In1.Cu, net /Communication/LTC_CHASSIS
- removed copper zone on In2.Cu, net /Communication/LTC_CHASSIS
- removed copper zone on In2.Cu, net /Measurements/Isolated acu measurement/HV_+3.3V
- removed copper zone on F.Cu, net /Measurements/Isolated acu measurement/HV_+5V
- removed copper zone on In1.Cu, net /Measurements/Isolated acu measurement/HV_GND
- removed copper zone on In2.Cu, net /Measurements/Isolated car measurement/HV_+3.3V
- removed copper zone on F.Cu, net /Measurements/Isolated car measurement/HV_+5V
- removed copper zone on In1.Cu, net /Measurements/Isolated car measurement/HV_GND
- removed copper zone on B.Cu, net /Power/12V_SW
- removed copper zone on B.Cu, net /Power/12V_VIN
- removed copper zone on B.Cu, net /Power/5V_SW
- removed copper zone on B.Cu, net GND
- removed copper zone on F.Cu, net GND
- removed copper zone on In1.Cu, net GND
- removed copper zone on In2.Cu, net GND
- removed copper zone on F.Cu, net Net-(D14-K)
- removed copper zone on B.Cu, net Net-(IC2-LX)
- removed copper zone on B.Cu, net TSMS
- removed copper zone on B.Cu, net VBUS
- removed copper zone on F.Cu, net VBUS
- removed copper zone on B.Cu, net VDD
Other:
- board size 60 x 150 mm -> 244 x 150 mm

Commit message: new beginings tbc
Parts:
- removed C42, C43, C46, C51: 100nF, Capacitor_SMD:C_0603_1608Metric
- removed C44, C49: 22uF, Capacitor_SMD:C_0805_2012Metric
- removed C45: 1nF, Capacitor_SMD:C_0603_1608Metric
- removed FB3, FB4: GZ1608D601TF, Inductor_SMD:L_0603_1608Metric
- removed IC10: MCP3564T-E, Package_DFN_QFN:UQFN-20-1EP_3x3mm_P0.4mm_EP1.85x1.85mm
- removed IC6: UCC12040DVE, Package_SO:SOIC-16W_7.5x10.3mm_P1.27mm
- removed L6, L7, L8: 4.7uH, Inductor_SMD:L_1206_3216Metric
- removed R48, R49, R52, R53, R56, R57, R60: 100R, Resistor_SMD:R_0603_1608Metric
- removed R50, R51, R54, R55, R58, R59, R61: 10k, Resistor_SMD:R_0603_1608Metric
- added C59: 22uF, Capacitor_SMD:C_0805_2012Metric, F.Cu at (286.6, 75.3)
- added IC3: OPA1679-Q1, Package_DFN_QFN:QFN-16-1EP_4x4mm_P0.65mm_EP2.7x2.7mm, F.Cu at (205.0, 86.5)
- added IC4: ADS131M04, Package_DFN_QFN:WQFN-20-1EP_3x3mm_P0.4mm_EP1.7x1.7mm, F.Cu at (115.7, 81.8)
- added IC5: LTC1799, Package_TO_SOT_SMD:SOT-23-5, F.Cu at (115.7, 86.9)
- added J11: M80-5100442, Samacsys:M80-51004YY, F.Cu at (232.0, 34.5)
- added J8: M80-5100442, Samacsys:M80-51004YY, F.Cu at (244.0, 25.0)
- added R26: 8.2k, Resistor_SMD:R_0603_1608Metric, F.Cu at (111.1, 88.0)
- added R27: 0, Resistor_SMD:R_0603_1608Metric, F.Cu at (104.2, 79.5)
- added RN1: 100, Resistor_SMD:R_Array_Convex_4x0603, F.Cu at (111.2, 74.8)
- added RN10: 10k, Resistor_SMD:R_Array_Convex_4x0603, F.Cu at (123.6, 74.8)
- added RN8: 10k, Resistor_SMD:R_Array_Convex_4x0603, F.Cu at (115.3, 74.8)
- added RN9: 100, Resistor_SMD:R_Array_Convex_4x0603, F.Cu at (119.5, 74.8)
- added U4: UCC12040DVE, Package_SO:SOIC-16W_7.5x10.3mm_P1.27mm, F.Cu at (290.9, 67.9)
- C18, C58: value 100nF/1kV -> 10nF/1kV; footprint Capacitor_SMD:C_1812_4532Metric -> Capacitor_SMD:C_1206_3216Metric
- C27: value 22uF -> 220nF; footprint Capacitor_SMD:C_0805_2012Metric -> Capacitor_SMD:C_0603_1608Metric
- C35: value 4.7uF -> 100nF
- moved H2 128.8 mm to (271.5, 48.5)
- moved C27 110.5 mm to (111.1, 80.4)
- moved C53 81.5 mm to (127.5, 57.0)
- moved H1 75.8 mm to (218.5, 48.5)
- moved C35 53.7 mm to (111.1, 82.9)
- moved C41 48.6 mm to (111.1, 85.5)
- moved IC11 7.00 mm to (245.0, 77.0)
- moved IC7 7.00 mm to (256.0, 77.0)
- moved J10 7.00 mm to (219.0, 63.5)
- moved J7 7.00 mm to (271.0, 63.5)
- moved Q13 6.69 mm to (182.0, 93.0)
- moved D9 5.54 mm to (185.5, 83.0), turned to 90 degrees
- moved D10 5.42 mm to (185.5, 88.0), turned to 90 degrees
- moved D24 5.37 mm to (185.5, 93.0), turned to 90 degrees
- moved Q5 3.37 mm to (182.0, 88.0)
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Connections:
- C18 pad 2: unconnected-(C18-Pad2) -> /OUT+
- C27 pad 1: +3V3 -> GNDISO
- C27 pad 2: GND -> Net-(IC4-CAP)
- C35 pad 1: Net-(IC6-EN) -> +3.3VISO
- C35 pad 2: GND -> GNDISO
- C41 pad 1: +3V3 -> GNDISO
- C41 pad 2: GND -> +3.3VISO
- C53 pad 1: GND -> unconnected-(C53-Pad1)
- C53 pad 2: /LTC_CHASSIS -> unconnected-(C53-Pad2)
- C58 pad 2: unconnected-(C58-Pad2) -> /OUT-
- F1 pad 2: Net-(F1-Pad2) -> unconnected-(F1-Pad2)

Commit message: changes tbc
Parts:
- removed C36, C39: 100nF, Capacitor_SMD:C_0603_1608Metric
- removed R16, R18, R66: 100R, Resistor_SMD:R_0603_1608Metric
- removed R17, R19, R67: 10k, Resistor_SMD:R_0603_1608Metric
- removed U11: LTC6820IMS, Package_SO:MSOP-16_3x4.039mm_P0.5mm
- added C42: 100nF, Capacitor_SMD:C_0603_1608Metric, F.Cu at (172.8, 128.9)
- added C43: 100nF, Capacitor_SMD:C_0603_1608Metric, F.Cu at (172.8, 131.4)
- added IC6: LTC6820IMS, Package_SO:MSOP-16_3x4.039mm_P0.5mm, F.Cu at (178.8, 130.5)
- added K2: PB134024, Samacsys:PB134024, F.Cu at (200.0, 138.5)
- added R30: 1k, Resistor_SMD:R_0603_1608Metric, F.Cu at (172.8, 141.5)
- added R31: 1k, Resistor_SMD:R_0603_1608Metric, F.Cu at (172.8, 144.0)
- added RN11: 100, Resistor_SMD:R_Array_Convex_4x0603, F.Cu at (199.4, 100.3)
- added RN12: 10k, Resistor_SMD:R_Array_Convex_4x0603, F.Cu at (203.6, 100.3)
- C34: value 100nF -> 10nF
- C53, D19, D20, D23, D24, D9, Q12, Q5, Q8, Q9, U4: moved to B.Cu
- R20, R21: value 1k -> 0
- moved H4 147.8 mm to (271.5, 141.5)
- moved C53 113.8 mm to (239.5, 77.0)
- moved H3 110.6 mm to (218.5, 141.5)
- moved R27 90.8 mm to (172.8, 139.0)
- moved R21 87.5 mm to (172.8, 136.5)
- moved R20 87.5 mm to (172.8, 133.9)
- moved Q8 81.0 mm to (230.3, 86.0)
- moved Q9 80.9 mm to (230.3, 93.0)
- moved Q7 80.6 mm to (230.3, 89.5)
- moved Q6 80.6 mm to (230.3, 82.5)
- moved Q11 69.6 mm to (225.3, 93.0)
- moved Q12 69.6 mm to (225.3, 89.5)
- moved Q10 69.5 mm to (225.3, 86.0)
- moved D23 69.4 mm to (229.8, 89.5), turned to 180 degrees
- moved D21 69.2 mm to (229.8, 86.0), turned to 180 degrees
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Connections:
- net /AMS_FAULT_MCU renamed /Safety/IN
- C18 pad 1: unconnected-(C18-Pad1) -> /I-
- C34 pad 1: +3V3 -> /CAR_I_REF
- C34 pad 2: GND -> GNDISO
- C58 pad 1: unconnected-(C58-Pad1) -> /I+
- F1 pad 1: +5V -> +5VISO
- F1 pad 2: unconnected-(F1-Pad2) -> Net-(J11-Pin_4)
- IC3 pad 1: Net-(IC3A--) -> /ACU_V_ADC
- IC3 pad 11: unconnected-(IC3D-+-Pad11) -> /CAR_I_REF
- IC3 pad 12: Net-(IC3D--) -> /CAR_I_REF_ADC
- IC3 pad 14: Net-(IC3D--) -> /CAR_I_REF_ADC
- IC3 pad 15: Net-(IC3A--) -> /ACU_V_ADC
- IC3 pad 2: unconnected-(IC3A-+-Pad2) -> /ACU_V
- IC3 pad 4: unconnected-(IC3B-+-Pad4) -> /CAR_V
- IC3 pad 5: Net-(IC3B--) -> /CAR_V_ADC
- IC3 pad 6: Net-(IC3B--) -> /CAR_V_ADC
- IC3 pad 7: Net-(IC3C--) -> /CAR_I_ADC
- IC3 pad 8: Net-(IC3C--) -> /CAR_I_ADC
- IC3 pad 9: unconnected-(IC3C-+-Pad9) -> /CAR_I
- IC4 pad 1: unconnected-(IC4-CH0+-Pad1) -> /ACU_V_ADC
- IC4 pad 3: unconnected-(IC4-CH1+-Pad3) -> /CAR_V_ADC
- IC4 pad 5: unconnected-(IC4-CH2+-Pad5) -> /CAR_I_ADC
- IC4 pad 6: unconnected-(IC4-CH2--Pad6) -> /CAR_I_REF_ADC
- J11 pad 4: GNDISO -> Net-(J11-Pin_4)
- R20 pad 1: Net-(U11-ICMP) -> /CAR_I_REF
- R20 pad 2: Net-(U11-IBIAS) -> +3.3VISO
- R21 pad 1: GND -> /CAR_I_REF
- R21 pad 2: Net-(U11-ICMP) -> GNDISO
- R27 pad 1: unconnected-(R27-Pad1) -> /CAR_I_REF
- R27 pad 2: unconnected-(R27-Pad2) -> +5VISO
- U9 pad 1: +3.3V -> Net-(RN2A-R1.1)
- U9 pad 2: Net-(RN2A-R1.1) -> GND
- U9 pad 3: +3.3V -> Net-(RN2B-R2.1)
- U9 pad 4: Net-(RN2B-R2.1) -> GND
- U9 pad 5: +3.3V -> Net-(RN2C-R3.1)
- U9 pad 6: Net-(RN2C-R3.1) -> GND
- U9 pad 7: +3.3V -> Net-(RN2D-R4.1)
- U9 pad 8: Net-(RN2D-R4.1) -> GND
Other:
- board size 244 x 150 mm -> 60 x 100 mm

Commit message: sync
Parts:
- added J3: M80-51014XX, Samacsys:M80-51014YY, F.Cu at (218.5, 92.0)
- moved C59 81.6 mm to (205.0, 76.5)
- moved K2 45.0 mm to (241.5, 121.0)
- moved U1 32.0 mm to (114.5, 60.0)
- moved D20 5.00 mm to (225.5, 98.0)
- moved D22 5.00 mm to (230.0, 98.0)
- moved Q11 5.00 mm to (225.5, 98.0)
- moved Q9 5.00 mm to (230.5, 98.0)
- moved D18 4.50 mm to (225.5, 94.0)
- moved D23 4.50 mm to (230.0, 94.0)
- moved Q12 4.50 mm to (225.5, 94.0)
- moved Q7 4.50 mm to (230.5, 94.0)
- moved D19 4.00 mm to (225.5, 90.0)
- moved D21 4.00 mm to (230.0, 90.0)
- moved Q10 4.00 mm to (225.5, 90.0)
- moved Q8 4.00 mm to (230.5, 90.0)
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
Commit message: sync
Parts:
- added C36: 10nF/1kV, Capacitor_SMD:C_1206_3216Metric, F.Cu at (221.5, 32.7)
- added D5: ESDA5V3SC5, Package_TO_SOT_SMD:SOT-23-6, F.Cu at (246.4, 30.6)
- added J5: M80-51004XX, Samacsys:M80-51004YY, F.Cu at (244.2, 15.2)
- added J9: CDMM20M0F2500DET, Samacsys:CDMM20M0F2500DET, F.Cu at (233.5, 57.0)
- added R17: 10k, Resistor_SMD:R_0603_1608Metric, F.Cu at (237.6, 29.4)
- added R18: 10k, Resistor_SMD:R_0603_1608Metric, F.Cu at (237.6, 31.9)
- added RN13: 100, Resistor_SMD:R_Array_Convex_4x0603, F.Cu at (241.7, 30.5)
- D19, D20, D23, D24, D9, Q12, Q5, Q8, Q9: moved to F.Cu
- J11: value M80-5100442 -> CDMM20M0F2500DET; footprint Samacsys:M80-51004YY -> Samacsys:CDMM20M0F2500DET
- J8: value M80-5100442 -> M80-51004XX
- moved Q8 171.3 mm to (60.0, 106.5), turned to 180 degrees
- moved Q9 171.3 mm to (60.0, 114.5), turned to 180 degrees
- moved D23 170.8 mm to (60.0, 110.5), turned to 0 degrees
- moved D17 166.0 mm to (59.5, 84.0)
- moved D18 166.0 mm to (59.5, 92.0)
- moved D21 166.0 mm to (64.0, 88.0)
- moved D22 166.0 mm to (64.0, 96.0)
- moved Q10 166.0 mm to (59.5, 88.0)
- moved Q11 166.0 mm to (59.5, 96.0)
- moved Q6 166.0 mm to (64.5, 84.0)
- moved Q7 166.0 mm to (64.5, 92.0)
- moved D19 161.4 mm to (65.0, 106.5), turned to 180 degrees
- moved D20 161.4 mm to (65.0, 114.5), turned to 180 degrees
- moved Q12 161.4 mm to (65.0, 110.5), turned to 180 degrees
- moved J3 134.5 mm to (84.0, 92.0)
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Connections:
- net /CAR_I_REF renamed Net-(IC3D-+)
- net /Opto Isolation/OPT_OUT0 renamed /Opto Isolation/~{OPT_OUT1}
- net /Opto Isolation/OPT_OUT1 renamed /Opto Isolation/~{OPT_OUT2}
- net /Opto Isolation/OPT_OUT2 renamed /Opto Isolation/~{OPT_OUT3}
- net /Opto Isolation/OPT_OUT3 renamed /Opto Isolation/~{OPT_OUT4}
- net /Opto Isolation/OPT_OUT4 renamed /Opto Isolation/~{OPT_OUT5}
- net /Opto Isolation/OPT_OUT5 renamed /Opto Isolation/~{OPT_OUT6}
- net /Opto Isolation/OPT_OUT6 renamed /Opto Isolation/~{OPT_OUT7}
- net /Opto Isolation/OPT_OUT7 renamed /Opto Isolation/~{OPT_OUT8}
- net /Opto Isolation/~{OPT_IN0} renamed /Opto Isolation/OPT_IN1
- net /Opto Isolation/~{OPT_IN1} renamed /Opto Isolation/OPT_IN2
- net /Opto Isolation/~{OPT_IN2} renamed /Opto Isolation/OPT_IN3
- net /Opto Isolation/~{OPT_IN3} renamed /Opto Isolation/OPT_IN4
- net /Opto Isolation/~{OPT_IN4} renamed /Opto Isolation/OPT_IN5
- net /Opto Isolation/~{OPT_IN5} renamed /Opto Isolation/OPT_IN6
- net /Opto Isolation/~{OPT_IN6} renamed /Opto Isolation/OPT_IN7
- net /Opto Isolation/~{OPT_IN7} renamed /Opto Isolation/OPT_IN8
- C10 pad 2: /Power/SW_5V -> /Power/SW_12V
- C53 pad 1: unconnected-(C53-Pad1) -> GND
- C53 pad 2: unconnected-(C53-Pad2) -> GNDISO
- D4 pad 1: unconnected-(D4-A-Pad1) -> /CAR_I_REF_ADC
- D4 pad 2: Net-(D4-K) -> GNDISO
- D4 pad 3: unconnected-(D4-A-Pad3) -> Net-(RN13C-R3.1)
- D4 pad 4: unconnected-(D4-A-Pad4) -> Net-(IC3B-+)
- D4 pad 5: Net-(D4-K) -> GNDISO
- D4 pad 6: unconnected-(D4-A-Pad6) -> Net-(IC3A-+)
- F1 pad 2: Net-(J11-Pin_4) -> Net-(J8-Pin_3)
- IC3 pad 2: /ACU_V -> Net-(IC3A-+)
- IC3 pad 4: /CAR_V -> Net-(IC3B-+)
- IC3 pad 9: /CAR_I -> Net-(IC3C-+)
- J11 pad 1: unconnected-(J11-Pin_1-Pad1) -> Net-(J7-Pin_1)
- J11 pad 2: unconnected-(J11-Pin_2-Pad2) -> GNDISO
- J11 pad 3: GNDISO -> unconnected-(J11-Pad3)
- J8 pad 1: /OUT+ -> unconnected-(J8-Pin_1-Pad1)
- J8 pad 2: /OUT- -> unconnected-(J8-Pin_2-Pad2)
- J8 pad 4: Net-(J8-Pin_3) -> GNDISO
- L2 pad 1: /Power/SW_5V -> /Power/SW_12V
- U10 pad 1: +3.3V -> Net-(RN6A-R1.1)
- U10 pad 2: Net-(RN6A-R1.1) -> GND
- U10 pad 3: +3.3V -> Net-(RN6B-R2.1)
- U10 pad 4: Net-(RN6B-R2.1) -> GND
- U10 pad 5: +3.3V -> Net-(RN6C-R3.1)
- U10 pad 6: Net-(RN6C-R3.1) -> GND
- U10 pad 7: +3.3V -> Net-(RN6D-R4.1)
- U10 pad 8: Net-(RN6D-R4.1) -> GND
- U12 pad 8: /Power/SW_5V -> /Power/SW_12V

Commit message: sync
Parts:
- removed R32, R33: 33R, Resistor_SMD:R_0603_1608Metric
- removed U5: USBLC6-2SC6, Package_TO_SOT_SMD:SOT-23-6
- added FL2: Choke_Coilcraft_0603USB-142, Inductor_SMD:L_CommonModeChoke_Coilcraft_0603USB, F.Cu at (89.3, 67.3)
- added J1: M80-5100642, Samacsys:M80-51006YY, F.Cu at (137.0, 37.5)
- added J12: M80-51034XX, Samacsys:M80-51034YY, F.Cu at (99.0, 117.5)
- added J2: USB_C_Receptacle_USB2.0_14P, Connector_USB:USB_C_Receptacle_JAE_DX07S024WJ3R400, F.Cu at (136.0, 47.3)
- added J4: FTSH-107-01-L-D-K, Samacsys:FTSH-107-XX-YYY-D-K, F.Cu at (94.2, 56.9)
- added R16: 120, Resistor_SMD:R_0603_1608Metric, F.Cu at (94.5, 70.5)
- moved R7 31.4 mm to (131.0, 52.1)
- moved R8 31.4 mm to (131.0, 54.6)
- moved L4 2.68 mm to (191.6, 74.0)
- moved D22 1.00 mm to (63.0, 96.0), turned to -90 degrees
- moved D24 0.50 mm to (178.5, 92.5)
- moved D9 0.50 mm to (179.0, 84.5)
Other:
- board text added: "${REFERENCE}"
