File: hardware/PUTM_EV_BMS_HV_MASTER_2023.kicad_pcb (KiCad board)
At the start: 4 copper layers, 60 x 100 mm, 176 parts, among them IC1 3.3V/0.6A, IC11 ISO6760, IC2 TPS54202HDDCR, IC3 OPA1679-Q1, IC4 ADS131M04, IC5 LTC1799, IC6 LTC6820IMS, IC7 ISO6760, IC8 3.3V/0.6A, J1 M80-5100642, J10 M300-MV10345M1, J11 CDMM20M0F2500DET, J12 M80-51034XX, J2 USB_C_Receptacle_USB2.0_14P, J3 M80-51014XX, J4 FTSH-107-01-L-D-K, J5 M80-51004XX, J7 M300-MV10345M1, J8 M80-51004XX, J9 CDMM20M0F2500DET, K2 PB134024, Q1 2N7002, Q10 2SK3065, Q11 2SK3065, Q12 2SK3065, Q13 2SK3065, Q2 2N7002, Q3 2N7002, Q4 2SK3065, Q5 2SK3065, Q6 2SK3065, Q7 2SK3065, Q8 2SK3065, Q9 2SK3065, U1 STM32G484RETx, U10 TLP293-4, U12 LMR33640DDDA, U2 74LVC1G86, U3 74AUP1G32, U4 UCC12040DVE, U6 MCP2542FD-E/MF, U7 USBLC6-2SC6, U8 MCP2542FD-E/MF, U9 TLP293-4, Y1 X322516MLB4SI, Y2 Q13FC1350000400

Commit message: sync
Parts:
- removed C58: 10nF/1kV, Capacitor_SMD:C_1206_3216Metric
- removed FL2: Choke_Coilcraft_0603USB-142, Inductor_SMD:L_CommonModeChoke_Coilcraft_0603USB
- removed J11: CDMM20M0F2500DET, Samacsys:CDMM20M0F2500DET
- removed R26: 8.2k, Resistor_SMD:R_0603_1608Metric
- removed R27: 0, Resistor_SMD:R_0603_1608Metric
- removed R30, R31: 1k, Resistor_SMD:R_0603_1608Metric
- removed R38, R39: 33R, Resistor_SMD:R_0603_1608Metric
- removed U10: TLP293-4, Package_SO:SOIC-16_4.55x10.3mm_P1.27mm
- removed U8: MCP2542FD-E/MF, Package_DFN_QFN:DFN-8-1EP_3x3mm_P0.65mm_EP1.55x2.4mm
- added C39: 100nF, Capacitor_SMD:C_0603_1608Metric, F.Cu at (308.1, 65.0)
- added C44: 100nF, Capacitor_SMD:C_0603_1608Metric, F.Cu at (308.1, 67.5)
- added C45: 100nF, Capacitor_SMD:C_0603_1608Metric, F.Cu at (308.1, 70.0)
- added C46: 100nF, Capacitor_SMD:C_0603_1608Metric, F.Cu at (308.1, 72.5)
- added C49: 100nF, Capacitor_SMD:C_0603_1608Metric, F.Cu at (312.2, 40.6)
- added D11: ESDA5V3SC5, Package_TO_SOT_SMD:SOT-23-6, F.Cu at (150.0, 36.1)
- added D12: ESDA5V3SC5, Package_TO_SOT_SMD:SOT-23-6, F.Cu at (142.9, 40.8)
- added D13: ESDA5V3SC5, Package_TO_SOT_SMD:SOT-23-6, F.Cu at (150.0, 40.8)
- added D6: SML-D12U1WT86, LED_SMD:LED_0603_1608Metric, F.Cu at (245.0, 142.0)
- added FL1: Choke_Coilcraft_0603USB-142, Inductor_SMD:L_CommonModeChoke_Coilcraft_0603USB, F.Cu at (131.7, 45.5)
- added J6: CDMM20M0F2500DET, Samacsys:CDMM20M0F2500DET, F.Cu at (297.7, 41.9)
- added JP1: Jumper_3_Bridged12, Jumper:SolderJumper-3_P1.3mm_Bridged2Bar12_RoundedPad1.0x1.5mm, F.Cu at (312.9, 65.5)
- added Q14: 2N7002, Package_TO_SOT_SMD:SOT-23, F.Cu at (128.4, 141.9)
- added Q15: 2N7002, Package_TO_SOT_SMD:SOT-23, F.Cu at (128.4, 146.5)
- added Q16: 2N7002, Package_TO_SOT_SMD:SOT-23, F.Cu at (133.3, 141.9)
- added Q17: 2N7002, Package_TO_SOT_SMD:SOT-23, F.Cu at (133.3, 146.5)
- added Q18: 2N7002, Package_TO_SOT_SMD:SOT-23, F.Cu at (138.2, 141.9)
- added Q19: 2N7002, Package_TO_SOT_SMD:SOT-23, F.Cu at (138.2, 146.5)
- added Q20: 2N7002, Package_TO_SOT_SMD:SOT-23, F.Cu at (143.1, 141.9)
- added Q21: 2N7002, Package_TO_SOT_SMD:SOT-23, F.Cu at (143.1, 146.5)
- added R19: 1k, Resistor_SMD:R_0603_1608Metric, F.Cu at (291.3, 72.5)
- added RN14: 4x200, Resistor_SMD:R_Array_Convex_4x0603, F.Cu at (132.2, 137.1)
- added RN15: 4x10k, Resistor_SMD:R_Array_Convex_4x0603, F.Cu at (136.3, 137.1)
- added RN16: 1k, Resistor_SMD:R_Array_Convex_4x0603, F.Cu at (102.6, 144.3)
- added RN17: 4x200, Resistor_SMD:R_Array_Convex_4x0603, F.Cu at (141.1, 45.4)
- added U5: TLP293-4, Package_SO:SOIC-16_4.55x10.3mm_P1.27mm, F.Cu at (121.1, 135.9)
- C18: value 10nF/1kV -> 100nF; footprint Capacitor_SMD:C_1206_3216Metric -> Capacitor_SMD:C_0603_1608Metric
- C27: value 220nF -> 100nF
- C30: value 100nF -> 10nF
- C31: value 10nF -> 100nF
- C32: footprint Capacitor_SMD:C_0805_2012Metric -> Capacitor_SMD:C_0603_1608Metric
- C38: footprint Capacitor_SMD:C_0603_1608Metric -> Capacitor_SMD:C_0805_2012Metric
- C41: value 100nF -> 220nF
- C43, C50: value 100nF -> 10nF/1kV; footprint Capacitor_SMD:C_0603_1608Metric -> Capacitor_SMD:C_1206_3216Metric
- D8: value SML-D12U1WT86 -> ESDA5V3SC5; footprint LED_SMD:LED_0603_1608Metric -> Package_TO_SOT_SMD:SOT-23-6
- R1, R2, R3: value 1k -> 0
- R15: value 1k -> 10k
- R16: value 120 -> 1k
- R18: value 10k -> 8.2k
- R20: value 0 -> 120
- R21: value 0 -> 10k
- R7, R8: value 5.1k -> 33R
- RN2: value 2k -> 4x200
- RN3: value 500 -> 100
- RN5: value 500 -> 4x1M
- RN6: value 2k -> 100
- RN7: value 4x10k -> 4x1M
- U7: value USBLC6-2SC6 -> MCP2542FD-E/MF; footprint Package_TO_SOT_SMD:SOT-23-6 -> Package_DFN_QFN:DFN-8-1EP_3x3mm_P0.65mm_EP1.55x2.4mm
- moved C41 206.6 mm to (312.2, 38.1)
- moved C27 201.6 mm to (308.2, 38.1)
- moved C35 200.2 mm to (308.2, 48.1)
- moved IC4 199.7 mm to (314.0, 58.4)
- moved R16 196.8 mm to (291.3, 70.0)
- moved IC5 195.5 mm to (308.8, 56.4)
- moved R1 189.7 mm to (312.2, 43.1)
- moved R2 189.7 mm to (312.2, 45.6)
- moved R3 189.7 mm to (312.2, 48.1)
- moved J4 187.7 mm to (261.5, 142.0), turned to 180 degrees
- moved C34 175.6 mm to (308.2, 45.6)
- moved J12 172.5 mm to (271.5, 114.5), turned to -90 degrees
- moved R21 169.8 mm to (316.2, 45.6)
- moved F1 157.6 mm to (312.9, 69.7)
- moved R15 157.4 mm to (316.2, 38.1)
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Connections:
- net /8.192MHZ renamed /Isolated ADC/8.192MHZ
- net /ACU_V_ADC renamed /Isolated ADC/ACU_V_ADC
- net /AIR Control/DRAIN1 renamed /AIR_M
- net /AIR Control/DRAIN2 renamed /AIR_P
- net /AIR Control/DRAIN3 renamed /AIR_PRE
- net /CAR_I_ADC renamed /Isolated ADC/CAR_I_ADC
- net /CAR_V_ADC renamed /Isolated ADC/CAR_V_ADC
- net /FAN1- renamed /Fan drivers/FAN1-
- net /FAN2- renamed /Fan drivers/FAN2-
- net /FAN3- renamed /Fan drivers/FAN3-
- net /FAN4- renamed /Fan drivers/FAN4-
- net /FAN5- renamed /Fan drivers/FAN5-
- net /FAN6- renamed /Fan drivers/FAN6-
- net /FAN7- renamed /Fan drivers/FAN7-
- net /Safety/AMS_OK renamed /AMS_ERROR
- net AIR_M_DETECTION renamed /AIR_M_DETECTION
- net AIR_PRE_DETECTION renamed /AIR_PRE_DETECTION
- net AIR_P_DETECTION renamed /AIR_P_DETECTION
- net AMS_FAULT_COCKPIT renamed /AMS_FAULT_COCKPIT
- net BOOT0 renamed /BOOT0
- net CHARGER_DETECTION renamed /CHARGER_DETECTION
- net D+ renamed /D+
- net D- renamed /D-
- net EXT_RESET renamed /EXT_RESET
- net IMD_SENSENSOR renamed /IMD_SENSENSOR
- net Net-(J10-Pin_1) renamed /Isolated ADC/CAR_V
- net Net-(J5-Pin_3) renamed /SHIELD
- net Net-(J8-Pin_3) renamed I_VDDISO
- net SAFETY_TSMS_IN renamed /SAFETY_TSMS_IN
- C18 pad 1: /I- -> +3.3VISO
- C18 pad 2: /OUT+ -> GNDISO
- C27 pad 1: GNDISO -> +3.3VISO
- C27 pad 2: Net-(IC4-CAP) -> GNDISO
- C30 pad 1: +3.3VISO -> Net-(IC3D-+)
- C32 pad 1: GND -> +5V
- C32 pad 2: +3V3 -> GND
- C34 pad 1: Net-(IC3D-+) -> +3.3VISO
- C35 pad 1: +3.3VISO -> GNDISO
- C35 pad 2: GNDISO -> +3.3VISO
- C38 pad 1: +5V -> GND
- C38 pad 2: GND -> +3V3
- C41 pad 2: +3.3VISO -> Net-(IC4-CAP)
- C43 pad 1: +3.3VISO -> /Isolated SPI/I-
- C43 pad 2: GNDISO -> /Isolated SPI/OUT+
- C50 pad 1: GNDISO -> /Isolated SPI/I+
- C50 pad 2: +3.3VISO -> /Isolated SPI/OUT-
- D1 pad 1: Net-(D1-K) -> /LED3
- D2 pad 1: Net-(D2-K) -> /LED2
- D3 pad 1: Net-(D3-K) -> /LED1
- D4 pad 1: /CAR_I_REF_ADC -> /Isolated ADC/CAR_I_REF_ADC
- D5 pad 3: /I+ -> /Isolated SPI/I+
- D5 pad 4: /I- -> /Isolated SPI/I-
- D8 pad 1: GND -> unconnected-(D8-A-Pad1)
- D8 pad 2: Net-(D8-A) -> GND
- F1 pad 1: +5VISO -> Net-(JP1-C)
- IC11 pad 1: unconnected-(IC11-VCC1-Pad1) -> +3.3VISO
- IC11 pad 13: unconnected-(IC11-OUTC-Pad13) -> /MCU/LTC_MISO
- IC11 pad 14: unconnected-(IC11-OUTB-Pad14) -> /MCU/ADC_MISO
- IC11 pad 15: unconnected-(IC11-OUTA-Pad15) -> /MCU/~{ADC_DRY}
- IC11 pad 16: unconnected-(IC11-VCC2-Pad16) -> +3V3
- IC11 pad 2: unconnected-(IC11-INA-Pad2) -> /~{ISO_ADC_DRY}
- IC11 pad 3: unconnected-(IC11-INB-Pad3) -> /ISO_ADC_MISO
- IC11 pad 4: unconnected-(IC11-INC-Pad4) -> /ISO_LTC_MISO
- IC11 pad 5: unconnected-(IC11-IND-Pad5) -> GNDISO
- IC11 pad 6: unconnected-(IC11-INE-Pad6) -> GNDISO
- IC11 pad 7: unconnected-(IC11-INF-Pad7) -> GNDISO
- IC11 pad 8: unconnected-(IC11-GND1-Pad8) -> GNDISO
- IC11 pad 9: unconnected-(IC11-GND2-Pad9) -> GND
- IC3 pad 12: /CAR_I_REF_ADC -> /Isolated ADC/CAR_I_REF_ADC
- IC3 pad 14: /CAR_I_REF_ADC -> /Isolated ADC/CAR_I_REF_ADC
- IC4 pad 10: unconnected-(IC4-~{CS}-Pad10) -> /~{ISO_ADC_CS}
- IC4 pad 11: unconnected-(IC4-~{DRY}-Pad11) -> /~{ISO_ADC_DRY}
- IC4 pad 12: unconnected-(IC4-SCK-Pad12) -> /ISO_ADC_SCK
- IC4 pad 13: unconnected-(IC4-SDO-Pad13) -> /ISO_ADC_MISO
- IC4 pad 14: unconnected-(IC4-SDI-Pad14) -> /ISO_ADC_MOSI
- IC4 pad 6: /CAR_I_REF_ADC -> /Isolated ADC/CAR_I_REF_ADC
- IC4 pad 7: unconnected-(IC4-CH3+-Pad7) -> /Isolated ADC/CAR_I_REF_ADC
- IC4 pad 8: unconnected-(IC4-CH3--Pad8) -> GNDISO
- IC4 pad 9: unconnected-(IC4-~{SYNC}-Pad9) -> Net-(IC4-~{SYNC})
- IC6 pad 10: /I+ -> /Isolated SPI/I+
- IC6 pad 11: /I- -> /Isolated SPI/I-
- IC6 pad 2: unconnected-(IC6-MOSI-Pad2) -> /ISO_LTC_MOSI
- IC6 pad 3: unconnected-(IC6-MISO-Pad3) -> /ISO_LTC_MISO
- IC6 pad 4: unconnected-(IC6-SCK-Pad4) -> /ISO_LTC_SCK
- IC6 pad 5: unconnected-(IC6-~{CS}-Pad5) -> /~{ISO_LTC_CS}
- IC7 pad 1: unconnected-(IC7-VCC1-Pad1) -> +3V3
- IC7 pad 10: unconnected-(IC7-OUTF-Pad10) -> /~{ISO_LTC_CS}
- IC7 pad 11: unconnected-(IC7-OUTE-Pad11) -> /ISO_LTC_SCK
- IC7 pad 12: unconnected-(IC7-OUTD-Pad12) -> /ISO_LTC_MOSI
- IC7 pad 13: unconnected-(IC7-OUTC-Pad13) -> /~{ISO_ADC_CS}
- IC7 pad 14: unconnected-(IC7-OUTB-Pad14) -> /ISO_ADC_SCK
- IC7 pad 15: unconnected-(IC7-OUTA-Pad15) -> /ISO_ADC_MOSI
- IC7 pad 16: unconnected-(IC7-VCC2-Pad16) -> +3.3VISO
- IC7 pad 2: unconnected-(IC7-INA-Pad2) -> /MCU/ADC_MOSI
- IC7 pad 3: unconnected-(IC7-INB-Pad3) -> /MCU/ADC_SCK
- IC7 pad 4: unconnected-(IC7-INC-Pad4) -> /MCU/~{ADC_CS}
- IC7 pad 5: unconnected-(IC7-IND-Pad5) -> /MCU/LTC_MOSI
- IC7 pad 6: unconnected-(IC7-INE-Pad6) -> /MCU/LTC_SCK
- IC7 pad 7: unconnected-(IC7-INF-Pad7) -> /MCU/~{LTC_CS}
- IC7 pad 8: unconnected-(IC7-GND1-Pad8) -> GND
- IC7 pad 9: unconnected-(IC7-GND2-Pad9) -> GNDISO
- J12 pad 16: EX_D- -> unconnected-(J12-Pin_16-Pad16)
- J12 pad 17: EX_D+ -> unconnected-(J12-Pin_17-Pad17)
- J12 pad 24: CANFD1- -> /CANFD1-
- J12 pad 25: CANFD2- -> /CANFD2-
- J12 pad 34: EX_VBUS -> GND
- J12 pad 4: AMS_SAFETY_1 -> /AMS_SAFETY_1
- J12 pad 5: AMS_SAFETY_2 -> /AMS_SAFETY_2
- J12 pad 7: CANFD1+ -> /CANFD1+
- J12 pad 8: CANFD2+ -> /CANFD2+
- J2 pad A4: VBUS -> unconnected-(J2-VBUS-PadA4)
- J2 pad A5: Net-(J2-CC1) -> unconnected-(J2-CC1-PadA5)
- J2 pad A9: VBUS -> unconnected-(J2-VBUS-PadA4)_3
- J2 pad B4: VBUS -> unconnected-(J2-VBUS-PadA4)_2
- J2 pad B5: Net-(J2-CC2) -> unconnected-(J2-CC2-PadB5)
- J2 pad B9: VBUS -> unconnected-(J2-VBUS-PadA4)_1
- J4 pad 12: NRST -> /NRST
- J4 pad 4: SWDIO -> /SWDIO
- J4 pad 6: SWCLK -> /SWCLK
- J5 pad 1: /OUT+ -> /Isolated SPI/OUT-
- J5 pad 2: /OUT- -> /Isolated SPI/OUT+
- J7 pad 1: Net-(J7-Pin_1) -> /Isolated ADC/ACU_V
- J8 pad 1: unconnected-(J8-Pin_1-Pad1) -> /Isolated ADC/CAR_I
- J8 pad 2: unconnected-(J8-Pin_2-Pad2) -> /Isolated ADC/CAR_I_REF
- J9 pad 3: unconnected-(J9-Pad3) -> Net-(RN13B-R2.2)
- R1 pad 1: /MCU/SIGNAL_LED_3 -> Net-(IC3D-+)
- R1 pad 2: Net-(D1-K) -> +5VISO
- R15 pad 1: /Safety/AMS_FAULT -> Net-(RN13C-R3.1)
- R15 pad 2: Net-(D8-A) -> Net-(IC3C-+)
- R16 pad 1: /I- -> Net-(IC6-ICMP)
- R16 pad 2: /I+ -> Net-(IC6-IBIAS)
- R17 pad 1: Net-(RN13C-R3.1) -> Net-(IC3C-+)
- R17 pad 2: Net-(IC3C-+) -> GNDISO
- R18 pad 1: Net-(IC3C-+) -> Net-(IC5-SET)
- R18 pad 2: GNDISO -> +3.3VISO
- R2 pad 1: /MCU/SIGNAL_LED_2 -> Net-(IC3D-+)
- R2 pad 2: Net-(D2-K) -> +3.3VISO
- R20 pad 1: Net-(IC3D-+) -> /Isolated SPI/I-
- R20 pad 2: +3.3VISO -> /Isolated SPI/I+
- R21 pad 1: Net-(IC3D-+) -> Net-(IC4-~{SYNC})
- R21 pad 2: GNDISO -> +3.3VISO
- R3 pad 1: /MCU/SIGNAL_LED_1 -> Net-(IC3D-+)
- R3 pad 2: Net-(D3-K) -> GNDISO
- R4 pad 1: /MCU/NRST -> /NRST
- R5 pad 1: /MCU/MES_MISO -> /MCU/ADC_MISO
- R7 pad 1: Net-(J2-CC2) -> /Connectivity/MCU_D-
- R7 pad 2: GND -> Net-(FL1-Pad2)
- R8 pad 1: Net-(J2-CC1) -> Net-(FL1-Pad3)
- R8 pad 2: GND -> /Connectivity/MCU_D+
- RN13 pad 4: /CAR_I_REF_ADC -> /Isolated ADC/CAR_I_REF_ADC
- RN13 pad 5: /CAR_I_REF -> /Isolated ADC/CAR_I_REF
- RN13 pad 6: /CAR_I -> /Isolated ADC/CAR_I
- RN13 pad 7: /CAR_V -> Net-(RN13B-R2.2)
- RN13 pad 8: /ACU_V -> Net-(RN13A-R1.2)
- RN2 pad 1: Net-(RN2A-R1.1) -> +3.3V
- RN2 pad 2: Net-(RN2B-R2.1) -> +3.3V
- RN2 pad 3: Net-(RN2C-R3.1) -> +3.3V
- RN2 pad 4: Net-(RN2D-R4.1) -> +3.3V
- RN2 pad 5: Net-(RN2D-R4.2) -> Net-(RN2-R4.2)
- RN2 pad 6: Net-(RN2C-R3.2) -> Net-(RN2-R3.2)
- RN2 pad 7: Net-(RN2B-R2.2) -> Net-(RN2-R2.2)
- RN2 pad 8: Net-(RN2A-R1.2) -> Net-(RN2-R1.2)
- RN3 pad 1: Net-(RN3A-R1.1) -> Net-(Q14-G)
- RN3 pad 2: Net-(RN3B-R2.1) -> Net-(Q15-G)
- RN3 pad 3: Net-(RN3C-R3.1) -> Net-(Q16-G)
- RN3 pad 4: Net-(RN3D-R4.1) -> Net-(Q17-G)
- RN3 pad 5: /Opto Isolation/OPT_IN8 -> /Opto Isolation/OPT_IN4
- RN3 pad 6: /Opto Isolation/OPT_IN7 -> /Opto Isolation/OPT_IN3
- RN3 pad 7: /Opto Isolation/OPT_IN6 -> /Opto Isolation/OPT_IN2
- RN3 pad 8: /Opto Isolation/OPT_IN5 -> /Opto Isolation/OPT_IN1
- RN5 pad 1: Net-(RN2A-R1.2) -> Net-(Q17-G)
- RN5 pad 2: Net-(RN2B-R2.2) -> Net-(Q16-G)
- RN5 pad 3: Net-(RN2C-R3.2) -> Net-(Q15-G)
- RN5 pad 4: Net-(RN2D-R4.2) -> Net-(Q14-G)
- RN5 pad 5: /Opto Isolation/OPT_IN4 -> GND
- RN5 pad 6: /Opto Isolation/OPT_IN3 -> GND
- RN5 pad 7: /Opto Isolation/OPT_IN2 -> GND
- RN5 pad 8: /Opto Isolation/OPT_IN1 -> GND
- RN6 pad 1: Net-(RN6A-R1.1) -> Net-(Q18-G)
- RN6 pad 2: Net-(RN6B-R2.1) -> Net-(Q19-G)
- RN6 pad 3: Net-(RN6C-R3.1) -> Net-(Q20-G)
- RN6 pad 4: Net-(RN6D-R4.1) -> Net-(Q21-G)
- RN6 pad 5: Net-(RN3D-R4.1) -> /Opto Isolation/OPT_IN8
- RN6 pad 6: Net-(RN3C-R3.1) -> /Opto Isolation/OPT_IN7
- RN6 pad 7: Net-(RN3B-R2.1) -> /Opto Isolation/OPT_IN6
- RN6 pad 8: Net-(RN3A-R1.1) -> /Opto Isolation/OPT_IN5
- RN7 pad 1: +3.3V -> Net-(Q21-G)
- RN7 pad 2: +3.3V -> Net-(Q20-G)
- RN7 pad 3: +3.3V -> Net-(Q19-G)
- RN7 pad 4: +3.3V -> Net-(Q18-G)
- RN7 pad 5: /Opto Isolation/~{OPT_OUT5} -> GND
- RN7 pad 6: /Opto Isolation/~{OPT_OUT6} -> GND
- RN7 pad 7: /Opto Isolation/~{OPT_OUT7} -> GND
- RN7 pad 8: /Opto Isolation/~{OPT_OUT8} -> GND
- U1 pad 10: /MCU/FAN_5_CTRL -> /Fan drivers/FAN5_CTRL
- U1 pad 11: /MCU/FAN_4_CTRL -> /Fan drivers/FAN4_CTRL
- U1 pad 12: /MCU/FAN_3_CTRL -> /Fan drivers/FAN3_CTRL
- U1 pad 13: /MCU/FAN_2_CTRL -> /Fan drivers/FAN2_CTRL
- U1 pad 14: /MCU/FAN_1_CTRL -> /Fan drivers/FAN1_CTRL
- U1 pad 23: /MCU/SIGNAL_LED_1 -> /SIGNAL_LED_1
- U1 pad 24: /MCU/SIGNAL_LED_2 -> /SIGNAL_LED_2
- U1 pad 25: /MCU/SIGNAL_LED_3 -> /SIGNAL_LED_3
- U1 pad 33: /MCU/LTC_2_~{CS} -> /MCU/~{ADC_DRY}
- U1 pad 34: /MCU/LTC_1_~{CS} -> /MCU/~{LTC_CS}
- U1 pad 39: /MCU/SIGNAL_AIR_PRE -> /AIR Control/SIGNAL3
- U1 pad 40: /MCU/SIGNAL_AIR_P -> /AIR Control/SIGNAL2
- U1 pad 41: /MCU/SIGNAL_AIR_M -> /AIR Control/SIGNAL1
- U1 pad 42: /MCU/~{MES_I_SENS_CS} -> unconnected-(U1A-PA8-Pad42)
- U1 pad 43: /MCU/~{MES_EXT_V_CS} -> /Connectivity/IN4
- U1 pad 44: /MCU/~{MES_EXT_I_CS} -> unconnected-(U1A-PA10-Pad44)
- U1 pad 45: /MCU/MCU_D- -> /Connectivity/MCU_D-
- U1 pad 46: /MCU/MCU_D+ -> /Connectivity/MCU_D+
- U1 pad 49: /MCU/SWDIO -> /SWDIO
- U1 pad 50: /MCU/SWCLK -> /SWCLK
- U1 pad 51: /MCU/SIGNAL_AMS_FAULT -> /Safety/IN
- U1 pad 52: /MCU/MES_SCK -> /MCU/ADC_SCK
- U1 pad 53: /MCU/MES_MISO -> /MCU/ADC_MISO
- U1 pad 54: /MCU/MES_MOSI -> /MCU/ADC_MOSI
- U1 pad 55: /MCU/~{MES_V_CAR_CS} -> unconnected-(U1A-PD2-Pad55)
- U1 pad 56: /MCU/MCU_CANFD2_RX -> /Connectivity/MCU_CANFD2_RX
- U1 pad 57: /MCU/MCU_CANFD2_TX -> /Connectivity/MCU_CANFD2_TX
- U1 pad 58: /MCU/MCU_CANFD1_RX -> /Connectivity/MCU_CANFD1_RX
- U1 pad 59: /MCU/MCU_CANFD1_TX -> /Connectivity/MCU_CANFD1_TX
- U1 pad 60: /MCU/~{MES_V_ACU_CS} -> /MCU/~{ADC_CS}
- U1 pad 7: /MCU/NRST -> /NRST
- U1 pad 8: /MCU/FAN_7_CTRL -> /Fan drivers/FAN7_CTRL
- U1 pad 9: /MCU/FAN_6_CTRL -> /Fan drivers/FAN6_CTRL
- U6 pad 1: /MCU_CANFD2_TX -> /Connectivity/MCU_CANFD2_TX
- U6 pad 4: /MCU_CANFD2_RX -> /Connectivity/MCU_CANFD2_RX
- U6 pad 6: CANFD2- -> /Connectivity/CANFD2-
- U6 pad 7: CANFD2+ -> /Connectivity/CANFD2+
- U7 pad 1: /MCU_D- -> /Connectivity/MCU_CANFD1_TX
- U7 pad 3: /MCU_D+ -> +5V
- U7 pad 4: Net-(R38-Pad1) -> /Connectivity/MCU_CANFD1_RX
- U7 pad 5: EX_VBUS -> +3V3
- U7 pad 6: Net-(R39-Pad2) -> /Connectivity/CANFD1-
- U9 pad 1: Net-(RN2A-R1.1) -> Net-(RN2-R1.2)
- U9 pad 2: GND -> Net-(Q14-D)
- U9 pad 3: Net-(RN2B-R2.1) -> Net-(RN2-R2.2)
- U9 pad 4: GND -> Net-(Q15-D)
- U9 pad 5: Net-(RN2C-R3.1) -> Net-(RN2-R3.2)
- U9 pad 6: GND -> Net-(Q16-D)
- U9 pad 7: Net-(RN2D-R4.1) -> Net-(RN2-R4.2)
- U9 pad 8: GND -> Net-(Q17-D)
Other:
- board text added: "AIRS"
- board text added: "ERR1"
- board text added: "ERR2"
- board text added: "FANS"
- board text added: "ISENS"
- board text added: "LTC"
- board text added: "MAIN"
- board text added: "OK"
- board text added: "SWD"
- board text added: "USB 2.0"
- board text added: "WARN"
