File: hardware/PUTM_EV_AMS_MASTER_2025.kicad_pcb (KiCad board)
At the start: 4 copper layers, 60 x 100 mm, 263 parts, among them IC1 TPS7B92033DBVR, IC11 ISO6760, IC2 TPS54202HDDCR, IC3 BQ79600PWRQ1, IC5 LTC1799, IC6 LTC6820IMS, IC7 ISO6760, IC8 3.3V/0.5A, J1 M80-5100642, J10 M300-MV10345M1, J12 M80-51034XX, J2 USB_C_Receptacle_USB2.0_14P, J3 M80-51014XX, J4 FTSH-107-01-L-D-K, J5 M80-51004XX, J7 M300-MV10345M1, J8 M80-51004XX, K1 IMB03ITS, Q1 DMT6018LDR-7, Q2 DMT6018LDR-7, Q3 DMT6018LDR-7, Q4 DMT6018LDR-7, Q5 DMT6018LDR-7, Q6 2N7002, Q7 DMT6018LDR-7, Q8 2N7002, Q9 2N7002, T1 >100kHz, U1 MCP2542FD-E/MF, U10 STM32G484VEHx, U12 LMR33640DDDA, U13 LM397, U2 LM397, U3 74AUP1G32, U4 UCC12040DVE, U5 LM397, U6 MCP2542FD-E/MF, U7 MCP2542FD-E/MF, U8 LM397, U9 LM397, Y1 X322516MLB4SI

Commit message: some routing done
Parts:
- moved R49 100.1 mm to (134.2, 124.0)
- moved R50 100.1 mm to (134.2, 122.5)
- moved R51 100.1 mm to (137.2, 124.0)
- moved R52 100.1 mm to (137.2, 122.5)
- moved D12 99.9 mm to (135.8, 122.8)
- moved D11 96.7 mm to (135.8, 126.8)
- moved R7 95.2 mm to (137.2, 127.0)
- moved R8 95.2 mm to (137.2, 125.5)
- moved C30 45.7 mm to (147.5, 66.5)
- moved R2 45.5 mm to (151.5, 62.0), turned to -90 degrees
- moved R1 42.3 mm to (143.5, 62.0), turned to 90 degrees
- moved R6 42.0 mm to (147.5, 64.5)
- moved C67 35.2 mm to (124.5, 66.5)
- moved R53 31.9 mm to (120.5, 62.0)
- moved R54 31.5 mm to (128.5, 62.0)
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Connections:
- Q1 pad 1: /AIR Control/G2 -> /AIR Control/G3
- R45 pad 2: /AIR Control/G2 -> /AIR Control/G3
- R48 pad 2: /AIR Control/G2 -> /AIR Control/G3
- U10 pad F4: /MCU/PG_12V -> unconnected-(U10-PC1-PadF4)
- U10 pad G2: unconnected-(U10-PA1-PadG2) -> /MCU/PG_12V
- U10 pad H1: unconnected-(U10-PA2-PadH1) -> /SIGNAL_LED_2
- U10 pad H6: /SIGNAL_LED_2 -> unconnected-(U10-PE9-PadH6)
- U10 pad H7: /MCU/SIGNAL_AMS_ERROR -> unconnected-(U10-PE15-PadH7)
- U10 pad J8: unconnected-(U10-PB10-PadJ8) -> /MCU/SIGNAL_AMS_ERROR
Routing:
- net +24V: track 47.1 -> 113.1 mm
- net +5V: track 25.4 -> 90.3 mm
- net +3.3V: track 103.1 -> 152.0 mm
- net TSMS: track 0.00 -> 44.4 mm, vias 0 -> 1
- net GND: track 16.5 -> 53.3 mm, vias 6 -> 23
- net /TSMS_AIRS: track 0.00 -> 27.2 mm, vias 4 -> 5
- net VDD: track 0.00 -> 8.55 mm
- net /AIR_P: track 4.87 -> 12.4 mm
- net /AIR_M: track 3.47 -> 10.6 mm
- net /AIR_PRE: track 3.47 -> 10.2 mm
- net /Power/F_24V: track 0.00 -> 6.56 mm
- net /AIR Control/G2: track 11.0 -> 5.24 mm, vias 2 -> 1
- net /Isolated ADC/CAR-: track 0.00 -> 5.25 mm
- net /Isolated ADC/CAR+: track 0.00 -> 5.25 mm
- net /Isolated ADC/ACU-: track 0.00 -> 5.25 mm
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