File: hardware/FanControl.kicad_sch (KiCad schematic)
At the start: 25 parts, among them Q2 DMT6018LDR-7, Q3 DMT6018LDR-7, Q4 DMT6018LDR-7, Q5 DMT6018LDR-7

Commit message: bom update
Parts:
- D13, D17, D18, D19, D20, D21, D8: value VSSB410S-E3/52T -> 60V/0.5/3A; Manufacturer_Part_Number VSSB410S-E3/52T -> (none); Mouser Part Number 625-VSSB410S-E3/52T -> 637-SKL36; Mouser Price/Stock https://www.mouser.pl/ProductDetail/Vishay-General-Semicond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 -> (none)
- R30, R5, R58, R59, R62, R63, R66: Mouser Part Number (none) -> --
- R56, R57, R60, R61, R64, R65, R67: Mouser Part Number (none) -> --; Mouser Price/Stock https://www.mouser.pl/ProductDetail/YAGEO/RT0603DRE07100KL?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 -> (none)
Changed lines of the file:
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@@
 			)
 		)
-		(property "Value" "VSSB410S-E3/52T"
+		(property "Value" "60V/0.5/3A"
 			(at 166.37 31.4959 90)
 			(effects
@@
 			)
 		)
-		(property "Manufacturer_Part_Number" "VSSB410S-E3/52T"
+		(property "Manufacturer_Part_Number" ""
 			(at 163.83 30.48 0)
 			(effects
@@
 			)
 		)
-		(property "Mouser Part Number" "625-VSSB410S-E3/52T"
+		(property "Mouser Part Number" "637-SKL36"
 			(at 163.83 30.48 0)
 			(effects
@@
 			)
 		)
-		(property "Mouser Price/Stock" "https://www.mouser.pl/ProductDetail/Vishay-General-Semiconductor/VSSB410S-E3-52T?qs=HSPD0Bff7ib64J9oD9YilA%3D%3D"
+		(property "Mouser Price/Stock" ""
 			(at 163.83 30.48 0)
 			(effects
@@
 			)
 		)
-		(property "Mouser Price/Stock" "https://www.mouser.pl/ProductDetail/YAGEO/RT0603DRE07100KL?qs=sGAEpiMZZMvdGkrng054t1nmr2c61WvadC66rbrHowc%3D"
+		(property "Mouser Price/Stock" ""
+			(at 227.33 48.26 0)
+			(effects
+				(font
+					(size 1.27 1.27)
+				)
+				(hide yes)
+			)
+		)
+		(property "Mouser Part Number" "--"
 			(at 227.33 48.26 0)
 			(effects
@@
 			)
 		)
-		(property "Mouser Price/Stock" "https://www.mouser.pl/ProductDetail/YAGEO/RT0603DRE07100KL?qs=sGAEpiMZZMvdGkrng054t1nmr2c61WvadC66rbrHowc%3D"
+		(property "Mouser Price/Stock" ""
+			(at 153.67 111.76 0)
+			(effects
+				(font
+					(size 1.27 1.27)
+				)
+				(hide yes)
+			)
+		)
+		(property "Mouser Part Number" "--"
 			(at 153.67 111.76 0)
 			(effects
@@
 			)
 		)
-		(property "Value" "VSSB410S-E3/52T"
+		(property "Value" "60V/0.5/3A"
 			(at 92.71 153.4159 90)
 			(effects
@@
 			)
 		)
-		(property "Manufacturer_Part_Number" "VSSB410S-E3/52T"
+		(property "Manufacturer_Part_Number" ""
 			(at 90.17 152.4 0)
 			(effects
@@
 			)
 		)
-		(property "Mouser Part Number" "625-VSSB410S-E3/52T"
+		(property "Mouser Part Number" "637-SKL36"
 			(at 90.17 152.4 0)
 			(effects
@@
 			)
 		)
-		(property "Mouser Price/Stock" "https://www.mouser.pl/ProductDetail/Vishay-General-Semiconductor/VSSB410S-E3-52T?qs=HSPD0Bff7ib64J9oD9YilA%3D%3D"
+		(property "Mouser Price/Stock" ""
 			(at 90.17 152.4 0)
 			(effects
@@
 			)
 		)
-		(property "Mouser Price/Stock" "https://www.mouser.pl/ProductDetail/YAGEO/RT0603DRE07100KL?qs=sGAEpiMZZMvdGkrng054t1nmr2c61WvadC66rbrHowc%3D"
+		(property "Mouser Price/Stock" ""
+			(at 80.01 111.76 0)
+			(effects
+				(font
+					(size 1.27 1.27)
+				)
+				(hide yes)
+			)
+		)
+		(property "Mouser Part Number" "--"
 			(at 80.01 111.76 0)
 			(effects
@@
 			)
 		)
-		(property "Value" "VSSB410S-E3/52T"
+		(property "Value" "60V/0.5/3A"
 			(at 240.03 31.4959 90)
 			(effects
@@
 			)
 		)
-		(property "Manufacturer_Part_Number" "VSSB410S-E3/52T"
+		(property "Manufacturer_Part_Number" ""
 			(at 237.49 30.48 0)
 			(effects
@@
 			)
 		)
-		(property "Mouser Part Number" "625-VSSB410S-E3/52T"
+		(property "Mouser Part Number" "637-SKL36"
 			(at 237.49 30.48 0)
 			(effects
@@
 			)
 		)
-		(property "Mouser Price/Stock" "https://www.mouser.pl/ProductDetail/Vishay-General-Semiconductor/VSSB410S-E3-52T?qs=HSPD0Bff7ib64J9oD9YilA%3D%3D"
+		(property "Mouser Price/Stock" ""
 			(at 237.49 30.48 0)
 			(effects
@@
 			)
 		)
-		(property "Mouser Price/Stock" "https://www.mouser.pl/ProductDetail/YAGEO/RT0603DRE07100KL?qs=sGAEpiMZZMvdGkrng054t1nmr2c61WvadC66rbrHowc%3D"
+		(property "Mouser Price/Stock" ""
+			(at 80.01 48.26 0)
+			(effects
+				(font
+					(size 1.27 1.27)
+				)
+				(hide yes)
+			)
+		)
+		(property "Mouser Part Number" "--"
 			(at 80.01 48.26 0)
 			(effects
@@
 			)
 		)
+		(property "Mouser Part Number" "--"
+			(at 72.39 43.18 0)
+			(effects
+				(font
+					(size 1.27 1.27)
+				)
+				(hide yes)
+			)
+		)
 		(pin "1"
 		)
@@
 			)
 		)
-		(property "Value" "VSSB410S-E3/52T"
+		(property "Value" "60V/0.5/3A"
 			(at 92.71 94.9959 90)
 			(effects
@@
 			)
 		)
-		(property "Manufacturer_Part_Number" "VSSB410S-E3/52T"
+		(property "Manufacturer_Part_Number" ""
 			(at 90.17 93.98 0)
 			(effects
@@
 			)
 		)
-		(property "Mouser Part Number" "625-VSSB410S-E3/52T"
+		(property "Mouser Part Number" "637-SKL36"
 			(at 90.17 93.98 0)
 			(effects
@@
 			)
 		)
-		(property "Mouser Price/Stock" "https://www.mouser.pl/ProductDetail/Vishay-General-Semiconductor/VSSB410S-E3-52T?qs=HSPD0Bff7ib64J9oD9YilA%3D%3D"
+		(property "Mouser Price/Stock" ""
 			(at 90.17 93.98 0)
 			(effects
@@
 			)
 		)
-		(property "Value" "VSSB410S-E3/52T"
+		(property "Value" "60V/0.5/3A"
 			(at 92.71 31.4959 90)
 			(effects
@@
 			)
 		)
-		(property "Manufacturer_Part_Number" "VSSB410S-E3/52T"
+		(property "Manufacturer_Part_Number" ""
 			(at 90.17 30.48 0)
 			(effects
@@
 			)
 		)
-		(property "Mouser Part Number" "625-VSSB410S-E3/52T"
+		(property "Mouser Part Number" "637-SKL36"
 			(at 90.17 30.48 0)
 			(effects
@@
 			)
 		)
-		(property "Mouser Price/Stock" "https://www.mouser.pl/ProductDetail/Vishay-General-Semiconductor/VSSB410S-E3-52T?qs=HSPD0Bff7ib64J9oD9YilA%3D%3D"
+		(property "Mouser Price/Stock" ""
 			(at 90.17 30.48 0)
 			(effects
@@
 			)
 		)
+		(property "Mouser Part Number" "--"
+			(at 72.39 165.1 0)
+			(effects
+				(font
+					(size 1.27 1.27)
+				)
+				(hide yes)
+			)
+		)
 		(pin "1"
 		)
@@
 			)
 		)
-		(property "Value" "VSSB410S-E3/52T"
+		(property "Value" "60V/0.5/3A"
 			(at 240.03 94.9959 90)
 			(effects
@@
 			)
 		)
-		(property "Manufacturer_Part_Number" "VSSB410S-E3/52T"
+		(property "Manufacturer_Part_Number" ""
 			(at 237.49 93.98 0)
 			(effects
@@
 			)
 		)
-		(property "Mouser Part Number" "625-VSSB410S-E3/52T"
+		(property "Mouser Part Number" "637-SKL36"
 			(at 237.49 93.98 0)
 			(effects
@@
 			)
 		)
-		(property "Mouser Price/Stock" "https://www.mouser.pl/ProductDetail/Vishay-General-Semiconductor/VSSB410S-E3-52T?qs=HSPD0Bff7ib64J9oD9YilA%3D%3D"
+		(property "Mouser Price/Stock" ""
 			(at 237.49 93.98 0)
 			(effects
@@
 			)
 		)
-		(property "Mouser Price/Stock" "https://www.mouser.pl/ProductDetail/YAGEO/RT0603DRE07100KL?qs=sGAEpiMZZMvdGkrng054t1nmr2c61WvadC66rbrHowc%3D"
+		(property "Mouser Price/Stock" ""
+			(at 153.67 48.26 0)
+			(effects
+				(font
+					(size 1.27 1.27)
+				)
+				(hide yes)
+			)
+		)
+		(property "Mouser Part Number" "--"
 			(at 153.67 48.26 0)
 			(effects
@@
 			)
 		)
+		(property "Mouser Part Number" "--"
+			(at 146.05 43.18 0)
+			(effects
+				(font
+					(size 1.27 1.27)
+				)
+				(hide yes)
+			)
+		)
 		(pin "1"
 		)
@@
 			)
 		)
+		(property "Mouser Part Number" "--"
+			(at 219.71 106.68 0)
+			(effects
+				(font
+					(size 1.27 1.27)
+				)
+				(hide yes)
+			)
+		)
 		(pin "1"
 		)
@@
 			)
 		)
+		(property "Mouser Part Number" "--"
+			(at 146.05 106.68 0)
+			(effects
+				(font
+					(size 1.27 1.27)
+				)
+				(hide yes)
+			)
+		)
 		(pin "1"
 		)
@@
 			)
 		)
+		(property "Mouser Part Number" "--"
+			(at 219.71 43.18 0)
+			(effects
+				(font
+					(size 1.27 1.27)
+				)
+				(hide yes)
+			)
+		)
 		(pin "1"
 		)
@@
 			)
 		)
-		(property "Value" "VSSB410S-E3/52T"
+		(property "Value" "60V/0.5/3A"
 			(at 166.37 94.9959 90)
 			(effects
@@
 			)
 		)
-		(property "Manufacturer_Part_Number" "VSSB410S-E3/52T"
+		(property "Manufacturer_Part_Number" ""
 			(at 163.83 93.98 0)
 			(effects
@@
 			)
 		)
-		(property "Mouser Part Number" "625-VSSB410S-E3/52T"
+		(property "Mouser Part Number" "637-SKL36"
 			(at 163.83 93.98 0)
 			(effects
@@
 			)
 		)
-		(property "Mouser Price/Stock" "https://www.mouser.pl/ProductDetail/Vishay-General-Semiconductor/VSSB410S-E3-52T?qs=HSPD0Bff7ib64J9oD9YilA%3D%3D"
+		(property "Mouser Price/Stock" ""
 			(at 163.83 93.98 0)
 			(effects
@@
 			)
 		)
-		(property "Mouser Price/Stock" "https://www.mouser.pl/ProductDetail/YAGEO/RT0603DRE07100KL?qs=sGAEpiMZZMvdGkrng054t1nmr2c61WvadC66rbrHowc%3D"
+		(property "Mouser Price/Stock" ""
+			(at 80.01 170.18 0)
+			(effects
+				(font
+					(size 1.27 1.27)
+				)
+				(hide yes)
+			)
+		)
+		(property "Mouser Part Number" "--"
 			(at 80.01 170.18 0)
 			(effects
@@
 			)
 		)
-		(property "Mouser Price/Stock" "https://www.mouser.pl/ProductDetail/YAGEO/RT0603DRE07100KL?qs=sGAEpiMZZMvdGkrng054t1nmr2c61WvadC66rbrHowc%3D"
+		(property "Mouser Price/Stock" ""
+			(at 227.33 111.76 0)
+			(effects
+				(font
+					(size 1.27 1.27)
+				)
+				(hide yes)
+			)
+		)
+		(property "Mouser Part Number" "--"
 			(at 227.33 111.76 0)
 			(effects
@@
 			(at 72.39 106.68 0)
 			(effects
+				(font
+					(size 1.27 1.27)
+				)
+				(hide yes)
+			)
+		)
+		(property "Mouser Part Number" "--"
+			(at 72.39 106.68 0)
+			(effects
