File: hardware/IsolatedSPI.kicad_sch (KiCad schematic)
At the start: 18 parts, among them IC3 BQ79600PWRQ1, IC6 LTC6820IMS

Commit message: layotu done, some more routing done
Connections:
- net COM+: now reaches C79.2, IC3.13 (COMHP), R96.2, R97.2
- net COM-: now reaches C80.2, IC3.12 (COMHN), R97.1, R98.2
- net DVDD: now reaches C53.1, IC3.1 (DVDD)
Other:
- moved on the sheet: C53
Changed lines of the file:
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@@
 	(wire
 		(pts
-			(xy 167.64 100.33) (xy 170.18 100.33)
+			(xy 165.1 100.33) (xy 170.18 100.33)
 		)
 		(stroke
@@
 	(wire
 		(pts
-			(xy 160.02 100.33) (xy 162.56 100.33)
+			(xy 157.48 100.33) (xy 160.02 100.33)
 		)
 		(stroke
@@
 		)
 	)
-	(text_box "Dual compability only one, ic should be used at one time"
+	(text_box "Dual compability only one ic should be used at one time"
 		(exclude_from_sim no)
 		(at 45.72 132.08 0)
@@
 		)
 	)
+	(label "COM-"
+		(at 224.79 87.63 180)
+		(fields_autoplaced yes)
+		(effects
+			(font
+				(size 0.5 0.5)
+			)
+			(justify right bottom)
+		)
+	)
+	(label "DVDD"
+		(at 168.91 100.33 180)
+		(fields_autoplaced yes)
+		(effects
+			(font
+				(size 0.508 0.508)
+			)
+			(justify right bottom)
+		)
+	)
+	(label "COM+"
+		(at 224.79 85.09 180)
+		(fields_autoplaced yes)
+		(effects
+			(font
+				(size 0.5 0.5)
+			)
+			(justify right bottom)
+		)
+	)
 	(hierarchical_label "SPI_RDY"
 		(shape output)
@@
 		(lib_name "GND_17")
 		(lib_id "power:GND")
-		(at 160.02 100.33 270)
+		(at 157.48 100.33 270)
 		(unit 1)
 		(exclude_from_sim no)
@@
 		(dnp no)
 		(property "Reference" "#PWR0158"
-			(at 153.67 100.33 0)
+			(at 151.13 100.33 0)
 			(effects
 				(font
@@
 		)
 		(property "Value" "GNDISO"
-			(at 156.21 100.33 90)
+			(at 153.67 100.33 90)
 			(effects
 				(font
@@
 		)
 		(property "Footprint" ""
-			(at 160.02 100.33 0)
+			(at 157.48 100.33 0)
 			(effects
 				(font
@@
 		)
 		(property "Datasheet" ""
-			(at 160.02 100.33 0)
+			(at 157.48 100.33 0)
 			(effects
 				(font
@@
 		)
 		(property "Description" ""
-			(at 160.02 100.33 0)
+			(at 157.48 100.33 0)
 			(effects
 				(font
@@
 	(symbol
 		(lib_id "Device:C_Small")
-		(at 165.1 100.33 270)
+		(at 162.56 100.33 270)
 		(mirror x)
 		(unit 1)
@@
 		(dnp no)
 		(property "Reference" "C53"
-			(at 165.1 104.14 90)
+			(at 162.56 104.14 90)
 			(effects
 				(font
@@
 		)
 		(property "Value" "100nF"
-			(at 165.1 106.68 90)
+			(at 162.56 106.68 90)
 			(effects
 				(font
@@
 		)
 		(property "Footprint" "Capacitor_SMD:C_0603_1608Metric"
-			(at 165.1 100.33 0)
+			(at 162.56 100.33 0)
 			(effects
 				(font
@@
 		)
 		(property "Datasheet" "~"
-			(at 165.1 100.33 0)
+			(at 162.56 100.33 0)
 			(effects
 				(font
@@
 		)
 		(property "Description" ""
-			(at 165.1 100.33 0)
+			(at 162.56 100.33 0)
 			(effects
 				(font
@@
 		)
 		(property "Manufacturer_Name" "--"
-			(at 165.1 100.33 0)
+			(at 162.56 100.33 0)
 			(effects
 				(font
@@
 		)
 		(property "Manufacturer_Part_Number" "--"
-			(at 165.1 100.33 0)
+			(at 162.56 100.33 0)
 			(effects
 				(font
@@
 		)
 		(property "Arrow Part Number" ""
-			(at 165.1 100.33 0)
+			(at 162.56 100.33 0)
 			(effects
 				(font
@@
 		)
 		(property "Arrow Price/Stock" ""
-			(at 165.1 100.33 0)
+			(at 162.56 100.33 0)
 			(effects
 				(font
@@
 		)
 		(property "Mouser Price/Stock" "https://www.mouser.pl/ProductDetail/KEMET/C0603C104J3RACTU?qs=EHsFn6hSx4W0Oy0I8JUofQ%3D%3D"
-			(at 165.1 100.33 0)
+			(at 162.56 100.33 0)
 			(effects
 				(font

Commit message: bom update
Parts:
- C18, C42, C53, C78, R16, R19, R20, R95, R97, R99: Mouser Part Number (none) -> --
- C43: Mouser Part Number (none) -> 963-H168SC7224KTCA1J
- C79, C80: Mouser Part Number (none) -> 581-06035A101K
- IC6: Mouser Part Number LTC6820IMS#PBF -> 584-LTC6820IMS#PBF
- R94: Mouser Part Number (none) -> --; Mouser Price/Stock https://www.mouser.pl/ProductDetail/YAGEO/RT0603DRE07100KL?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 -> (none)
- R96, R98: Mouser Part Number (none) -> 594-MCT06030C5109FP5
Changed lines of the file:
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@@
+			)
+		)
+		(property "Mouser Part Number" "--"
+			(at 73.66 68.58 0)
+			(effects
+				(font
+					(size 1.27 1.27)
+				)
+				(hide yes)
 			)
 		)
@@
 			)
 		)
-		(property "Mouser Part Number" "LTC6820IMS#PBF"
+		(property "Mouser Part Number" "584-LTC6820IMS#PBF"
 			(at 92.71 82.55 0)
 			(effects
@@
 			)
 		)
+		(property "Mouser Part Number" "581-06035A101K"
+			(at 208.28 92.71 0)
+			(effects
+				(font
+					(size 1.27 1.27)
+				)
+				(hide yes)
+			)
+		)
 		(pin "1"
 		)
@@
 			)
 		)
+		(property "Mouser Part Number" "--"
+			(at 200.66 82.55 0)
+			(effects
+				(font
+					(size 1.27 1.27)
+				)
+				(hide yes)
+			)
+		)
 		(pin "1"
 		)
@@
 			)
 		)
+		(property "Mouser Part Number" "963-H168SC7224KTCA1J"
+			(at 200.66 64.77 0)
+			(effects
+				(font
+					(size 1.27 1.27)
+				)
+				(hide yes)
+			)
+		)
 		(pin "1"
 		)
@@
 		)
 		(property "Mouser Price/Stock" "https://www.mouser.pl/ProductDetail/YAGEO/RT0603DRE07100KL?qs=sGAEpiMZZMvdGkrng054t1nmr2c61WvadC66rbrHowc%3D"
+			(at 242.57 54.61 0)
+			(effects
+				(font
+					(size 1.27 1.27)
+				)
+				(hide yes)
+			)
+		)
+		(property "Mouser Part Number" "--"
 			(at 242.57 54.61 0)
 			(effects
@@
 			)
 		)
+		(property "Mouser Part Number" "--"
+			(at 73.66 63.5 0)
+			(effects
+				(font
+					(size 1.27 1.27)
+				)
+				(hide yes)
+			)
+		)
 		(pin "1"
 		)
@@
 		)
 		(property "Arrow Price/Stock" ""
+			(at 228.6 85.09 0)
+			(effects
+				(font
+					(size 1.27 1.27)
+				)
+				(hide yes)
+			)
+		)
+		(property "Mouser Part Number" "594-MCT06030C5109FP5"
 			(at 228.6 85.09 0)
 			(effects
@@
 			)
 		)
+		(property "Mouser Part Number" "--"
+			(at 233.68 54.61 0)
+			(effects
+				(font
+					(size 1.27 1.27)
+				)
+				(hide yes)
+			)
+		)
 		(pin "1"
 		)
@@
 			)
 		)
+		(property "Mouser Part Number" "581-06035A101K"
+			(at 218.44 92.71 0)
+			(effects
+				(font
+					(size 1.27 1.27)
+				)
+				(hide yes)
+			)
+		)
 		(pin "1"
 		)
@@
 			)
 		)
+		(property "Mouser Part Number" "--"
+			(at 162.56 64.77 0)
+			(effects
+				(font
+					(size 1.27 1.27)
+				)
+				(hide yes)
+			)
+		)
 		(pin "1"
 		)
@@
 			)
 		)
-		(property "Mouser Price/Stock" "https://www.mouser.pl/ProductDetail/YAGEO/RT0603DRE07100KL?qs=sGAEpiMZZMvdGkrng054t1nmr2c61WvadC66rbrHowc%3D"
+		(property "Mouser Price/Stock" ""
+			(at 250.19 54.61 0)
+			(effects
+				(font
+					(size 1.27 1.27)
+				)
+				(hide yes)
+			)
+		)
+		(property "Mouser Part Number" "--"
 			(at 250.19 54.61 0)
 			(effects
@@
 			)
 		)
+		(property "Mouser Part Number" "--"
+			(at 109.22 86.36 0)
+			(effects
+				(font
+					(size 1.27 1.27)
+				)
+				(hide yes)
+			)
+		)
 		(pin "1"
 		)
@@
 			)
 		)
+		(property "Mouser Part Number" "--"
+			(at 111.76 63.5 0)
+			(effects
+				(font
+					(size 1.27 1.27)
+				)
+				(hide yes)
+			)
+		)
 		(pin "1"
 		)
@@
 			)
 		)
+		(property "Mouser Part Number" "594-MCT06030C5109FP5"
+			(at 228.6 87.63 0)
+			(effects
+				(font
+					(size 1.27 1.27)
+				)
+				(hide yes)
+			)
+		)
 		(pin "1"
 		)
@@
 		)
 		(property "Arrow Price/Stock" ""
+			(at 113.03 93.98 0)
+			(effects
+				(font
+					(size 1.27 1.27)
+				)
+				(hide yes)
+			)
+		)
+		(property "Mouser Part Number" "--"
 			(at 113.03 93.98 0)
 			(effects
@@
 			(at 162.56 100.33 0)
 			(effects
+				(font
+					(size 1.27 1.27)
+				)
+				(hide yes)
+			)
+		)
+		(property "Mouser Part Number" "--"
+			(at 162.56 100.33 0)
+			(effects
