File: hardware/main board/Communication.kicad_sch (KiCad schematic)
At the start: 14 parts, among them U3 MCP2542FDxMF, U4 USBLC6-2SC6, U6 MCP2542FDxMF

Commit message: repairing demaged branch~
Parts:
- added FL1: DLW21SN501SK2L, Samacsys:DLW21SN121HQ2L, symbol dlw21sn501sk2l:DLW21SN501SK2L
- added R26, R36: 33, Resistor_SMD:R_0603_1608Metric, symbol Device:R_Small
- added U1: USBLC6-2SC6, Package_TO_SOT_SMD:SOT-23-6, symbol Power_Protection:USBLC6-2SC6
Connections:
- net GND: now also U1.2 (GND)
- net MCU_D+: now also U1.3 (I/O2)
- net MCU_D-: now also U1.1 (I/O1)
- new net: FL1.2, R36.1
- new net: FL1.3, R26.2
- new net: R26.1, U1.4 (I/O2)
- new net: R36.2, U1.6 (I/O1)
- new net EX_D+: FL1.4
- new net EX_D-: FL1.1
- new net EX_VBUS: U1.5 (VBUS)
Other:
- moved on the sheet: R49, R50, U4

Commit message: production version
Parts:
- C10, C21, C57, C60, R45, R67: Manufacturer_Name (none) -> --; Manufacturer_Part_Number (none) -> --
- O2: Manufacturer_Name (none) -> onsemi; Manufacturer_Part_Number (none) -> FOD8802DR2; Mouser Part Number (none) -> 863-FOD8802DR2; Mouser Price/Stock (none) -> https://www.mouser.pl/ProductDetail/onsemi/FOD8802DR2?qs=st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
- R26, R36, R49, R50: value 33 -> 33R; Manufacturer_Name (none) -> --; Manufacturer_Part_Number (none) -> --
- R40, R44: value 3.3k -> 2.7k; Manufacturer_Name (none) -> --; Manufacturer_Part_Number (none) -> --
- U1, U4: Manufacturer_Part_Number (none) -> USBLC6-2SC6; Mouser Part Number (none) -> 511-USBLC6-2SC6; Mouser Price/Stock (none) -> https://www.mouser.pl/ProductDetail/STMicroelectronics/USBL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
- U3, U6: Manufacturer_Part_Number (none) -> MCP2542FDT-H/MNY; Mouser Part Number (none) -> 579-MCP2542FDT-H/MNY; Mouser Price/Stock (none) -> https://www.mouser.pl/ProductDetail/Microchip-Technology/MC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
Changed lines of the file:
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@@
+      (effects (font (size 1.27 1.27)) hide)
+    )
+    (property "Manufacturer_Name" "onsemi" (at 166.37 129.54 0)
+      (effects (font (size 1.27 1.27)) hide)
+    )
+    (property "Manufacturer_Part_Number" "FOD8802DR2" (at 166.37 129.54 0)
+      (effects (font (size 1.27 1.27)) hide)
+    )
+    (property "Mouser Part Number" "863-FOD8802DR2" (at 166.37 129.54 0)
+      (effects (font (size 1.27 1.27)) hide)
+    )
+    (property "Mouser Price/Stock" "https://www.mouser.pl/ProductDetail/onsemi/FOD8802DR2?qs=stqOd1AaK7%2FrKOyi9z09cg%3D%3D" (at 166.37 129.54 0)
       (effects (font (size 1.27 1.27)) hide)
     )
@@
       (effects (font (size 1.27 1.27)))
     )
-    (property "Value" "3.3k" (at 147.32 132.08 90)
+    (property "Value" "2.7k" (at 147.32 132.08 90)
       (effects (font (size 1.27 1.27)))
     )
@@
     )
     (property "Datasheet" "~" (at 151.13 134.62 0)
+      (effects (font (size 1.27 1.27)) hide)
+    )
+    (property "Manufacturer_Name" "--" (at 151.13 134.62 0)
+      (effects (font (size 1.27 1.27)) hide)
+    )
+    (property "Manufacturer_Part_Number" "--" (at 151.13 134.62 0)
       (effects (font (size 1.27 1.27)) hide)
     )
@@
     )
     (property "Datasheet" "http://ww1.microchip.com/downloads/en/DeviceDoc/MCP2542FD-4FD-MCP2542WFD-4WFD-Data-Sheet20005514B.pdf" (at 237.49 57.15 0)
+      (effects (font (size 1.27 1.27)) hide)
+    )
+    (property "Manufacturer_Part_Number" "MCP2542FDT-H/MNY" (at 237.49 57.15 0)
+      (effects (font (size 1.27 1.27)) hide)
+    )
+    (property "Mouser Part Number" "579-MCP2542FDT-H/MNY" (at 237.49 57.15 0)
+      (effects (font (size 1.27 1.27)) hide)
+    )
+    (property "Mouser Price/Stock" "https://www.mouser.pl/ProductDetail/Microchip-Technology/MCP2542FDT-H-MNY?qs=qdgZG5p0FZ5ii0%252BaLco0zA%3D%3D" (at 237.49 57.15 0)
       (effects (font (size 1.27 1.27)) hide)
     )
@@
       (effects (font (size 1.27 1.27)) hide)
     )
+    (property "Manufacturer_Part_Number" "MCP2542FDT-H/MNY" (at 165.1 55.88 0)
+      (effects (font (size 1.27 1.27)) hide)
+    )
+    (property "Mouser Part Number" "579-MCP2542FDT-H/MNY" (at 165.1 55.88 0)
+      (effects (font (size 1.27 1.27)) hide)
+    )
+    (property "Mouser Price/Stock" "https://www.mouser.pl/ProductDetail/Microchip-Technology/MCP2542FDT-H-MNY?qs=qdgZG5p0FZ5ii0%252BaLco0zA%3D%3D" (at 165.1 55.88 0)
+      (effects (font (size 1.27 1.27)) hide)
+    )
     (pin "1")
     (pin "2")
@@
       (effects (font (size 1.27 1.27)) (justify right))
     )
-    (property "Value" "33" (at 29.337 147.5486 0)
+    (property "Value" "33R" (at 29.337 147.5486 0)
       (effects (font (size 1.27 1.27)) (justify right))
     )
@@
       (effects (font (size 1.27 1.27)) hide)
     )
+    (property "Manufacturer_Name" "--" (at 30.48 146.05 0)
+      (effects (font (size 1.27 1.27)) hide)
+    )
+    (property "Manufacturer_Part_Number" "--" (at 30.48 146.05 0)
+      (effects (font (size 1.27 1.27)) hide)
+    )
     (pin "1")
     (pin "2")
@@
     )
     (property "Datasheet" "https://www.st.com/resource/en/datasheet/usblc6-2.pdf" (at 62.23 171.45 0)
+      (effects (font (size 1.27 1.27)) hide)
+    )
+    (property "Manufacturer_Part_Number" "USBLC6-2SC6" (at 71.12 176.53 0)
+      (effects (font (size 1.27 1.27)) hide)
+    )
+    (property "Mouser Part Number" "511-USBLC6-2SC6" (at 71.12 176.53 0)
+      (effects (font (size 1.27 1.27)) hide)
+    )
+    (property "Mouser Price/Stock" "https://www.mouser.pl/ProductDetail/STMicroelectronics/USBLC6-2SC6?qs=po45yt2pPpu%2FhNIlwQdTlg%3D%3D" (at 71.12 176.53 0)
       (effects (font (size 1.27 1.27)) hide)
     )
@@
       (effects (font (size 1.27 1.27)) (justify right))
     )
-    (property "Value" "33" (at 62.357 190.7286 0)
+    (property "Value" "33R" (at 62.357 190.7286 0)
       (effects (font (size 1.27 1.27)) (justify right))
     )
@@
       (effects (font (size 1.27 1.27)) hide)
     )
+    (property "Manufacturer_Name" "--" (at 63.5 189.23 0)
+      (effects (font (size 1.27 1.27)) hide)
+    )
+    (property "Manufacturer_Part_Number" "--" (at 63.5 189.23 0)
+      (effects (font (size 1.27 1.27)) hide)
+    )
     (pin "1")
     (pin "2")
@@
     )
     (property "Datasheet" "~" (at 182.88 153.67 0)
+      (effects (font (size 1.27 1.27)) hide)
+    )
+    (property "Manufacturer_Name" "--" (at 182.88 153.67 0)
+      (effects (font (size 1.27 1.27)) hide)
+    )
+    (property "Manufacturer_Part_Number" "--" (at 182.88 153.67 0)
       (effects (font (size 1.27 1.27)) hide)
     )
@@
       (effects (font (size 1.27 1.27)) hide)
     )
+    (property "Manufacturer_Name" "--" (at 229.87 44.45 0)
+      (effects (font (size 1.27 1.27)) hide)
+    )
+    (property "Manufacturer_Part_Number" "--" (at 229.87 44.45 0)
+      (effects (font (size 1.27 1.27)) hide)
+    )
     (pin "1")
     (pin "2")
@@
       (effects (font (size 1.27 1.27)) hide)
     )
+    (property "Manufacturer_Name" "--" (at 175.26 153.67 0)
+      (effects (font (size 1.27 1.27)) hide)
+    )
+    (property "Manufacturer_Part_Number" "--" (at 175.26 153.67 0)
+      (effects (font (size 1.27 1.27)) hide)
+    )
     (pin "1")
     (pin "2")
@@
       (effects (font (size 1.27 1.27)) (justify right))
     )
-    (property "Value" "33" (at 31.623 119.1514 0)
+    (property "Value" "33R" (at 31.623 119.1514 0)
       (effects (font (size 1.27 1.27)) (justify right))
     )
@@
       (effects (font (size 1.27 1.27)) hide)
     )
+    (property "Manufacturer_Name" "--" (at 30.48 120.65 0)
+      (effects (font (size 1.27 1.27)) hide)
+    )
+    (property "Manufacturer_Part_Number" "--" (at 30.48 120.65 0)
+      (effects (font (size 1.27 1.27)) hide)
+    )
     (pin "1")
     (pin "2")
@@
       (effects (font (size 1.27 1.27)) hide)
     )
+    (property "Manufacturer_Name" "--" (at 170.18 43.18 0)
+      (effects (font (size 1.27 1.27)) hide)
+    )
+    (property "Manufacturer_Part_Number" "--" (at 170.18 43.18 0)
+      (effects (font (size 1.27 1.27)) hide)
+    )
     (pin "1")
     (pin "2")
@@
       (effects (font (size 1.27 1.27)))
     )
-    (property "Value" "3.3k" (at 147.32 140.97 90)
+    (property "Value" "2.7k" (at 147.32 140.97 90)
       (effects (font (size 1.27 1.27)))
     )
@@
     )
     (property "Datasheet" "~" (at 151.13 143.51 0)
+      (effects (font (size 1.27 1.27)) hide)
+    )
+    (property "Manufacturer_Name" "--" (at 151.13 143.51 0)
+      (effects (font (size 1.27 1.27)) hide)
+    )
+    (property "Manufacturer_Part_Number" "--" (at 151.13 143.51 0)
       (effects (font (size 1.27 1.27)) hide)
     )
@@
     )
     (property "Datasheet" "https://www.st.com/resource/en/datasheet/usblc6-2.pdf" (at 29.21 128.27 0)
+      (effects (font (size 1.27 1.27)) hide)
+    )
+    (property "Manufacturer_Part_Number" "USBLC6-2SC6" (at 38.1 133.35 0)
+      (effects (font (size 1.27 1.27)) hide)
+    )
+    (property "Mouser Part Number" "511-USBLC6-2SC6" (at 38.1 133.35 0)
+      (effects (font (size 1.27 1.27)) hide)
+    )
+    (property "Mouser Price/Stock" "https://www.mouser.pl/ProductDetail/STMicroelectronics/USBLC6-2SC6?qs=po45yt2pPpu%2FhNIlwQdTlg%3D%3D" (at 38.1 133.35 0)
       (effects (font (size 1.27 1.27)) hide)
     )
@@
       (effects (font (size 1.27 1.27)) hide)
     )
+    (property "Manufacturer_Name" "--" (at 242.57 44.45 0)
+      (effects (font (size 1.27 1.27)) hide)
+    )
+    (property "Manufacturer_Part_Number" "--" (at 242.57 44.45 0)
+      (effects (font (size 1.27 1.27)) hide)
+    )
     (pin "1")
     (pin "2")
@@
       (effects (font (size 1.27 1.27)) hide)
     )
+    (property "Manufacturer_Name" "--" (at 157.48 43.18 0)
+      (effects (font (size 1.27 1.27)) hide)
+    )
+    (property "Manufacturer_Part_Number" "--" (at 157.48 43.18 0)
+      (effects (font (size 1.27 1.27)) hide)
+    )
     (pin "1")
     (pin "2")
@@
       (effects (font (size 1.27 1.27)) (justify right))
     )
-    (property "Value" "33" (at 64.643 162.3314 0)
+    (property "Value" "33R" (at 64.643 162.3314 0)
       (effects (font (size 1.27 1.27)) (justify right))
     )
@@
       (effects (font (size 1.27 1.27)) hide)
     )
+    (property "Manufacturer_Name" "--" (at 63.5 163.83 0)
+      (effects (font (size 1.27 1.27)) hide)
+    )
+    (property "Manufacturer_Part_Number" "--" (at 63.5 163.83 0)
+      (effects (font (size 1.27 1.27)) hide)
+    )
