File: hardware/main board/Fan_drivers.kicad_sch (KiCad schematic)
At the start: 28 parts, among them Q1 2SK3065, Q12 2SK3065, Q13 2SK3065, Q14 2SK3065, Q15 2SK3065, Q7 2SK3065, Q9 2SK3065

Commit message: production version
Parts:
- D14, D15, D16, D17, D18, D19, D20: Manufacturer_Part_Number (none) -> CDBU0530; Mouser Part Number (none) -> 750-CDBU0530; Mouser Price/Stock (none) -> https://www.mouser.pl/ProductDetail/Comchip-Technology/CDBU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
- Q1, Q12, Q13, Q14, Q15, Q7, Q9: Manufacturer_Part_Number (none) -> 2SK3065T100; Mouser Part Number (none) -> 755-2SK3065T100; Mouser Price/Stock (none) -> https://www.mouser.pl/ProductDetail/ROHM-Semiconductor/2SK3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
- R30: value 10K -> 10k; Manufacturer_Name (none) -> --; Manufacturer_Part_Number (none) -> --
- R30: value 100 -> 100R; Manufacturer_Name (none) -> --; Manufacturer_Part_Number (none) -> --
