File: hardware/main board/HP_NMOS_PullDown.kicad_sch (KiCad schematic)
At the start: 4 parts, among them Q5 Q_NMOS_GDS

Commit message: production version
Parts:
- D12: value D_Small -> 4A/80V; Manufacturer_Part_Number (none) -> VSSB410S-E3/52T; Mouser Part Number (none) -> 625-VSSB410S-E3/52T; Mouser Price/Stock (none) -> https://www.mouser.pl/ProductDetail/Vishay-General-Semicond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
- Q5: value Q_NMOS_GDS -> STN4NF06L; Manufacturer_Part_Number (none) -> IRLL024ZTRPBF; Mouser Part Number (none) -> 942-IRLL024ZTRPBF; Mouser Price/Stock (none) -> https://www.mouser.pl/ProductDetail/Infineon-Technologies/I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; Url https://www.mouser.pl/ProductDetail/Infineon-Technologies/I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 -> (none)
- R30: value 100 -> 100R; Manufacturer_Name (none) -> --; Manufacturer_Part_Number (none) -> --
- R39: Manufacturer_Name (none) -> --; Manufacturer_Part_Number (none) -> --
Changed lines of the file:
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@@
+      (effects (font (size 1.27 1.27)) hide)
+    )
+    (property "Manufacturer_Name" "--" (at 134.62 92.71 0)
+      (effects (font (size 1.27 1.27)) hide)
+    )
+    (property "Manufacturer_Part_Number" "--" (at 134.62 92.71 0)
       (effects (font (size 1.27 1.27)) hide)
     )
@@
       (effects (font (size 1.27 1.27)))
     )
-    (property "Value" "100" (at 129.54 84.455 90)
+    (property "Value" "100R" (at 129.54 84.455 90)
       (effects (font (size 1.27 1.27)))
     )
@@
     )
     (property "Datasheet" "~" (at 129.54 87.63 0)
+      (effects (font (size 1.27 1.27)) hide)
+    )
+    (property "Manufacturer_Name" "--" (at 129.54 87.63 0)
+      (effects (font (size 1.27 1.27)) hide)
+    )
+    (property "Manufacturer_Part_Number" "--" (at 129.54 87.63 0)
       (effects (font (size 1.27 1.27)) hide)
     )
@@
   (symbol (lib_id "Device:Q_NMOS_GDS") (at 142.24 87.63 0) (unit 1)
     (in_bom yes) (on_board yes) (dnp no) (fields_autoplaced)
-    (property "Reference" "Q5" (at 147.955 86.3599 0)
+    (property "Reference" "Q5" (at 148.59 86.36 0)
       (effects (font (size 1.27 1.27)) (justify left))
     )
-    (property "Value" "Q_NMOS_GDS" (at 147.955 88.8999 0)
+    (property "Value" "STN4NF06L" (at 148.59 88.9 0)
       (effects (font (size 1.27 1.27)) (justify left))
     )
@@
       (effects (font (size 1.27 1.27)) hide)
     )
-    (property "Url" "https://www.mouser.pl/ProductDetail/Infineon-Technologies/IRLL024ZTRPBF?qs=9%252BKlkBgLFf1b4odHOQZ9nw%3D%3D" (at 142.24 87.63 0)
+    (property "Url" "" (at 142.24 87.63 0)
+      (effects (font (size 1.27 1.27)) hide)
+    )
+    (property "Manufacturer_Part_Number" "IRLL024ZTRPBF" (at 142.24 87.63 0)
+      (effects (font (size 1.27 1.27)) hide)
+    )
+    (property "Mouser Part Number" "942-IRLL024ZTRPBF" (at 142.24 87.63 0)
+      (effects (font (size 1.27 1.27)) hide)
+    )
+    (property "Mouser Price/Stock" "https://www.mouser.pl/ProductDetail/Infineon-Technologies/IRLL024ZTRPBF?qs=9%252BKlkBgLFf1b4odHOQZ9nw%3D%3D" (at 142.24 87.63 0)
       (effects (font (size 1.27 1.27)) hide)
     )
@@
       (effects (font (size 1.27 1.27)) (justify left))
     )
-    (property "Value" "D_Small" (at 146.685 76.1999 90)
+    (property "Value" "4A/80V" (at 146.685 76.1999 90)
       (effects (font (size 1.27 1.27)) (justify left))
     )
@@
       (effects (font (size 1.27 1.27)) hide)
     )
+    (property "Manufacturer_Part_Number" "VSSB410S-E3/52T" (at 144.78 74.93 0)
+      (effects (font (size 1.27 1.27)) hide)
+    )
+    (property "Mouser Part Number" "625-VSSB410S-E3/52T" (at 144.78 74.93 0)
+      (effects (font (size 1.27 1.27)) hide)
+    )
+    (property "Mouser Price/Stock" "https://www.mouser.pl/ProductDetail/Vishay-General-Semiconductor/VSSB410S-E3-52T?qs=HSPD0Bff7ib64J9oD9YilA%3D%3D" (at 144.78 74.93 0)
+      (effects (font (size 1.27 1.27)) hide)
+    )
