File: hardware/main board/IsolatedCommunication.kicad_sch (KiCad schematic)
At the start: 4 parts, among them U12 LTC6820IMS

Commit message: production version
Parts:
- C34: Manufacturer_Name (none) -> --; Manufacturer_Part_Number (none) -> --
- R57, R62: value 1K -> 1k; Manufacturer_Name (none) -> --; Manufacturer_Part_Number (none) -> --
- U12: Manufacturer_Part_Number (none) -> LTC6820IMS#TRPBF; Mouser Part Number (none) -> 584-LTC6820IMS#TRPBF; Mouser Price/Stock (none) -> https://www.mouser.pl/ProductDetail/Analog-Devices/LTC6820I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
Changed lines of the file:
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@@
+      (effects (font (size 1.27 1.27)) hide)
+    )
+    (property "Manufacturer_Part_Number" "LTC6820IMS#TRPBF" (at 131.445 89.535 0)
+      (effects (font (size 1.27 1.27)) hide)
+    )
+    (property "Mouser Part Number" "584-LTC6820IMS#TRPBF" (at 131.445 89.535 0)
+      (effects (font (size 1.27 1.27)) hide)
+    )
+    (property "Mouser Price/Stock" "https://www.mouser.pl/ProductDetail/Analog-Devices/LTC6820IMSTRPBF?qs=hVkxg5c3xu8J%252BEL4cIWawA%3D%3D" (at 131.445 89.535 0)
       (effects (font (size 1.27 1.27)) hide)
     )
@@
       (effects (font (size 1.27 1.27)) (justify right))
     )
-    (property "Value" "1K" (at 155.575 81.28 90)
+    (property "Value" "1k" (at 155.575 81.28 90)
       (effects (font (size 1.27 1.27)) (justify right))
     )
@@
     )
     (property "Datasheet" "~" (at 154.305 83.185 0)
+      (effects (font (size 1.27 1.27)) hide)
+    )
+    (property "Manufacturer_Name" "--" (at 154.305 83.185 0)
+      (effects (font (size 1.27 1.27)) hide)
+    )
+    (property "Manufacturer_Part_Number" "--" (at 154.305 83.185 0)
       (effects (font (size 1.27 1.27)) hide)
     )
@@
       (effects (font (size 1.27 1.27)))
     )
-    (property "Value" "1K" (at 146.685 78.74 90)
+    (property "Value" "1k" (at 146.685 78.74 90)
       (effects (font (size 1.27 1.27)))
     )
@@
     )
     (property "Datasheet" "~" (at 146.685 80.645 0)
+      (effects (font (size 1.27 1.27)) hide)
+    )
+    (property "Manufacturer_Name" "--" (at 146.685 80.645 0)
+      (effects (font (size 1.27 1.27)) hide)
+    )
+    (property "Manufacturer_Part_Number" "--" (at 146.685 80.645 0)
       (effects (font (size 1.27 1.27)) hide)
     )
@@
       (effects (font (size 1.27 1.27)) hide)
     )
+    (property "Manufacturer_Name" "--" (at 142.875 102.87 0)
+      (effects (font (size 1.27 1.27)) hide)
+    )
+    (property "Manufacturer_Part_Number" "--" (at 142.875 102.87 0)
+      (effects (font (size 1.27 1.27)) hide)
+    )
