File: hardware/main board/IsolatedMeasurement.kicad_sch (KiCad schematic)
At the start: 23 parts, among them IC12 UCC12040DVE, IC15 ISO6763FDWR, IC2 MCP3561T-E_NC, IC6 AP7365-33YRG-13, IC9 REF193GSZ-REEL, Q11 Q_NMOS_GSD

Commit message: repairing demaged branch~
Parts:
- RD2: Mouser Url (none) -> https://www.mouser.pl/ProductDetail/Vishay-Techno/CDMM20M0F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
Other:
- note added: "CDMM20M0F2500"
- note removed: "REF"
- note removed: "V_{mes_max} = 3V V_{in_max} = 600V A = 3 / 600 = 1 / 200 1 / 200 = R_{2} / R_{1} + R_{2} R_{1} = 199 R_{2}"
- moved on the sheet: C20, C9, FB1, IC9, L11

Commit message: production version
Parts:
- C13, C17, C18, C20, C36, C37, C38, C39: Manufacturer_Name (none) -> --; Manufacturer_Part_Number (none) -> --
- C7, C9: value 100nF -> 10uF; Manufacturer_Name (none) -> --; Manufacturer_Part_Number (none) -> --
- FB1: value ferrite_baud -> GZ1608D601TF; Manufacturer_Part_Number (none) -> --
- L11: value 6.8uH -> 1mH; Manufacturer_Part_Number (none) -> LB3218T102K; Mouser Part Number (none) -> 963-LB3218T102K; Mouser Price/Stock (none) -> https://www.mouser.pl/ProductDetail/TAIYO-YUDEN/LB3218T102K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
- L11: value 6.8uH -> 4.7uH; Manufacturer_Part_Number (none) -> LQM31PN4R7M00L; Mouser Part Number (none) -> 81-LQM31PN4R7M00L; Mouser Price/Stock (none) -> https://www.mouser.pl/ProductDetail/Murata-Electronics/LQM3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
- Q11: value Q_NMOS_GSD -> 2N7002; Manufacturer_Name (none) -> --; Manufacturer_Part_Number (none) -> --
- R23: value R -> 200R; Manufacturer_Name (none) -> --; Manufacturer_Part_Number (none) -> --
- RD2: value ~ -> CDMM20M0F2500; Manufacturer_Part_Number (none) -> CDMM20M0F2500DET; Mouser Part Number (none) -> 71-CDMM20M0F2500DET; Mouser Price/Stock (none) -> https://www.mouser.pl/ProductDetail/Vishay-Techno/CDMM20M0F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
Changed lines of the file:
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@@
       (effects (font (size 1.27 1.27)) (justify left))
     )
-    (property "Value" "100nF" (at 207.01 151.13 0)
+    (property "Value" "10uF" (at 207.01 151.13 0)
       (effects (font (size 1.27 1.27)) (justify left))
     )
@@
     )
     (property "Datasheet" "~" (at 214.63 149.86 0)
+      (effects (font (size 1.27 1.27)) hide)
+    )
+    (property "Manufacturer_Name" "--" (at 214.63 149.86 0)
+      (effects (font (size 1.27 1.27)) hide)
+    )
+    (property "Manufacturer_Part_Number" "--" (at 214.63 149.86 0)
       (effects (font (size 1.27 1.27)) hide)
     )
@@
       (effects (font (size 1.27 1.27)) (justify bottom))
     )
-    (property "Value" "6.8uH" (at 204.47 62.23 90)
+    (property "Value" "1mH" (at 204.47 62.23 90)
       (effects (font (size 1.27 1.27)) (justify bottom))
     )
@@
     )
     (property "Datasheet" "~" (at 204.47 58.42 0)
+      (effects (font (size 1.27 1.27)) hide)
+    )
+    (property "Manufacturer_Part_Number" "LB3218T102K" (at 204.47 58.42 0)
+      (effects (font (size 1.27 1.27)) hide)
+    )
+    (property "Mouser Part Number" "963-LB3218T102K" (at 204.47 58.42 0)
+      (effects (font (size 1.27 1.27)) hide)
+    )
+    (property "Mouser Price/Stock" "https://www.mouser.pl/ProductDetail/TAIYO-YUDEN/LB3218T102K?qs=I6KAKw0tg2xz0leHHx%252BE%252BA%3D%3D" (at 204.47 58.42 0)
       (effects (font (size 1.27 1.27)) hide)
     )
@@
       (effects (font (size 1.27 1.27)) hide)
     )
+    (property "Manufacturer_Name" "--" (at 110.49 63.5 0)
+      (effects (font (size 1.27 1.27)) hide)
+    )
+    (property "Manufacturer_Part_Number" "--" (at 110.49 63.5 0)
+      (effects (font (size 1.27 1.27)) hide)
+    )
     (pin "1")
     (pin "2")
@@
   )
   (symbol (lib_id "CDMM:CDMM2M50D4000DET") (at 165.1 127 0) (unit 1)
-    (in_bom yes) (on_board yes) (dnp no) (fields_autoplaced)
-    (property "Reference" "RD2" (at 165.1 120.65 0)
-      (effects (font (size 1.27 1.27)))
-    )
-    (property "Value" "~" (at 167.005 124.46 0)
+    (in_bom yes) (on_board yes) (dnp no)
+    (property "Reference" "RD2" (at 165.1 118.11 0)
+      (effects (font (size 1.27 1.27)))
+    )
+    (property "Value" "CDMM20M0F2500" (at 165.1 120.65 0)
       (effects (font (size 1.27 1.27)))
     )
@@
     )
     (property "Mouser Url" "https://www.mouser.pl/ProductDetail/Vishay-Techno/CDMM20M0F2500DET?qs=pUKx8fyJudDtrYAwlAh%252BkQ%3D%3D" (at 165.1 127 0)
+      (effects (font (size 1.27 1.27)) hide)
+    )
+    (property "Manufacturer_Part_Number" "CDMM20M0F2500DET" (at 165.1 127 0)
+      (effects (font (size 1.27 1.27)) hide)
+    )
+    (property "Mouser Part Number" "71-CDMM20M0F2500DET" (at 165.1 127 0)
+      (effects (font (size 1.27 1.27)) hide)
+    )
+    (property "Mouser Price/Stock" "https://www.mouser.pl/ProductDetail/Vishay-Techno/CDMM20M0F2500DET?qs=pUKx8fyJudDtrYAwlAh%252BkQ%3D%3D" (at 165.1 127 0)
       (effects (font (size 1.27 1.27)) hide)
     )
@@
       (effects (font (size 1.27 1.27)) (justify left))
     )
-    (property "Value" "Q_NMOS_GSD" (at 26.67 149.225 0)
+    (property "Value" "2N7002" (at 26.67 149.225 0)
       (effects (font (size 1.27 1.27)) (justify left))
     )
@@
       (effects (font (size 1.27 1.27)) hide)
     )
+    (property "Manufacturer_Name" "--" (at 33.02 147.32 0)
+      (effects (font (size 1.27 1.27)) hide)
+    )
+    (property "Manufacturer_Part_Number" "--" (at 33.02 147.32 0)
+      (effects (font (size 1.27 1.27)) hide)
+    )
     (pin "1")
     (pin "2")
@@
       (effects (font (size 1.27 1.27)) hide)
     )
+    (property "Manufacturer_Name" "--" (at 50.8 68.58 0)
+      (effects (font (size 1.27 1.27)) hide)
+    )
+    (property "Manufacturer_Part_Number" "--" (at 50.8 68.58 0)
+      (effects (font (size 1.27 1.27)) hide)
+    )
     (pin "1")
     (pin "2")
@@
       (effects (font (size 1.27 1.27)))
     )
-    (property "Value" "ferrite_baud" (at 207.645 52.705 90)
+    (property "Value" "GZ1608D601TF" (at 207.645 52.705 90)
       (effects (font (size 1.27 1.27)) hide)
     )
@@
     )
     (property "Datasheet" "~" (at 212.09 58.42 0)
+      (effects (font (size 1.27 1.27)) hide)
+    )
+    (property "Manufacturer_Part_Number" "--" (at 212.09 58.42 0)
       (effects (font (size 1.27 1.27)) hide)
     )
@@
       (effects (font (size 1.27 1.27)) hide)
     )
+    (property "Manufacturer_Name" "--" (at 251.46 149.86 0)
+      (effects (font (size 1.27 1.27)) hide)
+    )
+    (property "Manufacturer_Part_Number" "--" (at 251.46 149.86 0)
+      (effects (font (size 1.27 1.27)) hide)
+    )
     (pin "1")
     (pin "2")
@@
     )
     (property "Datasheet" "~" (at 57.15 162.56 0)
+      (effects (font (size 1.27 1.27)) hide)
+    )
+    (property "Manufacturer_Name" "--" (at 57.15 162.56 0)
+      (effects (font (size 1.27 1.27)) hide)
+    )
+    (property "Manufacturer_Part_Number" "--" (at 57.15 162.56 0)
       (effects (font (size 1.27 1.27)) hide)
     )
@@
       (effects (font (size 1.27 1.27)) (justify right))
     )
-    (property "Value" "R" (at 130.048 64.643 0)
+    (property "Value" "200R" (at 130.048 64.643 0)
       (effects (font (size 1.27 1.27)) (justify right))
     )
@@
       (effects (font (size 1.27 1.27)) hide)
     )
+    (property "Manufacturer_Name" "--" (at 128.27 63.5 0)
+      (effects (font (size 1.27 1.27)) hide)
+    )
+    (property "Manufacturer_Part_Number" "--" (at 128.27 63.5 0)
+      (effects (font (size 1.27 1.27)) hide)
+    )
     (pin "1")
     (pin "2")
@@
       (effects (font (size 1.27 1.27)) hide)
     )
+    (property "Manufacturer_Name" "--" (at 119.38 63.5 0)
+      (effects (font (size 1.27 1.27)) hide)
+    )
+    (property "Manufacturer_Part_Number" "--" (at 119.38 63.5 0)
+      (effects (font (size 1.27 1.27)) hide)
+    )
     (pin "1")
     (pin "2")
@@
       (effects (font (size 1.27 1.27)) hide)
     )
+    (property "Manufacturer_Name" "--" (at 252.73 60.96 0)
+      (effects (font (size 1.27 1.27)) hide)
+    )
+    (property "Manufacturer_Part_Number" "--" (at 252.73 60.96 0)
+      (effects (font (size 1.27 1.27)) hide)
+    )
     (pin "1")
     (pin "2")
@@
     )
     (property "Datasheet" "~" (at 96.52 162.56 0)
+      (effects (font (size 1.27 1.27)) hide)
+    )
+    (property "Manufacturer_Name" "--" (at 96.52 162.56 0)
+      (effects (font (size 1.27 1.27)) hide)
+    )
+    (property "Manufacturer_Part_Number" "--" (at 96.52 162.56 0)
       (effects (font (size 1.27 1.27)) hide)
     )
@@
       (effects (font (size 1.27 1.27)))
     )
-    (property "Value" "ferrite_baud" (at 205.105 139.065 90)
+    (property "Value" "GZ1608D601TF" (at 205.105 139.065 90)
       (effects (font (size 1.27 1.27)) hide)
     )
@@
     )
     (property "Datasheet" "~" (at 209.55 144.78 0)
+      (effects (font (size 1.27 1.27)) hide)
+    )
+    (property "Manufacturer_Part_Number" "--" (at 209.55 144.78 0)
       (effects (font (size 1.27 1.27)) hide)
     )
@@
   (symbol (lib_id "Device:L_Small") (at 201.93 144.78 90) (unit 1)
     (in_bom yes) (on_board yes) (dnp no)
-    (property "Reference" "L11" (at 201.93 146.05 90)
+    (property "Reference" "L11" (at 198.12 146.05 90)
       (effects (font (size 1.27 1.27)) (justify bottom))
     )
-    (property "Value" "6.8uH" (at 201.93 149.86 90)
+    (property "Value" "1mH" (at 198.12 148.59 90)
       (effects (font (size 1.27 1.27)) (justify bottom))
     )
@@
     )
     (property "Datasheet" "~" (at 201.93 144.78 0)
+      (effects (font (size 1.27 1.27)) hide)
+    )
+    (property "Manufacturer_Part_Number" "LB3218T102K" (at 201.93 144.78 0)
+      (effects (font (size 1.27 1.27)) hide)
+    )
+    (property "Mouser Part Number" "963-LB3218T102K" (at 201.93 144.78 0)
+      (effects (font (size 1.27 1.27)) hide)
+    )
+    (property "Mouser Price/Stock" "https://www.mouser.pl/ProductDetail/TAIYO-YUDEN/LB3218T102K?qs=I6KAKw0tg2xz0leHHx%252BE%252BA%3D%3D" (at 201.93 144.78 0)
       (effects (font (size 1.27 1.27)) hide)
     )
@@
       (effects (font (size 1.27 1.27)) hide)
     )
+    (property "Manufacturer_Name" "--" (at 151.13 63.5 0)
+      (effects (font (size 1.27 1.27)) hide)
+    )
+    (property "Manufacturer_Part_Number" "--" (at 151.13 63.5 0)
+      (effects (font (size 1.27 1.27)) hide)
+    )
     (pin "1")
     (pin "2")
@@
       (effects (font (size 1.27 1.27)) (justify left))
     )
-    (property "Value" "100nF" (at 212.09 72.39 90)
+    (property "Value" "10uF" (at 212.09 72.39 90)
       (effects (font (size 1.27 1.27)) (justify left))
     )
@@
     )
     (property "Datasheet" "~" (at 217.17 68.58 0)
+      (effects (font (size 1.27 1.27)) hide)
+    )
+    (property "Manufacturer_Name" "--" (at 217.17 68.58 0)
+      (effects (font (size 1.27 1.27)) hide)
+    )
+    (property "Manufacturer_Part_Number" "--" (at 217.17 68.58 0)
       (effects (font (size 1.27 1.27)) hide)
     )
@@
       (effects (font (size 1.27 1.27)) (justify bottom))
     )
-    (property "Value" "6.8uH" (at 45.72 60.96 90)
+    (property "Value" "4.7uH" (at 45.72 60.96 90)
       (effects (font (size 1.27 1.27)) (justify bottom))
     )
@@
       (effects (font (size 1.27 1.27)) hide)
     )
+    (property "Manufacturer_Part_Number" "LQM31PN4R7M00L" (at 45.72 63.5 0)
+      (effects (font (size 1.27 1.27)) hide)
+    )
+    (property "Mouser Part Number" "81-LQM31PN4R7M00L" (at 45.72 63.5 0)
+      (effects (font (size 1.27 1.27)) hide)
+    )
+    (property "Mouser Price/Stock" "https://www.mouser.pl/ProductDetail/Murata-Electronics/LQM31PN4R7M00L?qs=%2F%252BYoplLUB5ijpQp630h8dg%3D%3D" (at 45.72 63.5 0)
+      (effects (font (size 1.27 1.27)) hide)
+    )
