File: hardware/main board/Measurements.kicad_sch (KiCad schematic)
At the start: 13 parts, among them IC1 MCP1501-10E_SN, IC7 MCP3562T-E_NC, IC9 REF193GSZ-REEL

Commit message: production version
Parts:
- C2, C20, C4, C5: Manufacturer_Name (none) -> --; Manufacturer_Part_Number (none) -> --
- C7, C9: value 100nF -> 10uF; Manufacturer_Name (none) -> --; Manufacturer_Part_Number (none) -> --
- FB1: value ferrite_baud -> GZ1608D601TF; Manufacturer_Part_Number (none) -> --
- L11: value 6.8uH -> 1mH; Manufacturer_Part_Number (none) -> LB3218T102K; Mouser Part Number (none) -> 963-LB3218T102K; Mouser Price/Stock (none) -> https://www.mouser.pl/ProductDetail/TAIYO-YUDEN/LB3218T102K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
Changed lines of the file:
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@@
       (effects (font (size 1.27 1.27)) (justify left))
     )
-    (property "Value" "100nF" (at 218.44 128.27 90)
+    (property "Value" "10uF" (at 218.44 128.27 90)
       (effects (font (size 1.27 1.27)) (justify left))
     )
@@
     )
     (property "Datasheet" "~" (at 223.52 124.46 0)
+      (effects (font (size 1.27 1.27)) hide)
+    )
+    (property "Manufacturer_Name" "--" (at 223.52 124.46 0)
+      (effects (font (size 1.27 1.27)) hide)
+    )
+    (property "Manufacturer_Part_Number" "--" (at 223.52 124.46 0)
       (effects (font (size 1.27 1.27)) hide)
     )
@@
       (effects (font (size 1.27 1.27)) (justify bottom))
     )
-    (property "Value" "6.8uH" (at 104.14 181.61 90)
+    (property "Value" "1mH" (at 99.06 181.61 90)
       (effects (font (size 1.27 1.27)) (justify bottom))
     )
@@
     )
     (property "Datasheet" "~" (at 104.14 176.53 0)
+      (effects (font (size 1.27 1.27)) hide)
+    )
+    (property "Manufacturer_Part_Number" "LB3218T102K" (at 104.14 176.53 0)
+      (effects (font (size 1.27 1.27)) hide)
+    )
+    (property "Mouser Part Number" "963-LB3218T102K" (at 104.14 176.53 0)
+      (effects (font (size 1.27 1.27)) hide)
+    )
+    (property "Mouser Price/Stock" "https://www.mouser.pl/ProductDetail/TAIYO-YUDEN/LB3218T102K?qs=I6KAKw0tg2xz0leHHx%252BE%252BA%3D%3D" (at 104.14 176.53 0)
       (effects (font (size 1.27 1.27)) hide)
     )
@@
       (effects (font (size 1.27 1.27)))
     )
-    (property "Value" "ferrite_baud" (at 213.995 108.585 90)
+    (property "Value" "GZ1608D601TF" (at 213.995 108.585 90)
       (effects (font (size 1.27 1.27)) hide)
     )
@@
     )
     (property "Datasheet" "~" (at 218.44 114.3 0)
+      (effects (font (size 1.27 1.27)) hide)
+    )
+    (property "Manufacturer_Part_Number" "--" (at 218.44 114.3 0)
       (effects (font (size 1.27 1.27)) hide)
     )
@@
       (effects (font (size 1.27 1.27)))
     )
-    (property "Value" "ferrite_baud" (at 107.315 170.815 90)
+    (property "Value" "GZ1608D601TF" (at 107.315 170.815 90)
       (effects (font (size 1.27 1.27)) hide)
     )
@@
     )
     (property "Datasheet" "~" (at 111.76 176.53 0)
+      (effects (font (size 1.27 1.27)) hide)
+    )
+    (property "Manufacturer_Part_Number" "--" (at 111.76 176.53 0)
       (effects (font (size 1.27 1.27)) hide)
     )
@@
       (effects (font (size 1.27 1.27)) hide)
     )
+    (property "Manufacturer_Name" "--" (at 154.94 181.61 0)
+      (effects (font (size 1.27 1.27)) hide)
+    )
+    (property "Manufacturer_Part_Number" "--" (at 154.94 181.61 0)
+      (effects (font (size 1.27 1.27)) hide)
+    )
     (pin "1")
     (pin "2")
@@
     )
     (property "Datasheet" "~" (at 259.08 116.84 0)
+      (effects (font (size 1.27 1.27)) hide)
+    )
+    (property "Manufacturer_Name" "--" (at 259.08 116.84 0)
+      (effects (font (size 1.27 1.27)) hide)
+    )
+    (property "Manufacturer_Part_Number" "--" (at 259.08 116.84 0)
       (effects (font (size 1.27 1.27)) hide)
     )
@@
       (effects (font (size 1.27 1.27)) hide)
     )
+    (property "Manufacturer_Name" "--" (at 246.38 78.74 0)
+      (effects (font (size 1.27 1.27)) hide)
+    )
+    (property "Manufacturer_Part_Number" "--" (at 246.38 78.74 0)
+      (effects (font (size 1.27 1.27)) hide)
+    )
     (pin "1")
     (pin "2")
@@
       (effects (font (size 1.27 1.27)) (justify bottom))
     )
-    (property "Value" "6.8uH" (at 210.82 118.11 90)
+    (property "Value" "1mH" (at 210.82 118.11 90)
       (effects (font (size 1.27 1.27)) (justify bottom))
     )
@@
     )
     (property "Datasheet" "~" (at 210.82 114.3 0)
+      (effects (font (size 1.27 1.27)) hide)
+    )
+    (property "Manufacturer_Part_Number" "LB3218T102K" (at 210.82 114.3 0)
+      (effects (font (size 1.27 1.27)) hide)
+    )
+    (property "Mouser Part Number" "963-LB3218T102K" (at 210.82 114.3 0)
+      (effects (font (size 1.27 1.27)) hide)
+    )
+    (property "Mouser Price/Stock" "https://www.mouser.pl/ProductDetail/TAIYO-YUDEN/LB3218T102K?qs=I6KAKw0tg2xz0leHHx%252BE%252BA%3D%3D" (at 210.82 114.3 0)
       (effects (font (size 1.27 1.27)) hide)
     )
@@
       (effects (font (size 1.27 1.27)) hide)
     )
+    (property "Manufacturer_Name" "--" (at 210.82 78.74 0)
+      (effects (font (size 1.27 1.27)) hide)
+    )
+    (property "Manufacturer_Part_Number" "--" (at 210.82 78.74 0)
+      (effects (font (size 1.27 1.27)) hide)
+    )
     (pin "1")
     (pin "2")
@@
       (effects (font (size 1.27 1.27)) (justify left))
     )
-    (property "Value" "100nF" (at 109.22 182.88 0)
+    (property "Value" "10uF" (at 109.22 182.88 0)
       (effects (font (size 1.27 1.27)) (justify left))
     )
@@
       (effects (font (size 1.27 1.27)) hide)
     )
+    (property "Manufacturer_Name" "--" (at 116.84 181.61 0)
+      (effects (font (size 1.27 1.27)) hide)
+    )
+    (property "Manufacturer_Part_Number" "--" (at 116.84 181.61 0)
+      (effects (font (size 1.27 1.27)) hide)
+    )
