File: hardware/main board/Opto2CH.kicad_sch (KiCad schematic)
At the start: 5 parts

Commit message: production version
Parts:
- O2: Manufacturer_Name (none) -> onsemi; Manufacturer_Part_Number (none) -> FOD8802DR2; Mouser Part Number (none) -> 863-FOD8802DR2; Mouser Price/Stock (none) -> https://www.mouser.pl/ProductDetail/onsemi/FOD8802DR2?qs=st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
- R40, R44: value 3.3k -> 2.7k; Manufacturer_Name (none) -> --; Manufacturer_Part_Number (none) -> --
- R45, R67: Manufacturer_Name (none) -> --; Manufacturer_Part_Number (none) -> --
Changed lines of the file:
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@@
       (effects (font (size 1.27 1.27)))
     )
-    (property "Value" "3.3k" (at 128.905 95.885 90)
+    (property "Value" "2.7k" (at 128.905 95.885 90)
       (effects (font (size 1.27 1.27)))
     )
@@
       (effects (font (size 1.27 1.27)) hide)
     )
+    (property "Manufacturer_Name" "--" (at 132.715 98.425 0)
+      (effects (font (size 1.27 1.27)) hide)
+    )
+    (property "Manufacturer_Part_Number" "--" (at 132.715 98.425 0)
+      (effects (font (size 1.27 1.27)) hide)
+    )
     (pin "1")
     (pin "2")
@@
       (effects (font (size 1.27 1.27)) hide)
     )
+    (property "Manufacturer_Name" "--" (at 155.575 94.615 0)
+      (effects (font (size 1.27 1.27)) hide)
+    )
+    (property "Manufacturer_Part_Number" "--" (at 155.575 94.615 0)
+      (effects (font (size 1.27 1.27)) hide)
+    )
     (pin "1")
     (pin "2")
@@
     )
     (property "Datasheet" "" (at 146.685 93.345 0)
+      (effects (font (size 1.27 1.27)) hide)
+    )
+    (property "Manufacturer_Name" "onsemi" (at 146.685 93.345 0)
+      (effects (font (size 1.27 1.27)) hide)
+    )
+    (property "Manufacturer_Part_Number" "FOD8802DR2" (at 146.685 93.345 0)
+      (effects (font (size 1.27 1.27)) hide)
+    )
+    (property "Mouser Part Number" "863-FOD8802DR2" (at 146.685 93.345 0)
+      (effects (font (size 1.27 1.27)) hide)
+    )
+    (property "Mouser Price/Stock" "https://www.mouser.pl/ProductDetail/onsemi/FOD8802DR2?qs=stqOd1AaK7%2FrKOyi9z09cg%3D%3D" (at 146.685 93.345 0)
       (effects (font (size 1.27 1.27)) hide)
     )
@@
       (effects (font (size 1.27 1.27)) hide)
     )
+    (property "Manufacturer_Name" "--" (at 160.02 94.615 0)
+      (effects (font (size 1.27 1.27)) hide)
+    )
+    (property "Manufacturer_Part_Number" "--" (at 160.02 94.615 0)
+      (effects (font (size 1.27 1.27)) hide)
+    )
     (pin "1")
     (pin "2")
@@
       (effects (font (size 1.27 1.27)))
     )
-    (property "Value" "3.3k" (at 128.905 104.775 90)
+    (property "Value" "2.7k" (at 128.905 104.775 90)
       (effects (font (size 1.27 1.27)))
     )
@@
       (effects (font (size 1.27 1.27)) hide)
     )
+    (property "Manufacturer_Name" "--" (at 132.715 107.315 0)
+      (effects (font (size 1.27 1.27)) hide)
+    )
+    (property "Manufacturer_Part_Number" "--" (at 132.715 107.315 0)
+      (effects (font (size 1.27 1.27)) hide)
+    )
