File: hardware/main board/PUTM_EV_BMS_HV_Master_2021.kicad_sch (KiCad schematic)
At the start: 18 parts, among them U2 STM32G484RETx, Y1 20MHz, Y2 32.768kHz

Commit message: done power plane layout
Parts:
- added R21: 10k, Resistor_SMD:R_0603_1608Metric, symbol Device:R_Small
Connections:
- net +3V3: now also R21.2
- net NRST: now also R21.1
Other:
- note removed: "Memory"
Changed lines of the file:
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@@
     (stroke (width 1) (type default) (color 132 0 0 1))
+  )
+  (wire (pts (xy 82.55 182.88) (xy 85.09 182.88))
+    (stroke (width 0) (type default))
   )
   (wire (pts (xy 38.1 59.69) (xy 40.64 59.69))
@@
     (stroke (width 0) (type default))
   )
+  (wire (pts (xy 74.93 182.88) (xy 77.47 182.88))
+    (stroke (width 0) (type default))
+  )
   (wire (pts (xy 163.83 85.09) (xy 166.37 85.09))
     (stroke (width 0) (type default))
@@
   (wire (pts (xy 76.2 72.39) (xy 78.74 72.39))
     (stroke (width 0) (type default))
-  )
-  (text "Memory" (at 247.65 21.59 0)
-    (effects (font (size 5 5) (thickness 1) bold) (justify left bottom))
   )
   (text "Power" (at 73.66 147.32 0)
@@
     (effects (font (size 1.27 1.27)) (justify left))
     (property "Intersheetrefs" "${INTERSHEET_REFS}" (at 103.4404 67.2306 0)
+      (effects (font (size 1.27 1.27)) (justify left) hide)
+    )
+  )
+  (global_label "NRST" (shape input) (at 85.09 182.88 0) (fields_autoplaced)
+    (effects (font (size 1.27 1.27)) (justify left))
+    (property "Intersheetrefs" "${INTERSHEET_REFS}" (at 92.1192 182.88 0)
       (effects (font (size 1.27 1.27)) (justify left) hide)
     )
@@
     )
   )
+  (symbol (lib_id "power:+3.3V") (at 74.93 182.88 90) (unit 1)
+    (in_bom yes) (on_board yes) (dnp no)
+    (property "Reference" "#PWR07" (at 78.74 182.88 0)
+      (effects (font (size 1.27 1.27)) hide)
+    )
+    (property "Value" "+3.3V" (at 71.12 182.88 0)
+      (effects (font (size 1.27 1.27)))
+    )
+    (property "Footprint" "" (at 74.93 182.88 0)
+      (effects (font (size 1.27 1.27)) hide)
+    )
+    (property "Datasheet" "" (at 74.93 182.88 0)
+      (effects (font (size 1.27 1.27)) hide)
+    )
+    (pin "1")
+    (instances
+      (project "PUTM_EV_BMS_HV_Master_2021"
+        (path "/b456cffc-d9d7-4c91-91f2-36ec9a65dd1b"
+          (reference "#PWR07") (unit 1)
+        )
+      )
+    )
+  )
   (symbol (lib_id "Mechanical:MountingHole_Pad") (at 161.29 190.5 90) (mirror x) (unit 1)
     (in_bom yes) (on_board yes) (dnp no)
@@
         )
       )
+    )
+  )
+  (symbol (lib_id "Device:R_Small") (at 80.01 182.88 270) (unit 1)
+    (in_bom yes) (on_board yes) (dnp no)
+    (property "Reference" "R21" (at 80.01 177.8 90)
+      (effects (font (size 1.27 1.27)) (justify top))
+    )
+    (property "Value" "10k" (at 80.01 181.61 90)
+      (effects (font (size 1.27 1.27)) (justify bottom))
+    )
+    (property "Footprint" "Resistor_SMD:R_0603_1608Metric" (at 80.01 182.88 0)
+      (effects (font (size 1.27 1.27)) hide)
+    )
+    (property "Datasheet" "~" (at 80.01 182.88 0)
+      (effects (font (size 1.27 1.27)) hide)
+    )
+    (pin "1")
+    (pin "2")
+    (instances
+      (project "PUTM_EV_BMS_HV_Master_2021"
+        (path "/b456cffc-d9d7-4c91-91f2-36ec9a65dd1b"
+          (reference "R21") (unit 1)
+        )
+      )

Commit message: repairing demaged branch~
Connections:
- net SIGNAL_AIR_M: now also U2.41 (PC9); no longer U2.39 (PC7)
- net SIGNAL_AIR_PRE: now also U2.39 (PC7); no longer U2.41 (PC9)
Other:
- sheet Fan drivers ports: added FAN1_CTRL, FAN2_CTRL, FAN3_CTRL, FAN4_CTRL, FAN5_CTRL, FAN6_CTRL, FAN7_CTRL; removed FAN_1_CONTROL, FAN_2_CONTROL, FAN_3_CONTROL, FAN_4_CONTROL, FAN_5_CONTROL, FAN_6_CONTROL, FAN_7_CONTROL
- moved on the sheet: R69, R71, R72

Commit message: production version
Parts:
- C40, C41: value 22pF -> 25pF; Manufacturer_Part_Number (none) -> 06035A250GAT2A; Mouser Part Number (none) -> 581-06035A250GAT2A; Mouser Price/Stock (none) -> https://www.mouser.pl/ProductDetail/KYOCERA-AVX/06035A250GA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
- C43, C44: value 22pF -> 20pF; Manufacturer_Name (none) -> --; Manufacturer_Part_Number (none) -> --
- D5, D6, D7, H1, H2, H9, R21, R34, R42, R69, R71, R72: Manufacturer_Name (none) -> --; Manufacturer_Part_Number (none) -> --
- U2: Manufacturer_Part_Number (none) -> STM32G484RET6; Mouser Part Number (none) -> 511-STM32G484RET6; Mouser Price/Stock (none) -> https://www.mouser.pl/ProductDetail/STMicroelectronics/STM3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
- Y1: value 20MHz -> X322516MLB4SI; Manufacturer_Name (none) -> --; Manufacturer_Part_Number (none) -> --
- Y2: value 32.768kHz -> Q13FC1350000400; Manufacturer_Name (none) -> --; Manufacturer_Part_Number (none) -> --
Changed lines of the file:
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@@
       (effects (font (size 1.27 1.27)) (justify left))
     )
-    (property "Value" "22pF" (at 220.98 140.335 90)
+    (property "Value" "20pF" (at 220.98 140.335 90)
       (effects (font (size 1.27 1.27)) (justify left))
     )
@@
       (effects (font (size 1.27 1.27)) hide)
     )
+    (property "Manufacturer_Name" "--" (at 218.44 143.51 0)
+      (effects (font (size 1.27 1.27)) hide)
+    )
+    (property "Manufacturer_Part_Number" "--" (at 218.44 143.51 0)
+      (effects (font (size 1.27 1.27)) hide)
+    )
     (pin "1")
     (pin "2")
@@
       (effects (font (size 1.27 1.27)) (justify left))
     )
-    (property "Value" "22pF" (at 216.535 156.21 90)
+    (property "Value" "20pF" (at 216.535 156.21 90)
       (effects (font (size 1.27 1.27)) (justify left))
     )
@@
       (effects (font (size 1.27 1.27)) hide)
     )
+    (property "Manufacturer_Name" "--" (at 218.44 151.13 0)
+      (effects (font (size 1.27 1.27)) hide)
+    )
+    (property "Manufacturer_Part_Number" "--" (at 218.44 151.13 0)
+      (effects (font (size 1.27 1.27)) hide)
+    )
     (pin "1")
     (pin "2")
@@
       (effects (font (size 1.27 1.27)) hide)
     )
+    (property "Manufacturer_Name" "--" (at 148.59 190.5 0)
+      (effects (font (size 1.27 1.27)) hide)
+    )
+    (property "Manufacturer_Part_Number" "--" (at 148.59 190.5 0)
+      (effects (font (size 1.27 1.27)) hide)
+    )
     (instances
       (project "PUTM_EV_BMS_HV_Master_2021"
@@
       (effects (font (size 1.27 1.27)) hide)
     )
+    (property "Manufacturer_Name" "--" (at 217.17 81.28 0)
+      (effects (font (size 1.27 1.27)) hide)
+    )
+    (property "Manufacturer_Part_Number" "--" (at 217.17 81.28 0)
+      (effects (font (size 1.27 1.27)) hide)
+    )
     (pin "1")
     (pin "2")
@@
     )
     (property "Datasheet" "~" (at 217.17 87.63 90)
+      (effects (font (size 1.27 1.27)) hide)
+    )
+    (property "Manufacturer_Name" "--" (at 217.17 87.63 0)
+      (effects (font (size 1.27 1.27)) hide)
+    )
+    (property "Manufacturer_Part_Number" "--" (at 217.17 87.63 0)
       (effects (font (size 1.27 1.27)) hide)
     )
@@
       (effects (font (size 1.27 1.27)) hide)
     )
+    (property "Manufacturer_Name" "--" (at 217.17 93.98 0)
+      (effects (font (size 1.27 1.27)) hide)
+    )
+    (property "Manufacturer_Part_Number" "--" (at 217.17 93.98 0)
+      (effects (font (size 1.27 1.27)) hide)
+    )
     (pin "1")
     (pin "2")
@@
       (effects (font (size 1.27 1.27)) hide)
     )
+    (property "Manufacturer_Name" "--" (at 209.55 81.28 0)
+      (effects (font (size 1.27 1.27)) hide)
+    )
+    (property "Manufacturer_Part_Number" "--" (at 209.55 81.28 0)
+      (effects (font (size 1.27 1.27)) hide)
+    )
     (pin "1")
     (pin "2")
@@
       (effects (font (size 1.27 1.27)) hide)
     )
+    (property "Manufacturer_Name" "--" (at 209.55 87.63 0)
+      (effects (font (size 1.27 1.27)) hide)
+    )
+    (property "Manufacturer_Part_Number" "--" (at 209.55 87.63 0)
+      (effects (font (size 1.27 1.27)) hide)
+    )
     (pin "1")
     (pin "2")
@@
       (effects (font (size 1.27 1.27)) hide)
     )
+    (property "Manufacturer_Name" "--" (at 209.55 93.98 0)
+      (effects (font (size 1.27 1.27)) hide)
+    )
+    (property "Manufacturer_Part_Number" "--" (at 209.55 93.98 0)
+      (effects (font (size 1.27 1.27)) hide)
+    )
     (pin "1")
     (pin "2")
@@
   (symbol (lib_id "Device:C_Small") (at 243.84 151.13 270) (unit 1)
     (in_bom yes) (on_board yes) (dnp no)
-    (property "Reference" "C41" (at 241.935 154.305 90)
-      (effects (font (size 1.27 1.27)) (justify left))
-    )
-    (property "Value" "22pF" (at 241.935 156.21 90)
-      (effects (font (size 1.27 1.27)) (justify left))
+    (property "Reference" "C41" (at 245.11 154.94 90)
+      (effects (font (size 1.27 1.27)))
+    )
+    (property "Value" "25pF" (at 245.11 157.48 90)
+      (effects (font (size 1.27 1.27)))
     )
     (property "Footprint" "Capacitor_SMD:C_0603_1608Metric" (at 243.84 151.13 0)
@@
       (effects (font (size 1.27 1.27)) hide)
     )
+    (property "Manufacturer_Part_Number" "06035A250GAT2A" (at 243.84 151.13 0)
+      (effects (font (size 1.27 1.27)) hide)
+    )
+    (property "Mouser Part Number" "581-06035A250GAT2A" (at 243.84 151.13 0)
+      (effects (font (size 1.27 1.27)) hide)
+    )
+    (property "Mouser Price/Stock" "https://www.mouser.pl/ProductDetail/KYOCERA-AVX/06035A250GAT2A?qs=EbDiPP9peV9MB5ntHldHqw%3D%3D" (at 243.84 151.13 0)
+      (effects (font (size 1.27 1.27)) hide)
+    )
     (pin "1")
     (pin "2")
@@
   (symbol (lib_id "Device:C_Small") (at 243.84 143.51 90) (unit 1)
     (in_bom yes) (on_board yes) (dnp no)
-    (property "Reference" "C40" (at 245.745 138.43 90)
-      (effects (font (size 1.27 1.27)) (justify left))
-    )
-    (property "Value" "22pF" (at 246.38 140.335 90)
-      (effects (font (size 1.27 1.27)) (justify left))
+    (property "Reference" "C40" (at 243.84 137.16 90)
+      (effects (font (size 1.27 1.27)))
+    )
+    (property "Value" "25pF" (at 243.84 139.7 90)
+      (effects (font (size 1.27 1.27)))
     )
     (property "Footprint" "Capacitor_SMD:C_0603_1608Metric" (at 243.84 143.51 0)
@@
       (effects (font (size 1.27 1.27)) hide)
     )
+    (property "Manufacturer_Part_Number" "06035A250GAT2A" (at 243.84 143.51 0)
+      (effects (font (size 1.27 1.27)) hide)
+    )
+    (property "Mouser Part Number" "581-06035A250GAT2A" (at 243.84 143.51 0)
+      (effects (font (size 1.27 1.27)) hide)
+    )
+    (property "Mouser Price/Stock" "https://www.mouser.pl/ProductDetail/KYOCERA-AVX/06035A250GAT2A?qs=EbDiPP9peV9MB5ntHldHqw%3D%3D" (at 243.84 143.51 0)
+      (effects (font (size 1.27 1.27)) hide)
+    )
     (pin "1")
     (pin "2")
@@
     )
     (property "Datasheet" "~" (at 148.59 182.88 0)
+      (effects (font (size 1.27 1.27)) hide)
+    )
+    (property "Manufacturer_Name" "--" (at 148.59 182.88 0)
+      (effects (font (size 1.27 1.27)) hide)
+    )
+    (property "Manufacturer_Part_Number" "--" (at 148.59 182.88 0)
       (effects (font (size 1.27 1.27)) hide)
     )
@@
     )
     (property "Datasheet" "https://www.st.com/resource/en/datasheet/stm32g484re.pdf" (at 58.42 77.47 0)
+      (effects (font (size 1.27 1.27)) hide)
+    )
+    (property "Manufacturer_Part_Number" "STM32G484RET6" (at 58.42 77.47 0)
+      (effects (font (size 1.27 1.27)) hide)
+    )
+    (property "Mouser Part Number" "511-STM32G484RET6" (at 58.42 77.47 0)
+      (effects (font (size 1.27 1.27)) hide)
+    )
+    (property "Mouser Price/Stock" "https://www.mouser.pl/ProductDetail/STMicroelectronics/STM32G484RET6?qs=uwxL4vQweFOtmhtzOZPifQ%3D%3D" (at 58.42 77.47 0)
       (effects (font (size 1.27 1.27)) hide)
     )
@@
       (effects (font (size 1.27 1.27)) hide)
     )
+    (property "Manufacturer_Name" "--" (at 106.68 190.5 0)
+      (effects (font (size 1.27 1.27)) hide)
+    )
+    (property "Manufacturer_Part_Number" "--" (at 106.68 190.5 0)
+      (effects (font (size 1.27 1.27)) hide)
+    )
     (pin "1")
     (pin "2")
@@
     )
     (property "Datasheet" "~" (at 161.29 190.5 0)
+      (effects (font (size 1.27 1.27)) hide)
+    )
+    (property "Manufacturer_Name" "--" (at 161.29 190.5 0)
+      (effects (font (size 1.27 1.27)) hide)
+    )
+    (property "Manufacturer_Part_Number" "--" (at 161.29 190.5 0)
       (effects (font (size 1.27 1.27)) hide)
     )
@@
       (effects (font (size 1.27 1.27)) hide)
     )
+    (property "Manufacturer_Name" "--" (at 80.01 182.88 0)
+      (effects (font (size 1.27 1.27)) hide)
+    )
+    (property "Manufacturer_Part_Number" "--" (at 80.01 182.88 0)
+      (effects (font (size 1.27 1.27)) hide)
+    )
     (pin "1")
     (pin "2")
@@
       (effects (font (size 1.27 1.27)) hide)
     )
+    (property "Manufacturer_Name" "--" (at 106.68 182.88 0)
+      (effects (font (size 1.27 1.27)) hide)
+    )
+    (property "Manufacturer_Part_Number" "--" (at 106.68 182.88 0)
+      (effects (font (size 1.27 1.27)) hide)
+    )
     (pin "1")
     (pin "2")
@@
   (symbol (lib_id "Device:Crystal_GND24_Small") (at 222.25 147.32 90) (unit 1)
     (in_bom yes) (on_board yes) (dnp no)
-    (property "Reference" "Y1" (at 224.79 138.43 90)
-      (effects (font (size 1.27 1.27)))
-    )
-    (property "Value" "20MHz" (at 224.79 140.335 90)
+    (property "Reference" "Y1" (at 229.87 137.16 90)
+      (effects (font (size 1.27 1.27)))
+    )
+    (property "Value" "X322516MLB4SI" (at 229.87 139.7 90)
       (effects (font (size 1.27 1.27)))
     )
@@
     )
     (property "Datasheet" "~" (at 222.25 147.32 0)
+      (effects (font (size 1.27 1.27)) hide)
+    )
+    (property "Manufacturer_Name" "--" (at 222.25 147.32 0)
+      (effects (font (size 1.27 1.27)) hide)
+    )
+    (property "Manufacturer_Part_Number" "--" (at 222.25 147.32 0)
       (effects (font (size 1.27 1.27)) hide)
     )
@@
   )
   (symbol (lib_id "Device:Crystal_Small") (at 247.65 147.32 90) (unit 1)
-    (in_bom yes) (on_board yes) (dnp no) (fields_autoplaced)
-    (property "Reference" "Y2" (at 250.19 146.0499 90)
-      (effects (font (size 1.27 1.27)) (justify right))
-    )
-    (property "Value" "32.768kHz" (at 250.19 148.5899 90)
+    (in_bom yes) (on_board yes) (dnp no)
+    (property "Reference" "Y2" (at 260.35 144.78 90)
+      (effects (font (size 1.27 1.27)) (justify right))
+    )
+    (property "Value" "Q13FC1350000400" (at 252.73 147.32 90)
       (effects (font (size 1.27 1.27)) (justify right))
     )
@@
       (effects (font (size 1.27 1.27)) hide)
     )
+    (property "Manufacturer_Name" "--" (at 247.65 147.32 0)
+      (effects (font (size 1.27 1.27)) hide)
+    )
+    (property "Manufacturer_Part_Number" "--" (at 247.65 147.32 0)
+      (effects (font (size 1.27 1.27)) hide)
+    )
