File: hardware/main board/Power.kicad_sch (KiCad schematic)
At the start: 46 parts, among them IC13 MAX17643ATC+, IC14 RTQ2965GSP-QA, U5 LM1117-3.3

Commit message: done power plane layout
Parts:
- added C8: 47uF, Capacitor_SMD:C_0603_1608Metric, symbol Device:C_Small
- C68: value 22uF -> 47uF
Connections:
- net +5V: now also C8.1
- net GND: now also C8.2
Other:
- moved on the sheet: R1

Commit message: production version
Parts:
- C11, C3: Manufacturer_Part_Number (none) -> CGA6P1X7R1N106K250AC; Mouser Part Number (none) -> 810-CGA6P1X7R1N106K2; Mouser Price/Stock (none) -> https://www.mouser.pl/ProductDetail/TDK/CGA6P1X7R1N106K250A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
- C12, C15: Manufacturer_Part_Number (none) -> C0603C105K8RACTU; Mouser Part Number (none) -> 80-C0603C105K8R; Mouser Price/Stock (none) -> https://www.mouser.pl/ProductDetail/KEMET/C0603C105K8RACTU?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
- C14: Manufacturer_Part_Number (none) -> VZS101M1ATR-0506; Mouser Part Number (none) -> 140-VZS101M1ATR0506; Mouser Price/Stock (none) -> https://www.mouser.pl/ProductDetail/Lelon/VZS101M1ATR-0506?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
- C16, C19, C50, C51, C52, C54, C55, C66: Manufacturer_Name (none) -> --; Manufacturer_Part_Number (none) -> --
- C24: Manufacturer_Part_Number (none) -> CL32B225KCJSNNE; Mouser Part Number (none) -> 187-CL32B225KCJSNNE; Mouser Price/Stock (none) -> https://www.mouser.pl/ProductDetail/Samsung-Electro-Mechani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
- C61: Manufacturer_Part_Number (none) -> CC0603KRX7R9BB123; Mouser Part Number (none) -> 603-CC603KRX7R9BB123; Mouser Price/Stock (none) -> https://www.mouser.pl/ProductDetail/YAGEO/CC0603KRX7R9BB123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
- C62: Manufacturer_Part_Number (none) -> 06035A100JAT2A; Mouser Part Number (none) -> 581-06035A100J; Mouser Price/Stock (none) -> https://www.mouser.pl/ProductDetail/KYOCERA-AVX/06035A100JA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
- C65, C71: Manufacturer_Part_Number (none) -> CL10B104KC8NNNC; Mouser Part Number (none) -> 187-CL10B104KC8NNNC; Mouser Price/Stock (none) -> https://www.mouser.pl/ProductDetail/Samsung-Electro-Mechani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
- C67: Manufacturer_Part_Number (none) -> CL10A225KO8NNWC; Mouser Part Number (none) -> 187-CL10A225KO8NNWC; Mouser Price/Stock (none) -> https://www.mouser.pl/ProductDetail/Samsung-Electro-Mechani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
- C68, C8: Manufacturer_Part_Number (none) -> CM105X5R476M06AT; Mouser Part Number (none) -> 581-CM105X5R476M06AT; Mouser Price/Stock (none) -> https://www.mouser.pl/ProductDetail/KYOCERA-AVX/CM105X5R476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
- C69: Manufacturer_Part_Number (none) -> 06035C562KAT2A; Mouser Part Number (none) -> 581-06035C562K; Mouser Price/Stock (none) -> https://www.mouser.pl/ProductDetail/KYOCERA-AVX/06035C562KA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
- C72: Manufacturer_Part_Number (none) -> 865080342006; Mouser Part Number (none) -> 710-865080342006; Mouser Price/Stock (none) -> https://www.mouser.pl/ProductDetail/Wurth-Elektronik/865080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
- D1, D21: Manufacturer_Part_Number (none) -> TSZU52C13 RGG; Mouser Part Number (none) -> 821-TSZU52C13RGG; Mouser Price/Stock (none) -> https://www.mouser.pl/ProductDetail/Taiwan-Semiconductor/TS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
- D11, D3: Manufacturer_Part_Number (none) -> SMBJ26CA-13-F; Mouser Part Number (none) -> 621-SMBJ26CA-13-F; Mouser Price/Stock (none) -> https://www.mouser.pl/ProductDetail/Diodes-Incorporated/SMB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
- D15: Manufacturer_Part_Number (none) -> VSSB410S-E3/52T; Mouser Part Number (none) -> 625-VSSB410S-E3/52T; Mouser Price/Stock (none) -> https://www.mouser.pl/ProductDetail/Vishay-General-Semicond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
- F2, F3: value 1A -> 0.5A; Manufacturer_Part_Number (none) -> 0ZCH0050FF2G; Mouser Part Number (none) -> 530-0ZCH0050FF2G; Mouser Price/Stock (none) -> https://www.mouser.pl/ProductDetail/Bel-Fuse/0ZCH0050FF2G?q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
- FB1: value ~ -> GZ1608D601TF; Manufacturer_Part_Number (none) -> --
- IC14: Mouser Part Number (none) -> 835-RTQ2965GSP-QA; Mouser Price/Stock (none) -> https://www.mouser.pl/ProductDetail/Richtek/RTQ2965GSP-QA?q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
- L11: Manufacturer_Part_Number (none) -> XAL5050-103MEC; Mouser Part Number (none) -> 994-XAL5050-103MEC; Mouser Price/Stock (none) -> https://www.mouser.pl/ProductDetail/Coilcraft/XAL5050-103ME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
- L3: value 10uH -> 33uH; Manufacturer_Part_Number (none) -> SRP1038CC-330M; Mouser Part Number (none) -> 652-SRP1038CC-330M; Mouser Price/Stock (none) -> https://www.mouser.pl/ProductDetail/Bourns/SRP1038CC-330M?q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
- L4, L5: value 6.8uH -> 4.7uH; Manufacturer_Part_Number (none) -> LQM31PN4R7M00L; Mouser Part Number (none) -> 81-LQM31PN4R7M00L; Mouser Price/Stock (none) -> https://www.mouser.pl/ProductDetail/Murata-Electronics/LQM3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
- R1: Manufacturer_Part_Number (none) -> CRCW060340K2FKEB; Mouser Part Number (none) -> 71-CRCW060340K2FKEB; Mouser Price/Stock (none) -> https://www.mouser.pl/ProductDetail/Vishay-Dale/CRCW060340K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
- R1: value 4.7 -> 4.7R; Manufacturer_Part_Number (none) -> CRCW06034R70FKEA; Mouser Part Number (none) -> 71-CRCW06034R70FKEA; Mouser Price/Stock (none) -> https://www.mouser.pl/ProductDetail/Vishay-Dale/CRCW06034R7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
- R1: Manufacturer_Part_Number (none) -> CRCW060310K5FKEA; Mouser Part Number (none) -> 71-CRCW0603-10.5K-E3; Mouser Price/Stock (none) -> https://www.mouser.pl/ProductDetail/Vishay-Dale/CRCW060310K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
- R1: Manufacturer_Part_Number (none) -> CRCW060320K5FKEA; Mouser Part Number (none) -> 71-CRCW0603-20.5K-E3; Mouser Price/Stock (none) -> https://www.mouser.pl/ProductDetail/Vishay-Dale/CRCW060320K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
- R1: Manufacturer_Part_Number (none) -> RT0603FRE0723K2L; Mouser Part Number (none) -> 603-RT0603FRE0723K2L; Mouser Price/Stock (none) -> https://www.mouser.pl/ProductDetail/YAGEO/RT0603FRE0723K2L?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
- R1: Manufacturer_Part_Number (none) -> AC0603FR-07392KL; Mouser Part Number (none) -> 603-AC0603FR-07392KL; Mouser Price/Stock (none) -> https://www.mouser.pl/ProductDetail/YAGEO/AC0603FR-07392KL?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
- R1: Manufacturer_Part_Number (none) -> RT0603FRE07105KL; Mouser Part Number (none) -> 603-RT0603FRE07105KL; Mouser Price/Stock (none) -> https://www.mouser.pl/ProductDetail/YAGEO/RT0603FRE07105KL?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
- R1: Manufacturer_Part_Number (none) -> AC0603FR-07147KL; Mouser Part Number (none) -> 603-AC0603FR-07147KL; Mouser Price/Stock (none) -> https://www.mouser.pl/ProductDetail/YAGEO/AC0603FR-07147KL?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
- U5: Manufacturer_Part_Number (none) -> LM1117MP-3.3/NOPB; Mouser Part Number (none) -> 926-LM1117MP-3.3NOPB; Mouser Price/Stock (none) -> https://www.mouser.pl/ProductDetail/Texas-Instruments/LM111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
Other:
- note removed: "z jakiegoś powodu komunikacja dalej nawala podczas klikania airami - za duże pobory?"
