File: hardware/main board/Safeties.kicad_sch (KiCad schematic)
At the start: 20 parts, among them K2 6-1419128-4, Q2 2N7002, Q4 2N7002, Q8 Q_PMOS_GSD, U14 74AUP1G32, U8 74LVC1G86

Commit message: production version
Parts:
- C25, C30, C63, C64, D9, JP4, Q2, Q4, R1, R11, R2, R3, R32, R38, R77: Manufacturer_Name (none) -> --; Manufacturer_Part_Number (none) -> --
- D12: Manufacturer_Part_Number (none) -> SS16-LTP; Mouser Part Number (none) -> 833-SS16-LTP; Mouser Price/Stock (none) -> https://www.mouser.pl/ProductDetail/Micro-Commercial-Compon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
- Q8: value Q_PMOS_GSD -> AO3400A; Manufacturer_Name (none) -> --; Manufacturer_Part_Number (none) -> --
- U14: Manufacturer_Part_Number (none) -> SN74AUP1G32DBVR; Mouser Part Number (none) -> 595-SN74AUP1G32DBVR; Mouser Price/Stock (none) -> https://www.mouser.pl/ProductDetail/Texas-Instruments/SN74A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
- U8: Manufacturer_Part_Number (none) -> SN74LVC1G86DBVR; Mouser Part Number (none) -> 595-SN74LVC1G86DBVR; Mouser Price/Stock (none) -> https://www.mouser.pl/ProductDetail/Texas-Instruments/SN74L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
Changed lines of the file:
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@@
+      (effects (font (size 1.27 1.27)) hide)
+    )
+    (property "Manufacturer_Part_Number" "SN74LVC1G86DBVR" (at 97.79 125.73 0)
+      (effects (font (size 1.27 1.27)) hide)
+    )
+    (property "Mouser Part Number" "595-SN74LVC1G86DBVR" (at 97.79 125.73 0)
+      (effects (font (size 1.27 1.27)) hide)
+    )
+    (property "Mouser Price/Stock" "https://www.mouser.pl/ProductDetail/Texas-Instruments/SN74LVC1G86DBVR?qs=d9gICRQKuCcyH%2F0J6yE9tQ%3D%3D" (at 97.79 125.73 0)
       (effects (font (size 1.27 1.27)) hide)
     )
@@
       (effects (font (size 1.27 1.27)) hide)
     )
+    (property "Manufacturer_Name" "--" (at 175.26 110.49 0)
+      (effects (font (size 1.27 1.27)) hide)
+    )
+    (property "Manufacturer_Part_Number" "--" (at 175.26 110.49 0)
+      (effects (font (size 1.27 1.27)) hide)
+    )
     (pin "1")
     (pin "2")
@@
       (effects (font (size 1.27 1.27)) (justify right))
     )
-    (property "Value" "Q_PMOS_GSD" (at 227.33 55.88 0)
+    (property "Value" "AO3400A" (at 227.33 55.88 0)
       (effects (font (size 1.27 1.27)) (justify right))
     )
@@
       (effects (font (size 1.27 1.27)) hide)
     )
+    (property "Manufacturer_Name" "--" (at 224.79 63.5 0)
+      (effects (font (size 1.27 1.27)) hide)
+    )
+    (property "Manufacturer_Part_Number" "--" (at 224.79 63.5 0)
+      (effects (font (size 1.27 1.27)) hide)
+    )
     (pin "1")
     (pin "2")
@@
       (effects (font (size 1.27 1.27)) hide)
     )
+    (property "Manufacturer_Name" "--" (at 76.2 127 0)
+      (effects (font (size 1.27 1.27)) hide)
+    )
+    (property "Manufacturer_Part_Number" "--" (at 76.2 127 0)
+      (effects (font (size 1.27 1.27)) hide)
+    )
     (pin "1")
     (pin "2")
@@
     )
     (property "Datasheet" "~" (at 212.09 81.28 90)
+      (effects (font (size 1.27 1.27)) hide)
+    )
+    (property "Manufacturer_Part_Number" "SS16-LTP" (at 212.09 81.28 0)
+      (effects (font (size 1.27 1.27)) hide)
+    )
+    (property "Mouser Part Number" "833-SS16-LTP" (at 212.09 81.28 0)
+      (effects (font (size 1.27 1.27)) hide)
+    )
+    (property "Mouser Price/Stock" "https://www.mouser.pl/ProductDetail/Micro-Commercial-Components-MCC/SS16-LTP?qs=cLwp4wpikzDsiZm8qAd%2Fng%3D%3D" (at 212.09 81.28 0)
       (effects (font (size 1.27 1.27)) hide)
     )
@@
     )
     (property "Datasheet" "~" (at 123.19 130.81 0)
+      (effects (font (size 1.27 1.27)) hide)
+    )
+    (property "Manufacturer_Name" "--" (at 123.19 130.81 0)
+      (effects (font (size 1.27 1.27)) hide)
+    )
+    (property "Manufacturer_Part_Number" "--" (at 123.19 130.81 0)
       (effects (font (size 1.27 1.27)) hide)
     )
@@
       (effects (font (size 1.27 1.27)) hide)
     )
+    (property "Manufacturer_Name" "--" (at 162.56 132.08 0)
+      (effects (font (size 1.27 1.27)) hide)
+    )
+    (property "Manufacturer_Part_Number" "--" (at 162.56 132.08 0)
+      (effects (font (size 1.27 1.27)) hide)
+    )
     (pin "1")
     (pin "2")
@@
     )
     (property "Datasheet" "~" (at 181.61 132.08 90)
+      (effects (font (size 1.27 1.27)) hide)
+    )
+    (property "Manufacturer_Name" "--" (at 181.61 132.08 0)
+      (effects (font (size 1.27 1.27)) hide)
+    )
+    (property "Manufacturer_Part_Number" "--" (at 181.61 132.08 0)
       (effects (font (size 1.27 1.27)) hide)
     )
@@
       (effects (font (size 1.27 1.27)) (justify left) hide)
     )
+    (property "Manufacturer_Name" "--" (at 130.81 125.73 0)
+      (effects (font (size 1.27 1.27)) hide)
+    )
+    (property "Manufacturer_Part_Number" "--" (at 130.81 125.73 0)
+      (effects (font (size 1.27 1.27)) hide)
+    )
     (pin "1")
     (pin "2")
@@
       (effects (font (size 1.27 1.27)) hide)
     )
+    (property "Manufacturer_Name" "--" (at 181.61 124.46 0)
+      (effects (font (size 1.27 1.27)) hide)
+    )
+    (property "Manufacturer_Part_Number" "--" (at 181.61 124.46 0)
+      (effects (font (size 1.27 1.27)) hide)
+    )
     (pin "1")
     (pin "2")
@@
     )
     (property "Datasheet" "~" (at 208.28 129.54 0)
+      (effects (font (size 1.27 1.27)) hide)
+    )
+    (property "Manufacturer_Name" "--" (at 208.28 129.54 0)
+      (effects (font (size 1.27 1.27)) hide)
+    )
+    (property "Manufacturer_Part_Number" "--" (at 208.28 129.54 0)
       (effects (font (size 1.27 1.27)) hide)
     )
@@
       (effects (font (size 1.27 1.27)) (justify left) hide)
     )
+    (property "Manufacturer_Name" "--" (at 224.79 129.54 0)
+      (effects (font (size 1.27 1.27)) hide)
+    )
+    (property "Manufacturer_Part_Number" "--" (at 224.79 129.54 0)
+      (effects (font (size 1.27 1.27)) hide)
+    )
     (pin "1")
     (pin "2")
@@
       (effects (font (size 1.27 1.27)) hide)
     )
+    (property "Manufacturer_Name" "--" (at 102.87 115.57 0)
+      (effects (font (size 1.27 1.27)) hide)
+    )
+    (property "Manufacturer_Part_Number" "--" (at 102.87 115.57 0)
+      (effects (font (size 1.27 1.27)) hide)
+    )
     (pin "1")
     (pin "2")
@@
     )
     (property "Datasheet" "http://www.ti.com/lit/sg/scyt129e/scyt129e.pdf" (at 171.45 119.38 0)
+      (effects (font (size 1.27 1.27)) hide)
+    )
+    (property "Manufacturer_Part_Number" "SN74AUP1G32DBVR" (at 171.45 119.38 0)
+      (effects (font (size 1.27 1.27)) hide)
+    )
+    (property "Mouser Part Number" "595-SN74AUP1G32DBVR" (at 171.45 119.38 0)
+      (effects (font (size 1.27 1.27)) hide)
+    )
+    (property "Mouser Price/Stock" "https://www.mouser.pl/ProductDetail/Texas-Instruments/SN74AUP1G32DBVR?qs=iO7mgM19OaZv5mY3EPipeg%3D%3D" (at 171.45 119.38 0)
       (effects (font (size 1.27 1.27)) hide)
     )
@@
       (effects (font (size 1.27 1.27)) hide)
     )
+    (property "Manufacturer_Name" "--" (at 81.28 132.08 0)
+      (effects (font (size 1.27 1.27)) hide)
+    )
+    (property "Manufacturer_Part_Number" "--" (at 81.28 132.08 0)
+      (effects (font (size 1.27 1.27)) hide)
+    )
     (pin "1")
     (pin "2")
@@
       (effects (font (size 1.27 1.27)) hide)
     )
+    (property "Manufacturer_Name" "--" (at 217.17 134.62 0)
+      (effects (font (size 1.27 1.27)) hide)
+    )
+    (property "Manufacturer_Part_Number" "--" (at 217.17 134.62 0)
+      (effects (font (size 1.27 1.27)) hide)
+    )
     (pin "1")
     (pin "2")
@@
     )
     (property "Datasheet" "~" (at 147.32 125.73 0)
+      (effects (font (size 1.27 1.27)) hide)
+    )
+    (property "Manufacturer_Name" "--" (at 147.32 125.73 0)
+      (effects (font (size 1.27 1.27)) hide)
+    )
+    (property "Manufacturer_Part_Number" "--" (at 147.32 125.73 0)
       (effects (font (size 1.27 1.27)) hide)
     )
@@
       (effects (font (size 1.27 1.27)) hide)
     )
+    (property "Manufacturer_Name" "--" (at 147.32 113.03 0)
+      (effects (font (size 1.27 1.27)) hide)
+    )
+    (property "Manufacturer_Part_Number" "--" (at 147.32 113.03 0)
+      (effects (font (size 1.27 1.27)) hide)
+    )
     (pin "1")
     (pin "2")
@@
       (effects (font (size 1.27 1.27)) hide)
     )
+    (property "Manufacturer_Name" "--" (at 71.12 132.08 0)
+      (effects (font (size 1.27 1.27)) hide)
+    )
+    (property "Manufacturer_Part_Number" "--" (at 71.12 132.08 0)
+      (effects (font (size 1.27 1.27)) hide)
+    )
